File: hardware/01-ECAD/01-KiCAD Files/AWG1000/AWG1000.kicad_pcb (KiCad board)
At the start: 0 parts

Commit message: WIP: update
Parts:
- added C1: 220uF, awg1000:EEE-FK1H221GP, F.Cu at (43.2, 120.0)
- added C2: 220uF, awg1000:EEE-FK1H221GP, F.Cu at (43.2, 134.0)
- added J1: B4P-VH(LF)(SN), Connector_JST:JST_VH_B4P-VH_1x04_P3.96mm_Vertical, F.Cu at (31.8, 136.2)
- added U1: MC34PF3000A5EP, Package_DFN_QFN:NXP_LQFN-48-1EP_7x7mm_P0.5mm_EP3.5x3.5mm_16xMask0.45x0.45_ThermalVias, F.Cu at (65.8, 121.9)
Other:
- copper layers 0 -> 2
