File: hardware/01-ECAD/01-KiCAD Files/AWG1000/AWG1000.kicad_pcb (KiCad board)
At the start: 2 copper layers, 4 parts, among them J1 B4P-VH(LF)(SN), U1 MC34PF3000A5EP

Commit message: Update.
Parts:
- added C1: 4.7uF, awg1000:C0402_L, F.Cu at (-200.9, 13.7)
- added C10: 0.47uF, Resistor_SMD:R_0402_1005Metric_Pad0.72x0.64mm_HandSolder, F.Cu at (28.9, 159.8)
- added C100: 22uF, Capacitor_SMD:C_0603_1608Metric_Pad1.08x0.95mm_HandSolder, F.Cu at (-113.5, -93.2)
- added C101: 22uF, Capacitor_SMD:C_0603_1608Metric_Pad1.08x0.95mm_HandSolder, F.Cu at (-112.5, -96.7)
- added C102: 220nF, Resistor_SMD:R_0402_1005Metric_Pad0.72x0.64mm_HandSolder, F.Cu at (-103.3, -86.5)
- added C103: 22uF, Capacitor_SMD:C_0603_1608Metric_Pad1.08x0.95mm_HandSolder, F.Cu at (-114.1, -96.7)
- added C104: 4.7uF, awg1000:C0402_L, F.Cu at (147.4, 144.0)
- added C105: 22uF, Capacitor_SMD:C_0603_1608Metric_Pad1.08x0.95mm_HandSolder, F.Cu at (-119.2, -83.3)
- added C106: 4.7uF, awg1000:C0402_L, F.Cu at (150.6, 142.0)
- added C107: 22uF, Capacitor_SMD:C_0603_1608Metric_Pad1.08x0.95mm_HandSolder, F.Cu at (-119.2, -84.8)
- added C108: 22uF, Capacitor_SMD:C_0603_1608Metric_Pad1.08x0.95mm_HandSolder, F.Cu at (-119.2, -87.9)
- added C109: 220nF, Resistor_SMD:R_0402_1005Metric_Pad0.72x0.64mm_HandSolder, F.Cu at (-103.3, -85.3)
- added C11: 0.47uF, Resistor_SMD:R_0402_1005Metric_Pad0.72x0.64mm_HandSolder, F.Cu at (57.6, -115.8)
- added C110: 22uF, Capacitor_SMD:C_0603_1608Metric_Pad1.08x0.95mm_HandSolder, F.Cu at (-119.2, -86.4)
- added C111: 220nF, Resistor_SMD:R_0402_1005Metric_Pad0.72x0.64mm_HandSolder, F.Cu at (-111.8, -80.3)
- added C112: 220nF, Resistor_SMD:R_0402_1005Metric_Pad0.72x0.64mm_HandSolder, F.Cu at (-111.8, -79.2)
- added C113: 4.7uF, awg1000:C0402_L, F.Cu at (133.6, 144.0)
- added C114: 4.7uF, awg1000:C0402_L, F.Cu at (136.9, 144.0)
- added C115: 4.7uF, awg1000:C0402_L, F.Cu at (136.9, 145.9)
- added C116: 4.7uF, awg1000:C0402_L, F.Cu at (133.6, 142.0)
- added C117: 4.7uF, awg1000:C0402_L, F.Cu at (130.4, 145.9)
- added C118: 4.7uF, awg1000:C0402_L, F.Cu at (130.4, 144.0)
- added C119: 0.1uF, Resistor_SMD:R_0402_1005Metric_Pad0.72x0.64mm_HandSolder, F.Cu at (5.36, -157.0)
- added C12: 0.47uF, Resistor_SMD:R_0402_1005Metric_Pad0.72x0.64mm_HandSolder, F.Cu at (-42.2, -143.7)
- added C120: 0.1uF, Resistor_SMD:R_0402_1005Metric_Pad0.72x0.64mm_HandSolder, F.Cu at (15.1, -159.0)
- added C121: 0.1uF, Resistor_SMD:R_0402_1005Metric_Pad0.72x0.64mm_HandSolder, F.Cu at (18.4, -161.0)
- added C122: 0.1uF, Resistor_SMD:R_0402_1005Metric_Pad0.72x0.64mm_HandSolder, F.Cu at (8.61, -159.0)
- added C123: 0.1uF, Resistor_SMD:R_0402_1005Metric_Pad0.72x0.64mm_HandSolder, F.Cu at (11.9, -161.0)
- added C124: 0.1uF, Resistor_SMD:R_0402_1005Metric_Pad0.72x0.64mm_HandSolder, F.Cu at (11.9, -155.1)
- added C125: 0.1uF, Resistor_SMD:R_0402_1005Metric_Pad0.72x0.64mm_HandSolder, F.Cu at (8.61, -155.1)
- added C126: 0.1uF, Resistor_SMD:R_0402_1005Metric_Pad0.72x0.64mm_HandSolder, F.Cu at (11.9, -157.0)
- added C127: 4.7uF, awg1000:C0402_L, F.Cu at (130.4, 142.0)
- added C128: 0.1uF, Resistor_SMD:R_0402_1005Metric_Pad0.72x0.64mm_HandSolder, F.Cu at (15.1, -157.0)
- added C129: 0.1uF, Resistor_SMD:R_0402_1005Metric_Pad0.72x0.64mm_HandSolder, F.Cu at (5.36, -161.0)
- added C130: 4.7uF, awg1000:C0402_L, F.Cu at (136.9, 142.0)
- added C131: 0.1uF, Resistor_SMD:R_0402_1005Metric_Pad0.72x0.64mm_HandSolder, F.Cu at (8.61, -161.0)
- added C132: 0.1uF, Resistor_SMD:R_0402_1005Metric_Pad0.72x0.64mm_HandSolder, F.Cu at (15.1, -161.0)
- added C133: 22uF, Resistor_SMD:R_0402_1005Metric_Pad0.72x0.64mm_HandSolder, B.Cu at (-113.9, -113.6)
- added C134: 22uF, Resistor_SMD:R_0402_1005Metric_Pad0.72x0.64mm_HandSolder, F.Cu at (-290.9, -253.2)
- added C135: 220nF, Resistor_SMD:R_0402_1005Metric_Pad0.72x0.64mm_HandSolder, B.Cu at (-112.6, -111.3)
- added C136: 220nF, Resistor_SMD:R_0402_1005Metric_Pad0.72x0.64mm_HandSolder, B.Cu at (-111.6, -111.3)
- added C137: 0.22uF, Resistor_SMD:R_0402_1005Metric_Pad0.72x0.64mm_HandSolder, F.Cu at (5.36, -155.1)
- added C138: 220nF, Resistor_SMD:R_0402_1005Metric_Pad0.72x0.64mm_HandSolder, B.Cu at (-111.0, -111.3)
- added C139: 220nF, Resistor_SMD:R_0402_1005Metric_Pad0.72x0.64mm_HandSolder, B.Cu at (-108.4, -112.4)
- added C14: 0.47uF, Resistor_SMD:R_0402_1005Metric_Pad0.72x0.64mm_HandSolder, F.Cu at (230.4, -65.3)
- added C140: 22uF, Resistor_SMD:R_0402_1005Metric_Pad0.72x0.64mm_HandSolder, F.Cu at (-286.9, -255.7)
- added C141: 220nF, Resistor_SMD:R_0402_1005Metric_Pad0.72x0.64mm_HandSolder, B.Cu at (-111.0, -112.4)
- added C142: 220nF, Resistor_SMD:R_0402_1005Metric_Pad0.72x0.64mm_HandSolder, B.Cu at (-112.6, -112.4)
- added C143: 0.22uF, Resistor_SMD:R_0402_1005Metric_Pad0.72x0.64mm_HandSolder, F.Cu at (11.9, -159.0)
- added C144: 220nF, Resistor_SMD:R_0402_1005Metric_Pad0.72x0.64mm_HandSolder, B.Cu at (-111.6, -112.4)
- added C145: 220nF, Resistor_SMD:R_0402_1005Metric_Pad0.72x0.64mm_HandSolder, B.Cu at (-113.2, -112.4)
- added C146: 22uF, Resistor_SMD:R_0402_1005Metric_Pad0.72x0.64mm_HandSolder, B.Cu at (-107.9, -113.6)
- added C147: 22uF, Resistor_SMD:R_0402_1005Metric_Pad0.72x0.64mm_HandSolder, F.Cu at (-286.9, -253.2)
- added C148: 0.22uF, Resistor_SMD:R_0402_1005Metric_Pad0.72x0.64mm_HandSolder, F.Cu at (8.61, -157.0)
- added C149: 220nF, Resistor_SMD:R_0402_1005Metric_Pad0.72x0.64mm_HandSolder, B.Cu at (-107.8, -114.7)
- added C15: 4.7uF, awg1000:C0402_L, F.Cu at (90.6, 162.1)
- added C150: 220nF, Resistor_SMD:R_0402_1005Metric_Pad0.72x0.64mm_HandSolder, B.Cu at (-106.8, -111.3)
- added C151: 0.22uF, Resistor_SMD:R_0402_1005Metric_Pad0.72x0.64mm_HandSolder, F.Cu at (5.36, -159.0)
- added C152: 22uF, Resistor_SMD:R_0402_1005Metric_Pad0.72x0.64mm_HandSolder, F.Cu at (-290.9, -255.7)
- added C153: 220nF, Resistor_SMD:R_0402_1005Metric_Pad0.72x0.64mm_HandSolder, B.Cu at (-107.8, -111.3)
- added C154: 220nF, Resistor_SMD:R_0402_1005Metric_Pad0.72x0.64mm_HandSolder, B.Cu at (-106.8, -114.7)
- added C155: 220nF, Resistor_SMD:R_0402_1005Metric_Pad0.72x0.64mm_HandSolder, B.Cu at (-107.8, -112.4)
- added C156: 220nF, Resistor_SMD:R_0402_1005Metric_Pad0.72x0.64mm_HandSolder, B.Cu at (-106.8, -112.4)
- added C157: 4.7uF, awg1000:C0402_L, B.Cu at (-123.4, -109.9)
- added C158: 4.7uF, awg1000:C0402_L, B.Cu at (-123.4, -108.7)
- added C159: 4.7uF, awg1000:C0402_L, F.Cu at (-127.3, -107.0)
- added C16: 33uF, Capacitor_SMD:CP_Elec_6.3x7.7, F.Cu at (35.0, 170.3)
- added C160: 22uF, Resistor_SMD:R_0402_1005Metric_Pad0.72x0.64mm_HandSolder, B.Cu at (-109.7, -116.6)
- added C161: 220nF, Resistor_SMD:R_0402_1005Metric_Pad0.72x0.64mm_HandSolder, B.Cu at (-113.2, -117.0)
- added C162: 220nF, Resistor_SMD:R_0402_1005Metric_Pad0.72x0.64mm_HandSolder, B.Cu at (-111.6, -117.0)
- added C163: 220nF, Resistor_SMD:R_0402_1005Metric_Pad0.72x0.64mm_HandSolder, B.Cu at (-111.0, -117.0)
- added C164: 4.7uF, awg1000:C0402_L, F.Cu at (-127.3, -110.1)
- added C165: 220nF, Resistor_SMD:R_0402_1005Metric_Pad0.72x0.64mm_HandSolder, B.Cu at (-114.2, -117.0)
- added C166: 220nF, Resistor_SMD:R_0402_1005Metric_Pad0.72x0.64mm_HandSolder, B.Cu at (-112.6, -117.0)
- added C167: 22uF, Resistor_SMD:R_0402_1005Metric_Pad0.72x0.64mm_HandSolder, B.Cu at (-305.2, -244.8)
- added C168: 220nF, Resistor_SMD:R_0402_1005Metric_Pad0.72x0.64mm_HandSolder, B.Cu at (-282.7, -243.1)
- added C169: 220nF, Resistor_SMD:R_0402_1005Metric_Pad0.72x0.64mm_HandSolder, B.Cu at (-286.1, -241.1)
- added C17: 10uF, Capacitor_SMD:C_1206_3216Metric, F.Cu at (68.8, -111.5)
- added C170: 22uF, Resistor_SMD:R_0402_1005Metric_Pad0.72x0.64mm_HandSolder, B.Cu at (-305.5, -252.7)
- added C171: 220nF, Resistor_SMD:R_0402_1005Metric_Pad0.72x0.64mm_HandSolder, B.Cu at (-283.6, -243.7)
- added C172: 220nF, Resistor_SMD:R_0402_1005Metric_Pad0.72x0.64mm_HandSolder, B.Cu at (-283.5, -245.5)
- added C173: 22uF, Resistor_SMD:R_0402_1005Metric_Pad0.72x0.64mm_HandSolder, B.Cu at (-109.7, -111.8)
- added C174: 220nF, Resistor_SMD:R_0402_1005Metric_Pad0.72x0.64mm_HandSolder, B.Cu at (-284.6, -243.6)
- added C175: 220nF, Resistor_SMD:R_0402_1005Metric_Pad0.72x0.64mm_HandSolder, B.Cu at (-282.2, -244.6)
- added C176: 22uF, Resistor_SMD:R_0402_1005Metric_Pad0.72x0.64mm_HandSolder, B.Cu at (-109.7, -119.0)
- added C177: 22uF, Resistor_SMD:R_0402_1005Metric_Pad0.72x0.64mm_HandSolder, B.Cu at (-117.7, -115.8)
- added C178: 220nF, Resistor_SMD:R_0402_1005Metric_Pad0.72x0.64mm_HandSolder, B.Cu at (-285.7, -243.4)
- added C179: 220nF, Resistor_SMD:R_0402_1005Metric_Pad0.72x0.64mm_HandSolder, B.Cu at (-286.1, -240.1)
- added C18: 33uF, Capacitor_SMD:CP_Elec_6.3x7.7, F.Cu at (-36.0, -134.3)
- added C180: 220nF, Resistor_SMD:R_0402_1005Metric_Pad0.72x0.64mm_HandSolder, B.Cu at (-279.2, -244.0)
- added C181: 220nF, Resistor_SMD:R_0402_1005Metric_Pad0.72x0.64mm_HandSolder, B.Cu at (-286.1, -242.0)
- added C182: 220nF, Resistor_SMD:R_0402_1005Metric_Pad0.72x0.64mm_HandSolder, B.Cu at (-286.1, -239.2)
- added C183: 220nF, Resistor_SMD:R_0402_1005Metric_Pad0.72x0.64mm_HandSolder, B.Cu at (-274.7, -238.6)
- added C184: 220nF, Resistor_SMD:R_0402_1005Metric_Pad0.72x0.64mm_HandSolder, B.Cu at (-278.3, -243.9)
- added C185: 220nF, Resistor_SMD:R_0402_1005Metric_Pad0.72x0.64mm_HandSolder, B.Cu at (-286.1, -236.8)
- added C186: 22uF, Resistor_SMD:R_0402_1005Metric_Pad0.72x0.64mm_HandSolder, B.Cu at (-109.7, -109.4)
- added C187: 22uF, Resistor_SMD:R_0402_1005Metric_Pad0.72x0.64mm_HandSolder, B.Cu at (-111.5, -113.6)
- added C188: 22uF, Resistor_SMD:R_0402_1005Metric_Pad0.72x0.64mm_HandSolder, B.Cu at (-109.7, -114.2)
- added C189: 22uF, Resistor_SMD:R_0402_1005Metric_Pad0.72x0.64mm_HandSolder, B.Cu at (-116.0, -117.4)
- added C19: 33uF, Capacitor_SMD:CP_Elec_6.3x7.7, F.Cu at (223.5, -65.5)
- added C190: 220nF, Resistor_SMD:R_0402_1005Metric_Pad0.72x0.64mm_HandSolder, B.Cu at (-114.8, -114.7)
- added C191: 220nF, Resistor_SMD:R_0402_1005Metric_Pad0.72x0.64mm_HandSolder, B.Cu at (-113.2, -114.7)
- added C192: 220nF, Resistor_SMD:R_0402_1005Metric_Pad0.72x0.64mm_HandSolder, B.Cu at (-111.6, -115.9)
- added C193: 220nF, Resistor_SMD:R_0402_1005Metric_Pad0.72x0.64mm_HandSolder, B.Cu at (-104.3, -126.2)
- added C194: 220nF, Resistor_SMD:R_0402_1005Metric_Pad0.72x0.64mm_HandSolder, B.Cu at (-108.4, -114.7)
- added C195: 220nF, Resistor_SMD:R_0402_1005Metric_Pad0.72x0.64mm_HandSolder, B.Cu at (-112.6, -114.7)
- added C196: 220nF, Resistor_SMD:R_0402_1005Metric_Pad0.72x0.64mm_HandSolder, B.Cu at (-112.6, -115.9)
- added C197: 220nF, Resistor_SMD:R_0402_1005Metric_Pad0.72x0.64mm_HandSolder, B.Cu at (-107.8, -115.9)
- added C198: 220nF, Resistor_SMD:R_0402_1005Metric_Pad0.72x0.64mm_HandSolder, B.Cu at (-111.0, -114.7)
- added C199: 220nF, Resistor_SMD:R_0402_1005Metric_Pad0.72x0.64mm_HandSolder, B.Cu at (-111.6, -109.4)
- added C2: 4.7uF, awg1000:C0402_L, F.Cu at (28.9, 162.1)
- added C20: 33uF, Capacitor_SMD:CP_Elec_6.3x7.7, F.Cu at (63.8, -105.9)
- added C200: 220nF, Resistor_SMD:R_0402_1005Metric_Pad0.72x0.64mm_HandSolder, B.Cu at (-106.8, -115.9)
- added C201: 220nF, Resistor_SMD:R_0402_1005Metric_Pad0.72x0.64mm_HandSolder, B.Cu at (-111.0, -115.9)
- added C202: 220nF, Resistor_SMD:R_0402_1005Metric_Pad0.72x0.64mm_HandSolder, B.Cu at (-111.6, -114.7)
- added C203: 220nF, Resistor_SMD:R_0402_1005Metric_Pad0.72x0.64mm_HandSolder, B.Cu at (-108.4, -109.4)
- added C204: 220nF, Resistor_SMD:R_0402_1005Metric_Pad0.72x0.64mm_HandSolder, B.Cu at (-114.8, -115.9)
- added C205: 220nF, Resistor_SMD:R_0402_1005Metric_Pad0.72x0.64mm_HandSolder, B.Cu at (-114.2, -115.9)
- added C206: 220nF, Resistor_SMD:R_0402_1005Metric_Pad0.72x0.64mm_HandSolder, B.Cu at (-114.2, -114.7)
- added C207: 220nF, Resistor_SMD:R_0402_1005Metric_Pad0.72x0.64mm_HandSolder, B.Cu at (-111.0, -109.4)
- added C208: 220nF, Resistor_SMD:R_0402_1005Metric_Pad0.72x0.64mm_HandSolder, B.Cu at (-113.2, -115.9)
- added C209: 220nF, Resistor_SMD:R_0402_1005Metric_Pad0.72x0.64mm_HandSolder, B.Cu at (-108.4, -115.9)
- added C21: 10uF, Capacitor_SMD:C_1206_3216Metric, F.Cu at (30.1, 170.5)
- added C210: 220nF, Resistor_SMD:R_0402_1005Metric_Pad0.72x0.64mm_HandSolder, F.Cu at (-244.4, -125.3)
- added C211: 22uF, Resistor_SMD:R_0402_1005Metric_Pad0.72x0.64mm_HandSolder, B.Cu at (-104.5, -113.6)
- added C212: 22uF, Resistor_SMD:R_0402_1005Metric_Pad0.72x0.64mm_HandSolder, B.Cu at (-106.4, -118.5)
- added C213: 22uF, Resistor_SMD:R_0402_1005Metric_Pad0.72x0.64mm_HandSolder, F.Cu at (-78.0, -106.0)
- added C214: 22uF, Resistor_SMD:R_0402_1005Metric_Pad0.72x0.64mm_HandSolder, F.Cu at (-94.7, -117.8)
- added C215: 22uF, Resistor_SMD:R_0402_1005Metric_Pad0.72x0.64mm_HandSolder, F.Cu at (-94.6, -124.9)
- added C216: 22uF, Resistor_SMD:R_0402_1005Metric_Pad0.72x0.64mm_HandSolder, F.Cu at (-77.9, -124.5)
- added C217: 22uF, Resistor_SMD:R_0402_1005Metric_Pad0.72x0.64mm_HandSolder, F.Cu at (-94.6, -110.3)
- added C218: 22uF, Resistor_SMD:R_0402_1005Metric_Pad0.72x0.64mm_HandSolder, F.Cu at (-94.7, -103.0)
- added C219: 220nF, Resistor_SMD:R_0402_1005Metric_Pad0.72x0.64mm_HandSolder, B.Cu at (-105.2, -116.3)
- added C22: 10uF, Capacitor_SMD:C_1206_3216Metric, F.Cu at (267.4, 137.0)
- added C22: 10uF, Capacitor_SMD:C_1206_3216Metric, F.Cu at (39.9, 164.3)
- added C220: 220nF, Resistor_SMD:R_0402_1005Metric_Pad0.72x0.64mm_HandSolder, B.Cu at (-105.2, -112.7)
- added C221: 220nF, Resistor_SMD:R_0402_1005Metric_Pad0.72x0.64mm_HandSolder, B.Cu at (-105.5, -117.8)
- added C222: 220nF, Resistor_SMD:R_0402_1005Metric_Pad0.72x0.64mm_HandSolder, B.Cu at (-105.2, -114.7)
- added C223: 220nF, Resistor_SMD:R_0402_1005Metric_Pad0.72x0.64mm_HandSolder, B.Cu at (-105.2, -110.9)
- added C224: 220nF, Resistor_SMD:R_0402_1005Metric_Pad0.72x0.64mm_HandSolder, B.Cu at (-105.2, -109.9)
- added C225: 220nF, Resistor_SMD:R_0402_1005Metric_Pad0.72x0.64mm_HandSolder, B.Cu at (-105.2, -115.7)
- added C226: 220nF, Resistor_SMD:R_0402_1005Metric_Pad0.72x0.64mm_HandSolder, B.Cu at (-105.2, -111.5)
- added C227: 220nF, Resistor_SMD:R_0402_1005Metric_Pad0.72x0.64mm_HandSolder, F.Cu at (-41.3, -261.0)
- added C228: 220nF, Resistor_SMD:R_0402_1005Metric_Pad0.72x0.64mm_HandSolder, F.Cu at (-80.5, -112.0)
- added C229: 220nF, Resistor_SMD:R_0402_1005Metric_Pad0.72x0.64mm_HandSolder, F.Cu at (-90.9, -127.0)
- added C23: 33uF, Capacitor_SMD:CP_Elec_6.3x7.7, F.Cu at (-145.7, -80.0)
- added C230: 220nF, Resistor_SMD:R_0402_1005Metric_Pad0.72x0.64mm_HandSolder, B.Cu at (-107.8, -117.9)
- added C231: 220nF, Resistor_SMD:R_0402_1005Metric_Pad0.72x0.64mm_HandSolder, F.Cu at (-88.3, -127.0)
- added C232: 220nF, Resistor_SMD:R_0402_1005Metric_Pad0.72x0.64mm_HandSolder, F.Cu at (-79.5, -100.1)
- added C233: 220nF, Resistor_SMD:R_0402_1005Metric_Pad0.72x0.64mm_HandSolder, F.Cu at (-88.3, -100.1)
- added C234: 220nF, Resistor_SMD:R_0402_1005Metric_Pad0.72x0.64mm_HandSolder, F.Cu at (-88.4, -115.1)
- added C235: 220nF, Resistor_SMD:R_0402_1005Metric_Pad0.72x0.64mm_HandSolder, F.Cu at (-93.4, -115.1)
- added C236: 220nF, Resistor_SMD:R_0402_1005Metric_Pad0.72x0.64mm_HandSolder, F.Cu at (-82.2, -115.1)
- added C237: 220nF, Resistor_SMD:R_0402_1005Metric_Pad0.72x0.64mm_HandSolder, F.Cu at (-93.4, -100.1)
- added C238: 220nF, Resistor_SMD:R_0402_1005Metric_Pad0.72x0.64mm_HandSolder, F.Cu at (-88.7, -112.0)
- added C239: 220nF, Resistor_SMD:R_0402_1005Metric_Pad0.72x0.64mm_HandSolder, F.Cu at (-82.0, -127.0)
- added C24: 220nF, Resistor_SMD:R_0402_1005Metric_Pad0.72x0.64mm_HandSolder, F.Cu at (66.6, -111.5)
- added C240: 220nF, Resistor_SMD:R_0402_1005Metric_Pad0.72x0.64mm_HandSolder, F.Cu at (-85.2, -112.0)
- added C241: 220nF, Resistor_SMD:R_0402_1005Metric_Pad0.72x0.64mm_HandSolder, F.Cu at (-93.4, -112.0)
- added C242: 220nF, Resistor_SMD:R_0402_1005Metric_Pad0.72x0.64mm_HandSolder, F.Cu at (-89.6, -127.0)
- added C243: 220nF, Resistor_SMD:R_0402_1005Metric_Pad0.72x0.64mm_HandSolder, F.Cu at (-90.9, -115.1)
- added C244: 220nF, Resistor_SMD:R_0402_1005Metric_Pad0.72x0.64mm_HandSolder, F.Cu at (-92.1, -100.1)
- added C245: 220nF, Resistor_SMD:R_0402_1005Metric_Pad0.72x0.64mm_HandSolder, F.Cu at (-81.7, -112.0)
- added C246: 220nF, Resistor_SMD:R_0402_1005Metric_Pad0.72x0.64mm_HandSolder, F.Cu at (-92.1, -115.1)
- added C247: 220nF, Resistor_SMD:R_0402_1005Metric_Pad0.72x0.64mm_HandSolder, F.Cu at (-90.9, -100.1)
- added C248: 220nF, Resistor_SMD:R_0402_1005Metric_Pad0.72x0.64mm_HandSolder, F.Cu at (-89.8, -112.0)
- added C249: 220nF, Resistor_SMD:R_0402_1005Metric_Pad0.72x0.64mm_HandSolder, F.Cu at (-91.0, -112.0)
- added C25: 10uF, Capacitor_SMD:C_1206_3216Metric, F.Cu at (-40.8, -133.3)
- added C250: 220nF, Resistor_SMD:R_0402_1005Metric_Pad0.72x0.64mm_HandSolder, F.Cu at (-84.0, -112.0)
- added C251: 220nF, Resistor_SMD:R_0402_1005Metric_Pad0.72x0.64mm_HandSolder, F.Cu at (-82.1, -100.1)
- added C252: 220nF, Resistor_SMD:R_0402_1005Metric_Pad0.72x0.64mm_HandSolder, F.Cu at (-81.0, -115.1)
- added C253: 220nF, Resistor_SMD:R_0402_1005Metric_Pad0.72x0.64mm_HandSolder, F.Cu at (-87.0, -127.0)
- added C254: 220nF, Resistor_SMD:R_0402_1005Metric_Pad0.72x0.64mm_HandSolder, F.Cu at (-79.3, -127.0)
- added C255: 220nF, Resistor_SMD:R_0402_1005Metric_Pad0.72x0.64mm_HandSolder, F.Cu at (-92.2, -112.0)
- added C256: 220nF, Resistor_SMD:R_0402_1005Metric_Pad0.72x0.64mm_HandSolder, F.Cu at (-89.6, -100.1)
- added C257: 220nF, Resistor_SMD:R_0402_1005Metric_Pad0.72x0.64mm_HandSolder, F.Cu at (-83.3, -100.1)
- added C258: 220nF, Resistor_SMD:R_0402_1005Metric_Pad0.72x0.64mm_HandSolder, F.Cu at (-87.0, -100.1)
- added C259: 220nF, Resistor_SMD:R_0402_1005Metric_Pad0.72x0.64mm_HandSolder, F.Cu at (-80.7, -127.0)
- added C26: 10uF, Capacitor_SMD:C_1206_3216Metric, F.Cu at (312.2, 178.8)
- added C260: 220nF, Resistor_SMD:R_0402_1005Metric_Pad0.72x0.64mm_HandSolder, F.Cu at (-84.7, -115.1)
- added C261: 220nF, Resistor_SMD:R_0402_1005Metric_Pad0.72x0.64mm_HandSolder, F.Cu at (-85.7, -127.0)
- added C262: 220nF, Resistor_SMD:R_0402_1005Metric_Pad0.72x0.64mm_HandSolder, F.Cu at (-83.5, -115.1)
- added C263: 220nF, Resistor_SMD:R_0402_1005Metric_Pad0.72x0.64mm_HandSolder, F.Cu at (-79.7, -115.1)
- added C264: 220nF, Resistor_SMD:R_0402_1005Metric_Pad0.72x0.64mm_HandSolder, F.Cu at (-89.6, -115.1)
- added C265: 220nF, Resistor_SMD:R_0402_1005Metric_Pad0.72x0.64mm_HandSolder, F.Cu at (-93.6, -127.0)
- added C266: 220nF, Resistor_SMD:R_0402_1005Metric_Pad0.72x0.64mm_HandSolder, F.Cu at (-92.3, -127.0)
- added C267: 220nF, Resistor_SMD:R_0402_1005Metric_Pad0.72x0.64mm_HandSolder, F.Cu at (-82.9, -112.0)
- added C268: 220nF, Resistor_SMD:R_0402_1005Metric_Pad0.72x0.64mm_HandSolder, F.Cu at (-80.8, -100.1)
- added C269: 220nF, Resistor_SMD:R_0402_1005Metric_Pad0.72x0.64mm_HandSolder, F.Cu at (-106.6, -132.7)
- added C27: 10uF, Capacitor_SMD:C_1206_3216Metric, F.Cu at (207.0, -53.8)
- added C270: 220nF, Resistor_SMD:R_0402_1005Metric_Pad0.72x0.64mm_HandSolder, B.Cu at (-201.8, -175.5)
- added C271: 220nF, Resistor_SMD:R_0402_1005Metric_Pad0.72x0.64mm_HandSolder, B.Cu at (-206.1, -180.2)
- added C272: 220nF, Resistor_SMD:R_0402_1005Metric_Pad0.72x0.64mm_HandSolder, B.Cu at (-197.5, -175.5)
- added C273: 220nF, Resistor_SMD:R_0402_1005Metric_Pad0.72x0.64mm_HandSolder, B.Cu at (-203.9, -177.1)
- added C274: 9.1pF, Resistor_SMD:R_0402_1005Metric_Pad0.72x0.64mm_HandSolder, F.Cu at (5.36, -175.8)
- added C275: 220nF, Resistor_SMD:R_0402_1005Metric_Pad0.72x0.64mm_HandSolder, B.Cu at (-199.7, -180.2)
- added C276: 220nF, Resistor_SMD:R_0402_1005Metric_Pad0.72x0.64mm_HandSolder, B.Cu at (-197.5, -177.1)
- added C277: 27pF, Resistor_SMD:R_0402_1005Metric_Pad0.72x0.64mm_HandSolder, F.Cu at (15.1, -167.8)
- added C278: 10uF, Resistor_SMD:R_0402_1005Metric_Pad0.72x0.64mm_HandSolder, F.Cu at (8.61, -167.8)
- added C279: 10uF, Resistor_SMD:R_0402_1005Metric_Pad0.72x0.64mm_HandSolder, F.Cu at (11.9, -175.8)
- added C28: 10uF, Capacitor_SMD:C_1206_3216Metric, F.Cu at (212.6, -53.8)
- added C280: 10uF, Resistor_SMD:R_0402_1005Metric_Pad0.72x0.64mm_HandSolder, F.Cu at (24.9, -173.8)
- added C281: 10uF, Resistor_SMD:R_0402_1005Metric_Pad0.72x0.64mm_HandSolder, F.Cu at (11.9, -169.8)
- added C282: 10uF, Resistor_SMD:R_0402_1005Metric_Pad0.72x0.64mm_HandSolder, F.Cu at (18.4, -175.8)
- added C283: 10uF, Resistor_SMD:R_0402_1005Metric_Pad0.72x0.64mm_HandSolder, F.Cu at (15.1, -173.8)
- added C284: 10nF, Resistor_SMD:R_0402_1005Metric_Pad0.72x0.64mm_HandSolder, F.Cu at (8.61, -177.7)
- added C285: 4.5pF, Resistor_SMD:R_0402_1005Metric_Pad0.72x0.64mm_HandSolder, F.Cu at (15.1, -177.7)
- added C286: 4.5pF, Resistor_SMD:R_0402_1005Metric_Pad0.72x0.64mm_HandSolder, F.Cu at (24.9, -175.8)
- added C287: 220nF, Resistor_SMD:R_0402_1005Metric_Pad0.72x0.64mm_HandSolder, B.Cu at (-201.8, -180.2)
- added C288: 10nF, Resistor_SMD:R_0402_1005Metric_Pad0.72x0.64mm_HandSolder, F.Cu at (5.36, -177.7)
- added C289: 220nF, Resistor_SMD:R_0402_1005Metric_Pad0.72x0.64mm_HandSolder, B.Cu at (-197.5, -180.2)
- added C29: 10uF, Capacitor_SMD:C_1206_3216Metric, F.Cu at (56.4, -105.2)
- added C290: 220nF, Resistor_SMD:R_0402_1005Metric_Pad0.72x0.64mm_HandSolder, B.Cu at (-199.7, -177.1)
- added C291: 3.2pF, Resistor_SMD:R_0402_1005Metric_Pad0.72x0.64mm_HandSolder, F.Cu at (21.6, -171.8)
- added C292: 220nF, Resistor_SMD:R_0402_1005Metric_Pad0.72x0.64mm_HandSolder, B.Cu at (-203.9, -180.2)
- added C293: 220nF, Resistor_SMD:R_0402_1005Metric_Pad0.72x0.64mm_HandSolder, B.Cu at (-195.4, -180.2)
- added C294: 220nF, Resistor_SMD:R_0402_1005Metric_Pad0.72x0.64mm_HandSolder, B.Cu at (-195.4, -178.6)
- added C295: 22uF, Resistor_SMD:R_0402_1005Metric_Pad0.72x0.64mm_HandSolder, B.Cu at (28.1, -111.7)
- added C296: 220nF, Resistor_SMD:R_0402_1005Metric_Pad0.72x0.64mm_HandSolder, B.Cu at (-201.8, -178.6)
- added C297: 220nF, Resistor_SMD:R_0402_1005Metric_Pad0.72x0.64mm_HandSolder, B.Cu at (-201.8, -177.1)
- added C298: 9.1pF, Resistor_SMD:R_0402_1005Metric_Pad0.72x0.64mm_HandSolder, F.Cu at (11.9, -177.7)
- added C299: 10uF, Resistor_SMD:R_0402_1005Metric_Pad0.72x0.64mm_HandSolder, F.Cu at (15.1, -169.8)
- added C3: 4.7uF, awg1000:C0402_L, F.Cu at (-125.5, -94.0)
- added C30: 10uF, Capacitor_SMD:C_1206_3216Metric, F.Cu at (27.7, 170.5)
- added C300: 10uF, Resistor_SMD:R_0402_1005Metric_Pad0.72x0.64mm_HandSolder, F.Cu at (8.61, -171.8)
- added C301: 8.2pF, Resistor_SMD:R_0402_1005Metric_Pad0.72x0.64mm_HandSolder, F.Cu at (29.4, -104.6)
- added C302: 27pF, Resistor_SMD:R_0402_1005Metric_Pad0.72x0.64mm_HandSolder, F.Cu at (15.1, -171.8)
- added C303: 10uF, Resistor_SMD:R_0402_1005Metric_Pad0.72x0.64mm_HandSolder, F.Cu at (21.6, -177.7)
- added C304: 10uF, Resistor_SMD:R_0402_1005Metric_Pad0.72x0.64mm_HandSolder, F.Cu at (18.4, -171.8)
- added C305: 27pF, Resistor_SMD:R_0402_1005Metric_Pad0.72x0.64mm_HandSolder, F.Cu at (35.3, -108.0)
- added C306: 10uF, Resistor_SMD:R_0402_1005Metric_Pad0.72x0.64mm_HandSolder, F.Cu at (18.4, -173.8)
- added C307: 10uF, Resistor_SMD:R_0402_1005Metric_Pad0.72x0.64mm_HandSolder, F.Cu at (5.36, -173.8)
- added C308: 22uF, Resistor_SMD:R_0402_1005Metric_Pad0.72x0.64mm_HandSolder, F.Cu at (33.6, -107.6)
- added C309: 10nF, Resistor_SMD:R_0402_1005Metric_Pad0.72x0.64mm_HandSolder, F.Cu at (11.9, -167.8)
- added C31: 220nF, Resistor_SMD:R_0402_1005Metric_Pad0.72x0.64mm_HandSolder, F.Cu at (37.9, 164.3)
- added C310: 220nF, Resistor_SMD:R_0402_1005Metric_Pad0.72x0.64mm_HandSolder, B.Cu at (-203.9, -178.6)
- added C311: 10nF, Resistor_SMD:R_0402_1005Metric_Pad0.72x0.64mm_HandSolder, F.Cu at (8.61, -173.8)
- added C312: 220nF, Resistor_SMD:R_0402_1005Metric_Pad0.72x0.64mm_HandSolder, B.Cu at (-195.4, -177.1)
- added C313: 0.1uF, Resistor_SMD:R_0402_1005Metric_Pad0.72x0.64mm_HandSolder, F.Cu at (18.4, -169.8)
- added C314: 10nF, Resistor_SMD:R_0402_1005Metric_Pad0.72x0.64mm_HandSolder, F.Cu at (11.9, -173.8)
- added C315: 4.5pF, Resistor_SMD:R_0402_1005Metric_Pad0.72x0.64mm_HandSolder, F.Cu at (8.61, -175.8)
- added C316: 4.5pF, Resistor_SMD:R_0402_1005Metric_Pad0.72x0.64mm_HandSolder, F.Cu at (18.4, -177.7)
- added C317: 220nF, Resistor_SMD:R_0402_1005Metric_Pad0.72x0.64mm_HandSolder, B.Cu at (-195.4, -175.5)
- added C318: 10nF, Resistor_SMD:R_0402_1005Metric_Pad0.72x0.64mm_HandSolder, F.Cu at (24.9, -177.7)
- added C319: 3.2pF, Resistor_SMD:R_0402_1005Metric_Pad0.72x0.64mm_HandSolder, F.Cu at (5.36, -169.8)
- added C32: 10uF, Capacitor_SMD:C_1206_3216Metric, F.Cu at (-124.9, -78.3)
- added C320: 22uF, Resistor_SMD:R_0402_1005Metric_Pad0.72x0.64mm_HandSolder, F.Cu at (-270.9, -273.2)
- added C321: 22uF, Resistor_SMD:R_0402_1005Metric_Pad0.72x0.64mm_HandSolder, F.Cu at (-290.9, -265.7)
- added C322: 22uF, Resistor_SMD:R_0402_1005Metric_Pad0.72x0.64mm_HandSolder, F.Cu at (-278.9, -268.2)
- added C323: 22uF, Resistor_SMD:R_0402_1005Metric_Pad0.72x0.64mm_HandSolder, F.Cu at (-286.9, -268.2)
- added C324: 22uF, Resistor_SMD:R_0402_1005Metric_Pad0.72x0.64mm_HandSolder, F.Cu at (-282.9, -265.7)
- added C325: 22uF, Resistor_SMD:R_0402_1005Metric_Pad0.72x0.64mm_HandSolder, F.Cu at (-286.9, -263.2)
- added C326: 22uF, Resistor_SMD:R_0402_1005Metric_Pad0.72x0.64mm_HandSolder, F.Cu at (-270.9, -270.7)
- added C327: 22uF, Resistor_SMD:R_0402_1005Metric_Pad0.72x0.64mm_HandSolder, F.Cu at (-278.9, -270.7)
- added C328: 22uF, Resistor_SMD:R_0402_1005Metric_Pad0.72x0.64mm_HandSolder, F.Cu at (-286.9, -265.7)
- added C329: 220nF, Resistor_SMD:R_0402_1005Metric_Pad0.72x0.64mm_HandSolder, B.Cu at (-197.5, -178.6)
- added C33: 10uF, Capacitor_SMD:C_1206_3216Metric, F.Cu at (-125.8, -92.8)
- added C330: 22uF, Resistor_SMD:R_0402_1005Metric_Pad0.72x0.64mm_HandSolder, F.Cu at (-290.9, -270.7)
- added C331: 22uF, Resistor_SMD:R_0402_1005Metric_Pad0.72x0.64mm_HandSolder, F.Cu at (-290.9, -268.2)
- added C332: 22uF, Resistor_SMD:R_0402_1005Metric_Pad0.72x0.64mm_HandSolder, F.Cu at (-274.9, -270.7)
- added C333: 22uF, Resistor_SMD:R_0402_1005Metric_Pad0.72x0.64mm_HandSolder, F.Cu at (-282.9, -268.2)
- added C334: 8.2pF, Resistor_SMD:R_0402_1005Metric_Pad0.72x0.64mm_HandSolder, F.Cu at (15.1, -175.8)
- added C335: 22uF, Resistor_SMD:R_0402_1005Metric_Pad0.72x0.64mm_HandSolder, F.Cu at (-282.9, -270.7)
- added C336: 22uF, Resistor_SMD:R_0402_1005Metric_Pad0.72x0.64mm_HandSolder, F.Cu at (-274.9, -273.2)
- added C337: 27pF, Resistor_SMD:R_0402_1005Metric_Pad0.72x0.64mm_HandSolder, F.Cu at (5.36, -171.8)
- added C338: 22uF, Resistor_SMD:R_0402_1005Metric_Pad0.72x0.64mm_HandSolder, F.Cu at (-278.9, -265.7)
- added C339: 0, Resistor_SMD:R_0402_1005Metric_Pad0.72x0.64mm_HandSolder, F.Cu at (11.9, -171.8)
- added C34: 10uF, Capacitor_SMD:C_1206_3216Metric, F.Cu at (-43.3, -133.3)
- added C340: 22uF, Resistor_SMD:R_0402_1005Metric_Pad0.72x0.64mm_HandSolder, F.Cu at (-290.9, -263.2)
- added C341: 10nF, Resistor_SMD:R_0402_1005Metric_Pad0.72x0.64mm_HandSolder, F.Cu at (5.36, -167.8)
- added C342: 22uF, Resistor_SMD:R_0402_1005Metric_Pad0.72x0.64mm_HandSolder, F.Cu at (-274.9, -265.7)
- added C343: 220nF, Resistor_SMD:R_0402_1005Metric_Pad0.72x0.64mm_HandSolder, B.Cu at (-199.7, -175.5)
- added C344: 22uF, Resistor_SMD:R_0402_1005Metric_Pad0.72x0.64mm_HandSolder, F.Cu at (-282.9, -273.2)
- added C345: 22uF, Resistor_SMD:R_0402_1005Metric_Pad0.72x0.64mm_HandSolder, F.Cu at (-282.9, -263.2)
- added C346: 10nF, Resistor_SMD:R_0402_1005Metric_Pad0.72x0.64mm_HandSolder, F.Cu at (21.6, -173.8)
- added C347: 22uF, Resistor_SMD:R_0402_1005Metric_Pad0.72x0.64mm_HandSolder, F.Cu at (-286.9, -270.7)
- added C348: 22uF, Resistor_SMD:R_0402_1005Metric_Pad0.72x0.64mm_HandSolder, F.Cu at (-278.9, -273.2)
- added C349: 220nF, Resistor_SMD:R_0402_1005Metric_Pad0.72x0.64mm_HandSolder, B.Cu at (-199.7, -178.6)
- added C35: 220nF, Resistor_SMD:R_0402_1005Metric_Pad0.72x0.64mm_HandSolder, F.Cu at (-33.1, -139.6)
- added C350: 22uF, Resistor_SMD:R_0402_1005Metric_Pad0.72x0.64mm_HandSolder, F.Cu at (-286.9, -273.2)
- added C351: 22uF, Resistor_SMD:R_0402_1005Metric_Pad0.72x0.64mm_HandSolder, F.Cu at (-290.9, -273.2)
- added C352: 220uF, awg1000:EEE-FK1H221GP, F.Cu at (76.1, 95.0)
- added C353: 0.1uF, Resistor_SMD:R_0402_1005Metric_Pad0.72x0.64mm_HandSolder, F.Cu at (32.8, -175.8)
- added C354: 0.1uF, Resistor_SMD:R_0402_1005Metric_Pad0.72x0.64mm_HandSolder, F.Cu at (36.0, -177.7)
- added C355: 0.1uF, Resistor_SMD:R_0402_1005Metric_Pad0.72x0.64mm_HandSolder, F.Cu at (32.8, -177.7)
- added C36: 10uF, Capacitor_SMD:C_1206_3216Metric, F.Cu at (101.8, 164.3)
- added C37: 10uF, Capacitor_SMD:C_1206_3216Metric, F.Cu at (231.6, -67.9)
- added C38: 220nF, Resistor_SMD:R_0402_1005Metric_Pad0.72x0.64mm_HandSolder, F.Cu at (228.4, -60.5)
- added C39: 10uF, Capacitor_SMD:C_1206_3216Metric, F.Cu at (58.8, -105.2)
- added C4: 4.7uF, awg1000:C0402_L, F.Cu at (-42.3, -141.8)
- added C40: 0.47uF, Resistor_SMD:R_0402_1005Metric_Pad0.72x0.64mm_HandSolder, F.Cu at (90.6, 159.9)
- added C41: 4.7uF, awg1000:C0402_L, F.Cu at (-5.11, -136.8)
- added C42: 10uF, Capacitor_SMD:C_1206_3216Metric, F.Cu at (-127.4, -78.3)
- added C43: 220nF, Resistor_SMD:R_0402_1005Metric_Pad0.72x0.64mm_HandSolder, F.Cu at (-127.1, -91.1)
- added C44: 220nF, Resistor_SMD:R_0402_1005Metric_Pad0.72x0.64mm_HandSolder, F.Cu at (99.7, 164.3)
- added C45: 4.7uF, awg1000:C0402_L, F.Cu at (56.8, -141.8)
- added C47: 33uF, Capacitor_SMD:CP_Elec_6.3x7.7, F.Cu at (96.9, 169.6)
- added C48: 10uF, Capacitor_SMD:C_1206_3216Metric, F.Cu at (89.4, 170.5)
- added C49: 0.47uF, Resistor_SMD:R_0402_1005Metric_Pad0.72x0.64mm_HandSolder, F.Cu at (-5.11, -139.1)
- added C49: 0.47uF, Resistor_SMD:R_0402_1005Metric_Pad0.72x0.64mm_HandSolder, F.Cu at (307.4, 175.2)
- added C49: 0.47uF, Resistor_SMD:R_0402_1005Metric_Pad0.72x0.64mm_HandSolder, F.Cu at (291.6, 188.7)
- added C50: 0.47uF, Resistor_SMD:R_0402_1005Metric_Pad0.72x0.64mm_HandSolder, F.Cu at (-154.5, -22.6)
- added C51: 0.47uF, Resistor_SMD:R_0402_1005Metric_Pad0.72x0.64mm_HandSolder, F.Cu at (-144.4, -31.8)
- added C52: 0.47uF, Resistor_SMD:R_0402_1005Metric_Pad0.72x0.64mm_HandSolder, F.Cu at (56.8, -144.0)
- added C53: 0.47uF, Resistor_SMD:R_0402_1005Metric_Pad0.72x0.64mm_HandSolder, F.Cu at (-138.8, -37.2)
- added C54: 10uF, Capacitor_SMD:C_1206_3216Metric, F.Cu at (91.9, 170.5)
- added C55: 33uF, Capacitor_SMD:CP_Elec_6.3x7.7, F.Cu at (0.90, -129.4)
- added C56: 4.7uF, awg1000:C0402_L, F.Cu at (127.4, 162.1)
- added C57: 10uF, Capacitor_SMD:C_1206_3216Metric, F.Cu at (67.7, -139.6)
- added C57: 10uF, Capacitor_SMD:C_1206_3216Metric, F.Cu at (130.4, 42.8)
- added C58: 33uF, Capacitor_SMD:CP_Elec_6.3x7.7, F.Cu at (62.7, -134.1)
- added C59: 10uF, Capacitor_SMD:C_1206_3216Metric, F.Cu at (-3.96, -128.5)
- added C6: 0.47uF, Resistor_SMD:R_0402_1005Metric_Pad0.72x0.64mm_HandSolder, F.Cu at (-128.1, -89.9)
- added C60: 10uF, Capacitor_SMD:C_1206_3216Metric, F.Cu at (5.72, -134.7)
- added C61: 220nF, Resistor_SMD:R_0402_1005Metric_Pad0.72x0.64mm_HandSolder, F.Cu at (65.7, -139.6)
- added C62: 10uF, Capacitor_SMD:C_1206_3216Metric, F.Cu at (55.3, -133.4)
- added C63: 10uF, Capacitor_SMD:C_1206_3216Metric, F.Cu at (-6.33, -128.5)
- added C64: 220nF, Resistor_SMD:R_0402_1005Metric_Pad0.72x0.64mm_HandSolder, F.Cu at (3.73, -134.7)
- added C65: 10uF, Capacitor_SMD:C_1206_3216Metric, F.Cu at (138.7, 164.2)
- added C66: 33uF, Capacitor_SMD:CP_Elec_6.3x7.7, F.Cu at (-151.3, -34.1)
- added C67: 10uF, Capacitor_SMD:C_1206_3216Metric, F.Cu at (57.8, -133.4)
- added C68: 10uF, Capacitor_SMD:C_1206_3216Metric, F.Cu at (321.1, 149.9)
- added C69: 10uF, Capacitor_SMD:C_1206_3216Metric, F.Cu at (342.0, 130.2)
- added C7: 0.47uF, Resistor_SMD:R_0402_1005Metric_Pad0.72x0.64mm_HandSolder, F.Cu at (-139.8, -93.3)
- added C70: 0.47uF, Resistor_SMD:R_0402_1005Metric_Pad0.72x0.64mm_HandSolder, F.Cu at (127.4, 159.9)
- added C71: 10uF, Capacitor_SMD:C_1206_3216Metric, F.Cu at (-143.2, -36.5)
- added C72: 10uF, Capacitor_SMD:C_1206_3216Metric, F.Cu at (-162.2, -22.3)
- added C73: 220nF, Resistor_SMD:R_0402_1005Metric_Pad0.72x0.64mm_HandSolder, F.Cu at (136.5, 164.2)
- added C74: 10uF, Capacitor_SMD:C_1206_3216Metric, F.Cu at (-167.9, -22.3)
- added C75: 220nF, Resistor_SMD:R_0402_1005Metric_Pad0.72x0.64mm_HandSolder, F.Cu at (-157.8, -20.6)
- added C76: 33uF, Capacitor_SMD:CP_Elec_6.3x7.7, F.Cu at (133.6, 169.5)
- added C77: 10uF, Capacitor_SMD:C_1206_3216Metric, F.Cu at (325.6, 141.7)
- added C78: 10uF, Capacitor_SMD:C_1206_3216Metric, F.Cu at (325.6, 138.4)
- added C79: 10uF, Capacitor_SMD:C_1206_3216Metric, F.Cu at (126.2, 170.5)
- added C80: 10uF, Capacitor_SMD:C_1206_3216Metric, F.Cu at (128.7, 170.5)
- added C81: 10uF, Capacitor_SMD:C_1206_3216Metric, F.Cu at (331.6, 141.7)
- added C82: 10uF, Capacitor_SMD:C_1206_3216Metric, F.Cu at (315.1, 153.2)
- added C83: 22uF, Capacitor_SMD:C_0603_1608Metric_Pad1.08x0.95mm_HandSolder, F.Cu at (-110.3, -74.3)
- added C84: 22uF, Capacitor_SMD:C_0603_1608Metric_Pad1.08x0.95mm_HandSolder, F.Cu at (-109.4, -96.7)
- added C85: 22uF, Capacitor_SMD:C_0603_1608Metric_Pad1.08x0.95mm_HandSolder, B.Cu at (-106.2, -85.8)
- added C86: 22uF, Capacitor_SMD:C_0603_1608Metric_Pad1.08x0.95mm_HandSolder, B.Cu at (-110.7, -88.0)
- added C87: 22uF, Capacitor_SMD:C_0603_1608Metric_Pad1.08x0.95mm_HandSolder, F.Cu at (-110.3, -75.8)
- added C88: 22uF, Capacitor_SMD:C_0603_1608Metric_Pad1.08x0.95mm_HandSolder, F.Cu at (-106.4, -96.7)
- added C89: 22uF, Capacitor_SMD:C_0603_1608Metric_Pad1.08x0.95mm_HandSolder, B.Cu at (-109.2, -88.0)
- added C9: 0.47uF, Resistor_SMD:R_0402_1005Metric_Pad0.72x0.64mm_HandSolder, F.Cu at (-138.2, -91.7)
- added C90: 22uF, Capacitor_SMD:C_0603_1608Metric_Pad1.08x0.95mm_HandSolder, B.Cu at (-109.5, -83.1)
- added C91: 22uF, Capacitor_SMD:C_0603_1608Metric_Pad1.08x0.95mm_HandSolder, F.Cu at (-107.0, -75.8)
- added C92: 22uF, Capacitor_SMD:C_0603_1608Metric_Pad1.08x0.95mm_HandSolder, F.Cu at (-107.9, -96.7)
- added C93: 22uF, Capacitor_SMD:C_0603_1608Metric_Pad1.08x0.95mm_HandSolder, B.Cu at (-107.7, -88.0)
- added C94: 22uF, Capacitor_SMD:C_0603_1608Metric_Pad1.08x0.95mm_HandSolder, B.Cu at (-108.0, -83.1)
- added C95: 4.7uF, awg1000:C0402_L, F.Cu at (147.4, 142.0)
- added C96: 22uF, Capacitor_SMD:C_0603_1608Metric_Pad1.08x0.95mm_HandSolder, F.Cu at (-107.0, -74.3)
- added C97: 22uF, Capacitor_SMD:C_0603_1608Metric_Pad1.08x0.95mm_HandSolder, F.Cu at (-110.9, -96.7)
- added C98: 22uF, Capacitor_SMD:C_0603_1608Metric_Pad1.08x0.95mm_HandSolder, B.Cu at (-111.3, -85.6)
- added C99: 22uF, Capacitor_SMD:C_0603_1608Metric_Pad1.08x0.95mm_HandSolder, B.Cu at (-111.2, -84.3)
- added D1: D_TVS, Diode_SMD:D_SMC, F.Cu at (-237.3, -160.9)
- added FB1: FerriteBead, Inductor_SMD:L_0402_1005Metric_Pad0.77x0.64mm_HandSolder, F.Cu at (-23.2, -170.3)
- added FB10: FerriteBead, Inductor_SMD:L_0402_1005Metric_Pad0.77x0.64mm_HandSolder, F.Cu at (-8.71, -164.5)
- added FB11: FerriteBead, Inductor_SMD:L_0402_1005Metric_Pad0.77x0.64mm_HandSolder, F.Cu at (-5.46, -162.5)
- added FB12: FerriteBead, Inductor_SMD:L_0402_1005Metric_Pad0.77x0.64mm_HandSolder, F.Cu at (-8.71, -162.5)
- added FB13: FerriteBead, Inductor_SMD:L_0402_1005Metric_Pad0.77x0.64mm_HandSolder, F.Cu at (-5.46, -164.5)
- added FB14: FerriteBead, Inductor_SMD:L_0402_1005Metric_Pad0.77x0.64mm_HandSolder, F.Cu at (-8.71, -172.3)
- added FB15: FerriteBead, Inductor_SMD:L_0402_1005Metric_Pad0.77x0.64mm_HandSolder, F.Cu at (-5.46, -172.3)
- added FB16: FerriteBead, Inductor_SMD:L_0402_1005Metric_Pad0.77x0.64mm_HandSolder, F.Cu at (-8.71, -170.3)
- added FB2: FerriteBead, Inductor_SMD:L_0402_1005Metric_Pad0.77x0.64mm_HandSolder, F.Cu at (-20.0, -168.3)
- added FB3: FerriteBead, Inductor_SMD:L_0402_1005Metric_Pad0.77x0.64mm_HandSolder, F.Cu at (-23.2, -168.3)
- added FB4: FerriteBead, Inductor_SMD:L_0402_1005Metric_Pad0.77x0.64mm_HandSolder, F.Cu at (-20.0, -172.3)
- added FB5: FerriteBead, Inductor_SMD:L_0402_1005Metric_Pad0.77x0.64mm_HandSolder, F.Cu at (-16.7, -172.3)
- added FB6: FerriteBead, Inductor_SMD:L_0402_1005Metric_Pad0.77x0.64mm_HandSolder, F.Cu at (-16.7, -170.3)
- added FB7: FerriteBead, Inductor_SMD:L_0402_1005Metric_Pad0.77x0.64mm_HandSolder, F.Cu at (-20.0, -170.3)
- added FB8: FerriteBead, Inductor_SMD:L_0402_1005Metric_Pad0.77x0.64mm_HandSolder, F.Cu at (-23.2, -172.3)
- added FB9: FerriteBead, Inductor_SMD:L_0402_1005Metric_Pad0.77x0.64mm_HandSolder, F.Cu at (-23.2, -162.8)
- added J11: 5-1634503-1, awg1000:5-1634503-1, F.Cu at (100.7, -66.3)
- added J12: 5-1634503-1, awg1000:5-1634503-1, F.Cu at (28.9, -66.3)
- added J13: 5-1634503-1, awg1000:5-1634503-1, F.Cu at (43.3, -66.3)
- added J14: 5-1634503-1, awg1000:5-1634503-1, F.Cu at (14.6, -66.3)
- added J15: 5-1634503-1, awg1000:5-1634503-1, F.Cu at (57.6, -66.3)
- added J16: 5-1634503-1, awg1000:5-1634503-1, F.Cu at (72.0, -66.3)
- added J17: 5-1634503-1, awg1000:5-1634503-1, F.Cu at (0.24, -66.3)
- added J18: 5-1634503-1, awg1000:5-1634503-1, F.Cu at (86.3, -66.3)
- added J3: USB1040-GF-L-B, Connector_USB:USB_A_Molex_67643_Horizontal, F.Cu at (268.4, 75.5)
- added J4: TF31-50S-0.5SH(800), awg1000:TF31-50S-0.5SH(800), F.Cu at (63.7, 75.2)
- added J5: USB_B, Connector_USB:USB_B_OST_USB-B1HSxx_Horizontal, F.Cu at (267.1, 89.9)
- added J8: HDMI_A, Connector_HDMI:HDMI_A_Contact_Technology_HDMI-19APL2_Horizontal, F.Cu at (267.1, 56.6)
- added J9: RJ45_Amphenol_RJMG1BD3B8K1ANR, Connector_RJ:RJ45_Amphenol_RJMG1BD3B8K1ANR, F.Cu at (265.1, 38.6)
- added K1: EE2-5NU, Relay_SMD:Relay_DPDT_Kemet_EE2_NU, F.Cu at (54.4, 45.2)
- added K2: EE2-5NU, Relay_SMD:Relay_DPDT_Kemet_EE2_NU, F.Cu at (78.1, 45.2)
- added K3: EE2-5NU, Relay_SMD:Relay_DPDT_Kemet_EE2_NU, F.Cu at (66.3, 45.2)
- added K4: EE2-5NU, Relay_SMD:Relay_DPDT_Kemet_EE2_NU, F.Cu at (90.0, 45.2)
- added L1: 47uH, Inductor_SMD:L_Bourns_SRR1260, F.Cu at (21.8, 161.2)
- added L10: 47uH, Inductor_SMD:L_Bourns_SRR1260, F.Cu at (120.0, 161.2)
- added L12: 1uH, awg1000:74404024010, F.Cu at (-108.9, -93.1)
- added L13: 1uH, awg1000:74404024010, F.Cu at (-111.4, -93.1)
- added L14: 1uH, awg1000:74404024010, F.Cu at (-115.8, -84.3)
- added L15: 1uH, awg1000:74404024010, F.Cu at (-108.8, -78.4)
- added L17: 30nH, Inductor_SMD:L_0402_1005Metric_Pad0.77x0.64mm_HandSolder, F.Cu at (-129.2, -35.2)
- added L18: 30nH, Inductor_SMD:L_0402_1005Metric_Pad0.77x0.64mm_HandSolder, F.Cu at (-129.2, -37.2)
- added L2: 47uH, Inductor_SMD:L_Bourns_SRR1260, F.Cu at (50.1, -114.5)
- added L20: 56nH, Inductor_SMD:L_0402_1005Metric_Pad0.77x0.64mm_HandSolder, F.Cu at (-132.4, -35.2)
- added L21: 30nH, Inductor_SMD:L_0402_1005Metric_Pad0.77x0.64mm_HandSolder, F.Cu at (-132.4, -37.2)
- added L22: 30nH, Inductor_SMD:L_0402_1005Metric_Pad0.77x0.64mm_HandSolder, F.Cu at (-125.9, -37.2)
- added L23: 56nH, Inductor_SMD:L_0402_1005Metric_Pad0.77x0.64mm_HandSolder, F.Cu at (-132.4, -33.2)
- added L3: 47uH, Inductor_SMD:L_Bourns_SRR1260, F.Cu at (-49.6, -142.8)
- added L4: 47uH, Inductor_SMD:L_Bourns_SRR1260, F.Cu at (211.2, -62.5)
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- renumbered C2 to C13, C1 to C8
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Connections:
- C13 pad 1: VCC -> VIN_ACDC
- C8 pad 1: VCC -> VIN_ACDC
- J1 pad 3: VCC -> VIN_ACDC
- J1 pad 4: VCC -> VIN_ACDC
- U1 pad 1: unconnected-(U1-Pad1) -> Net-(C10-Pad1)
- U1 pad 2: unconnected-(U1-Pad2) -> Net-(C10-Pad2)
- U1 pad 3: unconnected-(U1-Pad3) -> Net-(C2-Pad2)
- U1 pad 4: unconnected-(U1-Pad4) -> Net-(R2-Pad2)
- U1 pad 5: unconnected-(U1-Pad5) -> VIN_ACDC
- U1 pad 6: unconnected-(U1-Pad6) -> GND
- U1 pad 7: unconnected-(U1-Pad7) -> VIN_ACDC
- U1 pad 8: unconnected-(U1-Pad8) -> GND
- U1 pad 9: unconnected-(U1-Pad9) -> GND
Routing:
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- added copper zone on F.Cu, net +15V
- added copper zone on F.Cu, net +7V
- added copper zone on F.Cu, net -15V
- added copper zone on F.Cu, net -7V
- added copper zone on F.Cu, net /Power Mangement/2.5V_FPGA
- added copper zone on F.Cu, net /Power Mangement/3.6V
- added copper zone on F.Cu, net 1.2V_DAC_DVDD
- added copper zone on F.Cu, net 1.5V_DDR
- added copper zone on F.Cu, net 1.8V_SW
- added copper zone on F.Cu, net 3.3V_SW
- added copper zone on F.Cu, net 3V_VDDHIGH
- added copper zone on F.Cu, net GND
- added copper zone on F.Cu, net Net-(C10-Pad1)
- added copper zone on F.Cu, net Net-(C11-Pad1)
- added copper zone on F.Cu, net Net-(C12-Pad1)
- added copper zone on F.Cu, net Net-(C19-Pad1)
- added copper zone on F.Cu, net Net-(C40-Pad1)
- added copper zone on F.Cu, net Net-(C49-Pad1)
- added copper zone on F.Cu, net Net-(C70-Pad1)
- added copper zone on F.Cu, net Net-(L12-Pad2)
- added copper zone on F.Cu, net Net-(L13-Pad2)
- added copper zone on F.Cu, net Net-(L15-Pad1)
- added copper zone on F.Cu, net VDD_ARM_IN
- added copper zone on F.Cu, net VDD_SOC_IN
- added copper zone on F.Cu, net VIN_ACDC
Other:
- board outline added: 368.3 x 152.4 mm
- copper layers 2 -> 8
- rule pad_to_mask_clearance: 0 -> 0.127
- board text added: "0.1016 mm / 0.1016 mm"
- board text added: "0.3000 mm"
- board text added: "368.4000 mm x 152.5000 mm"
- board text added: "6"
- board text added: "7.7800 mm"
- board text added: "BOARD CHARACTERISTICS"
- board text added: "Board Thickness:"
- board text added: "Board overall dimensions:"
- board text added: "Castellated pads:"
- board text added: "Copper Finish:"
- board text added: "Copper Layer Count:"
- board text added: "Impedance Control:"
- board text added: "Min hole diameter:"
- board text added: "Min track/spacing:"
- board text added: "No"
- board text added: "None"
- board text added: "Plated Board Edge:"
