File: hardware/01-ECAD/01-KiCAD Files/AWG1000/untitled.kicad_sch (KiCad schematic)
At the start: 0 parts

Commit message: WIP.
Parts:
- added U? (x4): XC7A35T-1CSG325C, CSG324_ARTIX_XIL, symbol awg1000:XC7A35T-1CSG325C
