File: hardware/01-ECAD/01-KiCAD Files/AWG1000/MEMORY.kicad_sch (KiCad schematic)
At the start: 0 parts

Commit message: Update.
Parts:
- added C211, C212, C213, C214, C215, C216, C217, C218: 22uF, Resistor_SMD:R_0402_1005Metric_Pad0.72x0.64mm_HandSolder, symbol Device:C
- added C219, C220, C221, C222, C223, C224, C225, C226, C227, C228, C229, C230, C231, C232, C233, C234, C235, C236, C237, C238, C239, C240, C241, C242, C243, C244, C245, C246, C247, C248, C249, C250, C251, C252, C253, C254, C255, C256, C257, C258, C259, C260, C261, C262, C263, C264, C265, C266, C267, C268, C269: 220nF, Resistor_SMD:R_0402_1005Metric_Pad0.72x0.64mm_HandSolder, symbol Device:C
- added FB9: FerriteBead, Inductor_SMD:L_0402_1005Metric_Pad0.77x0.64mm_HandSolder, symbol Device:FerriteBead
- added J2: Micro_SD_Card_Det, symbol Connector:Micro_SD_Card_Det
- added R56, R57, R58, R59, R60: 240, Resistor_SMD:R_0402_1005Metric_Pad0.72x0.64mm_HandSolder, symbol Device:R_US
- added R61, R62: 49.9, Resistor_SMD:R_0402_1005Metric_Pad0.72x0.64mm_HandSolder, symbol Device:R_US
- added U17: MCIMX6S8DVM10AD, Package_BGA:BGA-625_21.0x21.0mm_Layout25x25_P0.8mm, symbol awg1000:MCIMX6S8DVM10AD
- added U22, U23, U24, U25: AS4C256M16D3LC-12BCN, Package_BGA:BGA-96_9.0x13.0mm_Layout2x3x16_P0.8mm, symbol awg1000:AS4C256M16D3LC-12BCN
- added U26: W25Q32JWSSIQ, Package_SO:SOIC-8_3.9x4.9mm_P1.27mm, symbol awg1000:W25Q32JWSSIQ
Connections:
- new net: R57.2, U23.L8 (ZQ)
- new net: R59.2, U24.L8 (ZQ)
- new net: FB9.1, J2.11 (SHIELD)
- new net: R56.2, U22.L8 (ZQ)
- new net: R58.2, U17.AE17 (ZQPAD)
- new net: R61.2, U26.3 (~{WP})
- new net: R62.2, U26.7 (~{HOLD})
- new net: R60.2, U25.L8 (ZQ)
- new net +VREF_DDR: U17.AC2 (DRAM_VREF), U22.H1 (VREFDQ), U22.M8 (VREFCA), U23.H1 (VREFDQ), U23.M8 (VREFCA), U24.H1 (VREFDQ), U24.M8 (VREFCA), U25.H1 (VREFDQ), U25.M8 (VREFCA)
- new net 1.5V_DDR: C211.1, C212.2, C213.1, C214.2, C215.1, C216.2, C217.1, C218.2, C219.1, C220.2, C221.1, C222.2, C223.1, C224.2, C225.1, C226.2, C227.1, C228.2, C229.1, C230.2, C231.1, C232.2, C233.1, C234.2, C235.1, C236.2, C237.1, C238.2, C239.1, C240.2, C241.1, C242.2, C243.1, C244.2, C245.1, C246.2, C247.1, C248.2, C249.1, C250.2, C251.1, C252.2, C253.1, C254.2, C255.1, C256.2, C257.1, C258.2, C259.1, C260.2, C261.1, C262.2, C263.1, C264.2, C265.1, C266.2, C267.1, C268.2, U17.R18 (NVCC_DRAM_1), U17.T18 (NVCC_DRAM_2), U17.U18 (NVCC_DRAM_3), U17.V10 (NVCC_DRAM_4), U17.V11 (NVCC_DRAM_5), U17.V12 (NVCC_DRAM_6), U17.V13 (NVCC_DRAM_7), U17.V14 (NVCC_DRAM_8), U17.V15 (NVCC_DRAM_9), U17.V16 (NVCC_DRAM_10), U17.V17 (NVCC_DRAM_11), U17.V18 (NVCC_DRAM_12), U17.V9 (NVCC_DRAM_13), U22.A1 (VDDQ), U22.A8 (VDDQ), U22.B2 (VDD), U22.C1 (VDDQ), U22.C9 (VDDQ), U22.D2 (VDDQ), U22.D9 (VDD), U22.E9 (VDDQ), U22.F1 (VDDQ), U22.G7 (VDD), U22.H2 (VDDQ), U22.H9 (VDDQ), U22.K2 (VDD), U22.K8 (VDD), U22.N1 (VDD), U22.N9 (VDD), U22.R1 (VDD), U22.R9 (VDD), U23.A1 (VDDQ), U23.A8 (VDDQ), U23.B2 (VDD), U23.C1 (VDDQ), U23.C9 (VDDQ), U23.D2 (VDDQ), U23.D9 (VDD), U23.E9 (VDDQ), U23.F1 (VDDQ), U23.G7 (VDD), U23.H2 (VDDQ), U23.H9 (VDDQ), U23.K2 (VDD), U23.K8 (VDD), U23.N1 (VDD), U23.N9 (VDD), U23.R1 (VDD), U23.R9 (VDD), U24.A1 (VDDQ), U24.A8 (VDDQ), U24.B2 (VDD), U24.C1 (VDDQ), U24.C9 (VDDQ), U24.D2 (VDDQ), U24.D9 (VDD), U24.E9 (VDDQ), U24.F1 (VDDQ), U24.G7 (VDD), U24.H2 (VDDQ), U24.H9 (VDDQ), U24.K2 (VDD), U24.K8 (VDD), U24.N1 (VDD), U24.N9 (VDD), U24.R1 (VDD), U24.R9 (VDD), U25.A1 (VDDQ), U25.A8 (VDDQ), U25.B2 (VDD), U25.C1 (VDDQ), U25.C9 (VDDQ), U25.D2 (VDDQ), U25.D9 (VDD), U25.E9 (VDDQ), U25.F1 (VDDQ), U25.G7 (VDD), U25.H2 (VDDQ), U25.H9 (VDDQ), U25.K2 (VDD), U25.K8 (VDD), U25.N1 (VDD), U25.N9 (VDD), U25.R1 (VDD), U25.R9 (VDD)
- new net 3.3V_SW_DELAYED: C269.1, R61.1, R62.1, U26.8 (VCC)
- new net DRAM_A0: U17.AC14 (DRAM_A0), U22.N3 (A0), U23.N3 (A0), U24.N3 (A0), U25.N3 (A0)
- new net DRAM_A1: U17.AB14 (DRAM_A1), U22.P7 (A1), U23.P7 (A1), U24.P7 (A1), U25.P7 (A1)
- new net DRAM_A10: U17.AA15 (DRAM_A10), U22.L7 (A10/AP), U23.L7 (A10/AP), U24.L7 (A10/AP), U25.L7 (A10/AP)
- new net DRAM_A11: U17.AC12 (DRAM_A11), U22.R7 (A11), U23.R7 (A11), U24.R7 (A11), U25.R7 (A11)
- new net DRAM_A12: U17.AD12 (DRAM_A12), U22.N7 (A12/~{BC}), U23.N7 (A12/~{BC}), U24.N7 (A12/~{BC}), U25.N7 (A12/~{BC})
- new net DRAM_A13: U17.AC17 (DRAM_A13), U22.T3 (A13), U23.T3 (A13), U24.T3 (A13), U25.T3 (A13)
- new net DRAM_A14: U17.AA12 (DRAM_A14), U22.T7 (A14), U23.T7 (A14), U24.T7 (A14), U25.T7 (A14)
- new net DRAM_A15: U17.Y12 (DRAM_A15)
- new net DRAM_A2: U17.AA14 (DRAM_A2), U22.P3 (A2), U23.P3 (A2), U24.P3 (A2), U25.P3 (A2)
- new net DRAM_A3: U17.Y14 (DRAM_A3), U22.N2 (A3), U23.N2 (A3), U24.N2 (A3), U25.N2 (A3)
- new net DRAM_A4: U17.W14 (DRAM_A4), U22.P8 (A4), U23.P8 (A4), U24.P8 (A4), U25.P8 (A4)
- new net DRAM_A5: U17.AE13 (DRAM_A5), U22.P2 (A5), U23.P2 (A5), U24.P2 (A5), U25.P2 (A5)
- new net DRAM_A6: U17.AC13 (DRAM_A6), U22.R8 (A6), U23.R8 (A6), U24.R8 (A6), U25.R8 (A6)
- new net DRAM_A7: U17.Y13 (DRAM_A7), U22.R2 (A7), U23.R2 (A7), U24.R2 (A7), U25.R2 (A7)
- new net DRAM_A8: U17.AB13 (DRAM_A8), U22.T8 (A8), U23.T8 (A8), U24.T8 (A8), U25.T8 (A8)
- new net DRAM_A9: U17.AE12 (DRAM_A9), U22.R3 (A9), U23.R3 (A9), U24.R3 (A9), U25.R3 (A9)
- new net DRAM_CAS_B: U17.AE16 (DRAM_CAS), U22.K3 (~{CAS}), U23.K3 (~{CAS}), U24.K3 (~{CAS}), U25.K3 (~{CAS})
- new net DRAM_CLK0_N: U17.AE15 (~{DRAM_SDCLK0})
- new net DRAM_CLK1_N: U17.AE14 (~{DRAM_SDCLK1}), U22.K7 (~{CK}), U23.K7 (~{CK}), U24.K7 (~{CK}), U25.K7 (~{CK})
- new net DRAM_CLK1_P: U17.AD14 (DRAM_SDCLK_1), U22.J7 (CK), U23.J7 (CK), U24.J7 (CK), U25.J7 (CK)
- new net DRAM_CLKO_P: U17.AD15 (DRAM_SDCLK_0)
- new net DRAM_CS0_B: U17.Y16 (DRAM_CS0), U22.L2 (~{CS}), U23.L2 (~{CS}), U24.L2 (~{CS}), U25.L2 (~{CS})
- new net DRAM_D0: U17.AD2 (DRAM_D0), U22.E3 (DQ0)
- new net DRAM_D1: U17.AE2 (DRAM_D1), U22.H3 (DQ4)
- new net DRAM_D10: U17.AA6 (DRAM_D10), U22.B8 (DQ14)
- new net DRAM_D11: U17.AE7 (DRAM_D11), U22.C8 (DQ10)
- new net DRAM_D12: U17.AB5 (DRAM_D12), U22.C2 (DQ11)
- new net DRAM_D13: U17.AC5 (DRAM_D13), U22.A3 (DQ15)
- new net DRAM_D14: U17.AB6 (DRAM_D14), U22.A2 (DQ13)
- new net DRAM_D15: U17.AC7 (DRAM_D15), U22.A7 (DQ12)
- new net DRAM_D16: U17.AB7 (DRAM_D16), U23.E3 (DQ0)
- new net DRAM_D17: U17.AA8 (DRAM_D17), U23.F7 (DQ1)
- new net DRAM_D18: U17.AB9 (DRAM_D18), U23.H3 (DQ4)
- new net DRAM_D19: U17.Y9 (DRAM_D19), U23.H8 (DQ5)
- new net DRAM_D2: U17.AC4 (DRAM_D2), U22.H7 (DQ7)
- new net DRAM_D20: U17.Y7 (DRAM_D20), U23.G2 (DQ6)
- new net DRAM_D21: U17.Y8 (DRAM_D21), U23.F8 (DQ3)
- new net DRAM_D22: U17.AC8 (DRAM_D22), U23.F2 (DQ2)
- new net DRAM_D23: U17.AA9 (DRAM_D23), U23.H7 (DQ7)
- new net DRAM_D24: U17.AE9 (DRAM_D24), U23.D7 (DQ8)
- new net DRAM_D25: U17.Y10 (DRAM_D25), U23.A2 (DQ13)
- new net DRAM_D26: U17.AE11 (DRAM_D26), U23.B8 (DQ14)
- new net DRAM_D27: U17.AB11 (DRAM_D27), U23.C2 (DQ11)
- new net DRAM_D28: U17.AC9 (DRAM_D28), U23.C3 (DQ9)
- new net DRAM_D29: U17.AD9 (DRAM_D29), U23.A7 (DQ12)
- new net DRAM_D3: U17.AA5 (DRAM_D3), U22.F8 (DQ3)
- new net DRAM_D30: U17.AD11 (DRAM_D30), U23.C8 (DQ10)
- new net DRAM_D31: U17.AC11 (DRAM_D31), U23.A3 (DQ15)
- new net DRAM_D32: U17.AA17 (DRAM_D32), U24.E3 (DQ0)
- new net DRAM_D33: U17.AA18 (DRAM_D33), U24.H3 (DQ4)
- new net DRAM_D34: U17.AC18 (DRAM_D34), U24.F7 (DQ1)
- new net DRAM_D35: U17.AE19 (DRAM_D35), U24.H7 (DQ7)
- new net DRAM_D36: U17.Y17 (DRAM_D36), U24.G2 (DQ6)
- new net DRAM_D37: U17.Y18 (DRAM_D37), U24.F2 (DQ2)
- new net DRAM_D38: U17.AB19 (DRAM_D38), U24.F8 (DQ3)
- new net DRAM_D39: U17.AC19 (DRAM_D39), U24.H8 (DQ5)
- new net DRAM_D4: U17.AC1 (DRAM_D4), U22.F2 (DQ2)
- new net DRAM_D40: U17.Y19 (DRAM_D40), U24.D7 (DQ8)
- new net DRAM_D41: U17.AB20 (DRAM_D41), U24.C2 (DQ11)
- new net DRAM_D42: U17.AB21 (DRAM_D42), U24.A7 (DQ12)
- new net DRAM_D43: U17.AD21 (DRAM_D43), U24.C8 (DQ10)
- new net DRAM_D44: U17.Y20 (DRAM_D44), U24.A2 (DQ13)
- new net DRAM_D45: U17.AA20 (DRAM_D45), U24.A3 (DQ15)
- new net DRAM_D46: U17.AE21 (DRAM_D46), U24.B8 (DQ14)
- new net DRAM_D47: U17.AC21 (DRAM_D47), U24.C3 (DQ9)
- new net DRAM_D48: U17.AC22 (DRAM_D48), U25.E3 (DQ0)
- new net DRAM_D49: U17.AE22 (DRAM_D49), U25.G2 (DQ6)
- new net DRAM_D5: U17.AD1 (DRAM_D5), U22.G2 (DQ6)
- new net DRAM_D50: U17.AE24 (DRAM_D50), U25.H7 (DQ7)
- new net DRAM_D51: U17.AC24 (DRAM_D51), U25.F8 (DQ3)
- new net DRAM_D52: U17.AB22 (DRAM_D52), U25.F2 (DQ2)
- new net DRAM_D53: U17.AC23 (DRAM_D53), U25.H3 (DQ4)
- new net DRAM_D54: U17.AD25 (DRAM_D54), U25.F7 (DQ1)
- new net DRAM_D55: U17.AC25 (DRAM_D55), U25.H8 (DQ5)
- new net DRAM_D56: U17.AD23 (DRAM_SDQS6), U25.D7 (DQ8)
- new net DRAM_D57: U17.AA21 (DRAM_D57), U25.C2 (DQ11)
- new net DRAM_D58: U17.Y25 (DRAM_D58), U25.B8 (DQ14)
- new net DRAM_D59: U17.Y22 (DRAM_D59), U25.A2 (DQ13)
- new net DRAM_D6: U17.AB4 (DRAM_D6), U22.F7 (DQ1)
- new net DRAM_D60: U17.AB23 (DRAM_D60), U25.C3 (DQ9)
- new net DRAM_D61: U17.AA23 (DRAM_D61), U25.A3 (DQ15)
- new net DRAM_D62: U17.Y23 (DRAM_D62), U25.A7 (DQ12)
- new net DRAM_D63: U17.W25 (DRAM_D63), U25.C8 (DQ10)
- new net DRAM_D7: U17.AE4 (DRAM_D7), U22.H8 (DQ5)
- new net DRAM_D8: U17.AD5 (DRAM_D8), U22.D7 (DQ8)
- new net DRAM_D9: U17.AE5 (DRAM_D9), U22.C3 (DQ9)
- new net DRAM_DQM0: U17.AC3 (DRAM_DQM0), U22.E7 (LDM)
- new net DRAM_DQM1: U17.AC6 (DRAM_DQM1), U22.D3 (UDM)
- new net DRAM_DQM2: U17.AB8 (DRAM_DQM2), U23.E7 (LDM)
- new net DRAM_DQM3: U17.AE10 (DRAM_DQM3), U23.D3 (UDM)
- new net DRAM_DQM4: U17.AB18 (DRAM_DQM4), U24.E7 (LDM)
- new net DRAM_DQM5: U17.AC20 (DRAM_DQM5), U24.D3 (UDM)
- new net DRAM_DQM6: U17.AB25 (DRAM_D56), U25.E7 (LDM)
- new net DRAM_DQM7: U17.Y21 (DRAM_DQM7), U25.D3 (UDM)
- new net DRAM_DQS0_N: U17.AD3 (~{DRAM_SDQS0}), U22.G3 (~{LDQS})
- new net DRAM_DQS0_P: U17.AE3 (DRAM_SDQS0), U22.F3 (LDQS)
- new net DRAM_DQS1_N: U17.AE6 (~{DRAM_SDQS1}), U22.B7 (~{UDQS})
- new net DRAM_DQS1_P: U17.AD6 (DRAM_SDQS1), U22.C7 (UDQS)
- new net DRAM_DQS2_P: U17.AD8 (DRAM_SDQS2), U17.AE8 (~{DRAM_SDQS2}), U23.F3 (LDQS), U23.G3 (~{LDQS})
- new net DRAM_DQS3_N: U17.AB10 (~{DRAM_SDQS3}), U23.B7 (~{UDQS})
- new net DRAM_DQS3_P: U17.AC10 (DRAM_SDQS3), U23.C7 (UDQS)
- new net DRAM_DQS4_N: U17.AE18 (~{DRAM_SDQS4}), U24.G3 (~{LDQS})
- new net DRAM_DQS4_P: U17.AD18 (DRAM_SDQS4), U24.F3 (LDQS)
- new net DRAM_DQS5_N: U17.AE20 (~{DRAM_SDQS5}), U24.B7 (~{UDQS})
- new net DRAM_DQS5_P: U17.AD20 (DRAM_SDQS5), U24.C7 (UDQS)
- new net DRAM_DQS6_N: U17.AD24 (DRAM_DQM6), U25.G3 (~{LDQS})
- new net DRAM_DQS6_P: U17.AE23 (~{DRAM_SDQS6}), U25.F3 (LDQS)
- new net DRAM_DQS7_N: U17.AA24 (~{DRAM_SDQS7}), U25.B7 (~{UDQS})
- new net DRAM_DQS7_P: U17.AA25 (DRAM_SDQS7), U25.C7 (UDQS)
- new net DRAM_RAS_B: U17.AB15 (DRAM_RAS), U22.J3 (~{RAS}), U23.J3 (~{RAS}), U24.J3 (~{RAS}), U25.J3 (~{RAS})
- new net DRAM_RESET_B: U17.Y6 (DRAM_RESET), U22.T2 (~{RESET}), U23.T2 (~{RESET}), U24.T2 (~{RESET}), U25.T2 (~{RESET})
- new net DRAM_SDBA0: U17.AC15 (DRAM_SDBA0), U22.M2 (BA0), U23.M2 (BA0), U24.M2 (BA0), U25.M2 (BA0)
- new net DRAM_SDBA1: U17.Y15 (DRAM_SDBA1), U22.N8 (BA1), U23.N8 (BA1), U24.N8 (BA1), U25.N8 (BA1)
- new net DRAM_SDBA2: U17.AB12 (DRAM_SDBA2), U22.M3 (BA2), U23.M3 (BA2), U24.M3 (BA2), U25.M3 (BA2)
- new net DRAM_SDCKE0: U17.Y11 (DRAM_SDCKE0), U22.K9 (CKE), U23.K9 (CKE), U24.K9 (CKE), U25.K9 (CKE)
- new net DRAM_SDODT0: U17.AC16 (DRAM_SDODT0), U22.K1 (ODT), U23.K1 (ODT), U24.K1 (ODT), U25.K1 (ODT)
- new net DRAM_WE_B: U17.AB16 (DRAM_SDWE), U22.L3 (~{WE}), U23.L3 (~{WE}), U24.L3 (~{WE}), U25.L3 (~{WE})
- new net GND: C211.2, C212.1, C213.2, C214.1, C215.2, C216.1, C217.2, C218.1, C219.2, C220.1, C221.2, C222.1, C223.2, C224.1, C225.2, C226.1, C227.2, C228.1, C229.2, C230.1, C231.2, C232.1, C233.2, C234.1, C235.2, C236.1, C237.2, C238.1, C239.2, C240.1, C241.2, C242.1, C243.2, C244.1, C245.2, C246.1, C247.2, C248.1, C249.2, C250.1, C251.2, C252.1, C253.2, C254.1, C255.2, C256.1, C257.2, C258.1, C259.2, C260.1, C261.2, C262.1, C263.2, C264.1, C265.2, C266.1, C267.2, C268.1, C269.2, FB9.2, J2.6 (VSS), R56.1, R57.1, R58.1, R59.1, R60.1, U22.A9 (VSS), U22.B1 (VSSQ), U22.B3 (VSS), U22.B9 (VSSQ), U22.D1 (VSSQ), U22.D8 (VSSQ), U22.E1 (VSS), U22.E2 (VSSQ), U22.E8 (VSSQ), U22.F9 (VSSQ), U22.G1 (VSSQ), U22.G8 (VSS), U22.G9 (VSSQ), U22.J2 (VSS), U22.J8 (VSS), U22.M1 (VSS), U22.M9 (VSS), U22.P1 (VSS), U22.P9 (VSS), U22.T1 (VSS), U22.T9 (VSS), U23.A9 (VSS), U23.B1 (VSSQ), U23.B3 (VSS), U23.B9 (VSSQ), U23.D1 (VSSQ), U23.D8 (VSSQ), U23.E1 (VSS), U23.E2 (VSSQ), U23.E8 (VSSQ), U23.F9 (VSSQ), U23.G1 (VSSQ), U23.G8 (VSS), U23.G9 (VSSQ), U23.J2 (VSS), U23.J8 (VSS), U23.M1 (VSS), U23.M9 (VSS), U23.P1 (VSS), U23.P9 (VSS), U23.T1 (VSS), U23.T9 (VSS), U24.A9 (VSS), U24.B1 (VSSQ), U24.B3 (VSS), U24.B9 (VSSQ), U24.D1 (VSSQ), U24.D8 (VSSQ), U24.E1 (VSS), U24.E2 (VSSQ), U24.E8 (VSSQ), U24.F9 (VSSQ), U24.G1 (VSSQ), U24.G8 (VSS), U24.G9 (VSSQ), U24.J2 (VSS), U24.J8 (VSS), U24.M1 (VSS), U24.M9 (VSS), U24.P1 (VSS), U24.P9 (VSS), U24.T1 (VSS), U24.T9 (VSS), U25.A9 (VSS), U25.B1 (VSSQ), U25.B3 (VSS), U25.B9 (VSSQ), U25.D1 (VSSQ), U25.D8 (VSSQ), U25.E1 (VSS), U25.E2 (VSSQ), U25.E8 (VSSQ), U25.F9 (VSSQ), U25.G1 (VSSQ), U25.G8 (VSS), U25.G9 (VSSQ), U25.J2 (VSS), U25.J8 (VSS), U25.M1 (VSS), U25.M9 (VSS), U25.P1 (VSS), U25.P9 (VSS), U25.T1 (VSS), U25.T9 (VSS), U26.4 (GND)
- new net NORF_CLK: U26.6 (CLK)
- new net NORF_CS: U26.1 (~{CE})
- new net NORF_MISO: U26.2 (DO)
- new net NORF_MOSI: U26.5 (DI)
- new net SD_CLK: J2.5 (CLK)
- new net SD_CMD: J2.3 (CMD)
- new net SD_D0: J2.7 (DAT0)
- new net SD_D1: J2.8 (DAT1)
- new net SD_D2: J2.1 (DAT2)
- new net SD_D3: J2.2 (DAT3/CD)
- no-connect marks 0 -> 3
Other:
- note added: "EEPROM"
- note added: "MPU DDR3L RAM 2 GIGABYTES"
- note added: "MPU NOR FLASH"
- note added: "SD CARD"
