File: hardware/01-ECAD/01-KiCAD Files/AWG1000/MEMORY.kicad_sch (KiCad schematic)
At the start: 74 parts, among them J2 Micro_SD_Card_Det, U17 MCIMX6S8DVM10AD, U22 AS4C256M16D3LC-12BCN, U23 AS4C256M16D3LC-12BCN, U24 AS4C256M16D3LC-12BCN, U25 AS4C256M16D3LC-12BCN, U26 W25Q32JWSSIQ

Commit message: Update.
Parts:
- removed C218: 22uF, Resistor_SMD:R_0402_1005Metric_Pad0.72x0.64mm_HandSolder, symbol Device:C
- removed C260, C261, C262, C263, C265, C266: 220nF, Resistor_SMD:R_0402_1005Metric_Pad0.72x0.64mm_HandSolder, symbol Device:C
- removed FB9: FerriteBead, Inductor_SMD:L_0402_1005Metric_Pad0.77x0.64mm_HandSolder, symbol Device:FerriteBead
- removed J2: Micro_SD_Card_Det, symbol Connector:Micro_SD_Card_Det
- added C211, C212, C213, C214, C215, C222, C224, C225, C226, C237, C238, C366, C367, C368, C369, C370, C371, C372, C373, C374, C375, C376, C378: 220nF, awg1000:C0201_L, symbol Device:C
- added R136, R137, R138, R139, R140, R141, R142, R143, R144, R145, R146, R147, R148, R149, R150, R151, R152, R153, R155, R156, R157, R158, R159: 49.9, Resistor_SMD:R_0402_1005Metric_Pad0.72x0.64mm_HandSolder, symbol Device:R_US
- C216: value 22uF -> 220nF; footprint Resistor_SMD:R_0402_1005Metric_Pad0.72x0.64mm_HandSolder -> awg1000:C0201_L; Part Number (none) -> UMK107B7224KA-TR; VOLTAGE 10V -> 16V
- C227: renamed from C219; footprint Resistor_SMD:R_0402_1005Metric_Pad0.72x0.64mm_HandSolder -> awg1000:C0201_L
- C228: renamed from C220; footprint Resistor_SMD:R_0402_1005Metric_Pad0.72x0.64mm_HandSolder -> awg1000:C0201_L
- C229: renamed from C221; footprint Resistor_SMD:R_0402_1005Metric_Pad0.72x0.64mm_HandSolder -> awg1000:C0201_L
- C230: renamed from C222; footprint Resistor_SMD:R_0402_1005Metric_Pad0.72x0.64mm_HandSolder -> awg1000:C0201_L
- C231: renamed from C223; footprint Resistor_SMD:R_0402_1005Metric_Pad0.72x0.64mm_HandSolder -> awg1000:C0201_L
- C232: renamed from C224; footprint Resistor_SMD:R_0402_1005Metric_Pad0.72x0.64mm_HandSolder -> awg1000:C0201_L
- C233: renamed from C225; footprint Resistor_SMD:R_0402_1005Metric_Pad0.72x0.64mm_HandSolder -> awg1000:C0201_L
- C234: renamed from C226; footprint Resistor_SMD:R_0402_1005Metric_Pad0.72x0.64mm_HandSolder -> awg1000:C0201_L
- C235: renamed from C227; footprint Resistor_SMD:R_0402_1005Metric_Pad0.72x0.64mm_HandSolder -> awg1000:C0201_L
- C236: renamed from C228; footprint Resistor_SMD:R_0402_1005Metric_Pad0.72x0.64mm_HandSolder -> awg1000:C0201_L
- C239: renamed from C229; footprint Resistor_SMD:R_0402_1005Metric_Pad0.72x0.64mm_HandSolder -> awg1000:C0201_L
- C240: renamed from C230; footprint Resistor_SMD:R_0402_1005Metric_Pad0.72x0.64mm_HandSolder -> awg1000:C0201_L
- C241: renamed from C231; footprint Resistor_SMD:R_0402_1005Metric_Pad0.72x0.64mm_HandSolder -> awg1000:C0201_L
- C242: renamed from C232; footprint Resistor_SMD:R_0402_1005Metric_Pad0.72x0.64mm_HandSolder -> awg1000:C0201_L
- C243: renamed from C233; footprint Resistor_SMD:R_0402_1005Metric_Pad0.72x0.64mm_HandSolder -> awg1000:C0201_L
- C244: renamed from C234; footprint Resistor_SMD:R_0402_1005Metric_Pad0.72x0.64mm_HandSolder -> awg1000:C0201_L
- C245: renamed from C235; footprint Resistor_SMD:R_0402_1005Metric_Pad0.72x0.64mm_HandSolder -> awg1000:C0201_L
- C246: renamed from C236; footprint Resistor_SMD:R_0402_1005Metric_Pad0.72x0.64mm_HandSolder -> awg1000:C0201_L
- C247: renamed from C237; footprint Resistor_SMD:R_0402_1005Metric_Pad0.72x0.64mm_HandSolder -> awg1000:C0201_L
- C248: renamed from C238; footprint Resistor_SMD:R_0402_1005Metric_Pad0.72x0.64mm_HandSolder -> awg1000:C0201_L
- C249: renamed from C239; footprint Resistor_SMD:R_0402_1005Metric_Pad0.72x0.64mm_HandSolder -> awg1000:C0201_L
- C250: renamed from C240; footprint Resistor_SMD:R_0402_1005Metric_Pad0.72x0.64mm_HandSolder -> awg1000:C0201_L
- C251: renamed from C241; footprint Resistor_SMD:R_0402_1005Metric_Pad0.72x0.64mm_HandSolder -> awg1000:C0201_L
- C252: renamed from C242; footprint Resistor_SMD:R_0402_1005Metric_Pad0.72x0.64mm_HandSolder -> awg1000:C0201_L
- C253: renamed from C243; footprint Resistor_SMD:R_0402_1005Metric_Pad0.72x0.64mm_HandSolder -> awg1000:C0201_L
- C254: renamed from C244; footprint Resistor_SMD:R_0402_1005Metric_Pad0.72x0.64mm_HandSolder -> awg1000:C0201_L
- C255: renamed from C245; footprint Resistor_SMD:R_0402_1005Metric_Pad0.72x0.64mm_HandSolder -> awg1000:C0201_L
- C256: renamed from C246; footprint Resistor_SMD:R_0402_1005Metric_Pad0.72x0.64mm_HandSolder -> awg1000:C0201_L
- C257: renamed from C247; footprint Resistor_SMD:R_0402_1005Metric_Pad0.72x0.64mm_HandSolder -> awg1000:C0201_L
- C258: renamed from C248; footprint Resistor_SMD:R_0402_1005Metric_Pad0.72x0.64mm_HandSolder -> awg1000:C0201_L
- C259: renamed from C249; footprint Resistor_SMD:R_0402_1005Metric_Pad0.72x0.64mm_HandSolder -> awg1000:C0201_L
- C260: renamed from C250; footprint Resistor_SMD:R_0402_1005Metric_Pad0.72x0.64mm_HandSolder -> awg1000:C0201_L
- C261: renamed from C251; footprint Resistor_SMD:R_0402_1005Metric_Pad0.72x0.64mm_HandSolder -> awg1000:C0201_L
- C262: renamed from C252; footprint Resistor_SMD:R_0402_1005Metric_Pad0.72x0.64mm_HandSolder -> awg1000:C0201_L
- C263: renamed from C253; footprint Resistor_SMD:R_0402_1005Metric_Pad0.72x0.64mm_HandSolder -> awg1000:C0201_L
- C264: renamed from C254; footprint Resistor_SMD:R_0402_1005Metric_Pad0.72x0.64mm_HandSolder -> awg1000:C0201_L
- C265: renamed from C255; footprint Resistor_SMD:R_0402_1005Metric_Pad0.72x0.64mm_HandSolder -> awg1000:C0201_L
- C266: renamed from C256; footprint Resistor_SMD:R_0402_1005Metric_Pad0.72x0.64mm_HandSolder -> awg1000:C0201_L
- C267: renamed from C257; footprint Resistor_SMD:R_0402_1005Metric_Pad0.72x0.64mm_HandSolder -> awg1000:C0201_L
- C268: renamed from C258; footprint Resistor_SMD:R_0402_1005Metric_Pad0.72x0.64mm_HandSolder -> awg1000:C0201_L
- C269: renamed from C259; footprint Resistor_SMD:R_0402_1005Metric_Pad0.72x0.64mm_HandSolder -> awg1000:C0201_L
- C274: renamed from C264; footprint Resistor_SMD:R_0402_1005Metric_Pad0.72x0.64mm_HandSolder -> awg1000:C0201_L
- C277: renamed from C267; footprint Resistor_SMD:R_0402_1005Metric_Pad0.72x0.64mm_HandSolder -> awg1000:C0201_L
- C278: renamed from C268; footprint Resistor_SMD:R_0402_1005Metric_Pad0.72x0.64mm_HandSolder -> awg1000:C0201_L
- C279: renamed from C269; footprint Resistor_SMD:R_0402_1005Metric_Pad0.72x0.64mm_HandSolder -> awg1000:C0201_L
- R56, R57, R58, R59, R60: footprint Resistor_SMD:R_0402_1005Metric_Pad0.72x0.64mm_HandSolder -> awg1000:C0201_L
- U17: footprint Package_BGA:BGA-625_21.0x21.0mm_Layout25x25_P0.8mm -> awg1000:BGA-625_21.0x21.0mm_Layout25x25_P0.8mm
- U22, U23, U24, U25: footprint Package_BGA:BGA-96_9.0x13.0mm_Layout2x3x16_P0.8mm -> awg1000:BGA-96_9.0x13.0mm_Layout2x3x16_P0.8mm
- renumbered C211 to C217, C212 to C218, C213 to C219, C214 to C220, C215 to C221, C217 to C223
Connections:
- net +VREF_DDR: now also C366.1, C367.2, C368.1, C369.2, C370.1, C371.2, C372.1, C373.2, R136.2, R137.2, R138.2, R139.2, R140.2, R141.2, R142.2, R143.2, R144.2, R145.2, R146.2, R147.2, R148.2, R149.2, R150.2, R151.2, R152.2, R153.2, R155.2, R156.2, R157.2, R158.2, R159.2
- net 1.5V_DDR: now also C211.1, C212.2, C213.1, C214.2, C215.1, C222.1, C224.2, C225.1, C226.2, C237.1, C238.2, C374.1, C375.2, C376.1, C378.1
- net DRAM_A1: now also R140.1
- net DRAM_A10: now also R149.1
- net DRAM_A11: now also R150.1
- net DRAM_A12: now also R151.1
- net DRAM_A13: now also R152.1
- net DRAM_A14: now also R153.1
- net DRAM_A2: now also R141.1
- net DRAM_A3: now also R142.1
- net DRAM_A4: now also R143.1
- net DRAM_A5: now also R144.1
- net DRAM_A6: now also R145.1
- net DRAM_A7: now also R146.1
- net DRAM_A8: now also R147.1
- net DRAM_A9: now also R148.1
- net DRAM_CAS_B: now also R157.1
- net DRAM_CLK0_N: now also U22.K7 (~{CK}), U23.K7 (~{CK}), U24.K7 (~{CK}), U25.K7 (~{CK})
- net DRAM_CLK1_N: no longer U22.K7 (~{CK}), U23.K7 (~{CK}), U24.K7 (~{CK}), U25.K7 (~{CK})
- net DRAM_CLK1_P: no longer U22.J7 (CK), U23.J7 (CK), U24.J7 (CK), U25.J7 (CK)
- net DRAM_CS0_B: now also R139.1
- net DRAM_RAS_B: now also R156.1
- net DRAM_RESET_B: now also R155.1
- net DRAM_SDBA0: now also R136.1
- net DRAM_SDBA1: now also R137.1
- net DRAM_SDBA2: now also R138.1
- net DRAM_SDODT0: now also R159.1
- net DRAM_WE_B: now also R158.1
- net GND: now also C211.2, C212.1, C213.2, C214.1, C215.2, C222.2, C224.1, C225.2, C226.1, C237.2, C238.1, C366.2, C367.1, C368.2, C369.1, C370.2, C371.1, C372.2, C373.1, C374.2, C375.1, C376.2, C378.2
- net DRAM_CLKO_P renamed DRAM_CLK0_P
- net DRAM_CLK0_P: now also U22.J7 (CK), U23.J7 (CK), U24.J7 (CK), U25.J7 (CK)
Other:
- note removed: "SD CARD"
- moved on the sheet: U17L

Commit message: Update.
Parts:
- removed C269: 220nF, awg1000:C0201_L, symbol Device:C
- removed unit 12 of U17
- added C354: 22uF, Resistor_SMD:R_0402_1005Metric_Pad0.72x0.64mm_HandSolder, symbol awg1000:CAP_UNPOL
- added C357, C358: 220nF, awg1000:C0201_L, symbol awg1000:CAP_UNPOL
- added U12: MT29F32G08CBACAWP-Z:C TR, Package_SO:TSOP-I-48_18.4x12mm_P0.5mm, symbol awg1000:MT29F32G08CBACAWP-Z{colon}C TR
- added U40, U41: AS4C256M16D3LC-12BCN, awg1000:BGA-96_9.0x13.0mm_Layout2x3x16_P0.8mm, symbol awg1000:AS4C256M16D3LC-12BCN
- C211, C212, C213, C214, C215, C216, C222, C224, C225, C226, C227, C228, C229, C230, C231, C232, C233, C234, C235, C236, C237, C238, C239, C240, C241, C242, C243, C244, C245, C246, C247, C248, C249, C250, C251, C252, C253, C254, C255, C256, C257, C258, C259, C260, C261, C262, C263, C264, C265, C266, C267, C268, C274, C277, C278, C279, C366, C367, C368, C369, C370, C371, C372, C373, C374, C375, C376, C378: symbol Device:C -> awg1000:CAP_UNPOL; Part Number UMK107B7224KA-TR -> (none)
- C217, C218, C219, C220, C221, C223: symbol Device:C -> awg1000:CAP_UNPOL
- R136, R137, R138, R139, R140, R141, R142, R143, R144, R145, R146, R147, R148, R149, R150, R151, R152, R153, R155, R156, R157, R158, R159, R56, R57, R58, R59, R60, R61, R62: symbol Device:R_US -> awg1000:R
Connections:
- net 1.5V_DDR: now also C225.2, C237.2, C238.1, C378.2; no longer C225.1, C237.1, C238.2, C378.1
- net 3.3V_SW_DELAYED: now also R61.2, C354.1, C357.1, C358.1, U12.12 (VCC1), U12.34 (DNU/VCCQ), U12.37 (VCC), U12.39 (DNU/VCCQ); no longer R61.1
- net DRAM_D56: now also U17.AB25 (DRAM_D56); no longer U17.AD23 (DRAM_SDQS6)
- net DRAM_DQM6: now also U17.AD24 (DRAM_DQM6); no longer U17.AB25 (DRAM_D56)
- net DRAM_DQS6_N: now also U17.AE23 (~{DRAM_SDQS6}); no longer U17.AD24 (DRAM_DQM6)
- net DRAM_DQS6_P: now also U17.AD23 (DRAM_SDQS6); no longer U17.AE23 (~{DRAM_SDQS6})
- net GND: now also C225.1, C237.1, C238.2, C378.1, C354.2, C357.2, C358.2, U12.13 (VSS1), U12.25 (DNU/VSSQ), U12.36 (VSS), U12.48 (DNU/VSSQ); no longer C225.2, C237.2, C238.1, C378.2
- net at U26.3 (~{WP}): now also R61.1; no longer R61.2
- net DRAM_CLK1_N: no longer names the net of U17.AE14 (~{DRAM_SDCLK1})
- net DRAM_CLK1_P: no longer names the net of U17.AD14 (DRAM_SDCLK_1)
- new net: U41.A1 (VDDQ), U41.A8 (VDDQ), U41.C1 (VDDQ), U41.C9 (VDDQ), U41.D2 (VDDQ), U41.E9 (VDDQ), U41.F1 (VDDQ), U41.H2 (VDDQ), U41.H9 (VDDQ)
- new net: U41.A9 (VSS), U41.B3 (VSS), U41.E1 (VSS), U41.G8 (VSS), U41.J2 (VSS), U41.J8 (VSS), U41.M1 (VSS), U41.M9 (VSS), U41.P1 (VSS), U41.P9 (VSS), U41.T1 (VSS), U41.T9 (VSS)
- new net: U41.B1 (VSSQ), U41.B9 (VSSQ), U41.D1 (VSSQ), U41.D8 (VSSQ), U41.E2 (VSSQ), U41.E8 (VSSQ), U41.F9 (VSSQ), U41.G1 (VSSQ), U41.G9 (VSSQ)
- new net: U41.B2 (VDD), U41.D9 (VDD), U41.G7 (VDD), U41.K2 (VDD), U41.K8 (VDD), U41.N1 (VDD), U41.N9 (VDD), U41.R1 (VDD), U41.R9 (VDD)
- new net: U40.A1 (VDDQ), U40.A8 (VDDQ), U40.C1 (VDDQ), U40.C9 (VDDQ), U40.D2 (VDDQ), U40.E9 (VDDQ), U40.F1 (VDDQ), U40.H2 (VDDQ), U40.H9 (VDDQ)
- new net: U40.A9 (VSS), U40.B3 (VSS), U40.E1 (VSS), U40.G8 (VSS), U40.J2 (VSS), U40.J8 (VSS), U40.M1 (VSS), U40.M9 (VSS), U40.P1 (VSS), U40.P9 (VSS), U40.T1 (VSS), U40.T9 (VSS)
- new net: U40.B1 (VSSQ), U40.B9 (VSSQ), U40.D1 (VSSQ), U40.D8 (VSSQ), U40.E2 (VSSQ), U40.E8 (VSSQ), U40.F9 (VSSQ), U40.G1 (VSSQ), U40.G9 (VSSQ)
- new net: U40.B2 (VDD), U40.D9 (VDD), U40.G7 (VDD), U40.K2 (VDD), U40.K8 (VDD), U40.N1 (VDD), U40.N9 (VDD), U40.R1 (VDD), U40.R9 (VDD)
- new net NANDF_ALE: U12.17 (ALE)
- new net NANDF_CLE: U12.16 (CLE)
- new net NANDF_CS0: U12.9 (CE#)
- new net NANDF_CS1: U12.10 (CE2#)
- new net NANDF_D0: U12.29 (DQ0)
- new net NANDF_D1: U12.30 (DQ1)
- new net NANDF_D2: U12.31 (DQ2)
- new net NANDF_D3: U12.32 (DQ3)
- new net NANDF_D4: U12.41 (DQ4)
- new net NANDF_D5: U12.42 (DQ5)
- new net NANDF_D6: U12.43 (DQ6)
- new net NANDF_D7: U12.44 (DQ7)
- new net NANDF_NWP: U12.19 (WP#)
- new net NAND_NRE: U12.8 (RE#)
- no-connect marks 3 -> 28
Other:
- note added: "32Gb Multi-level cell"
- note added: "MPU DDR3L RAM 2 GIGABYTES(D)"
- note added: "MPU NOR FLASH(D)"
- note added: "NAND FLASH(D)"
- note added: "replace all footprints with 0402"
- note removed: "EEPROM"
- note removed: "MPU DDR3L RAM 2 GIGABYTES"
- note removed: "MPU NOR FLASH"
- moved on the sheet: R136, R137, R138, R139, R140, R141, R142, R143, R144, R145, R146, R147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
