File: hardware/01-ECAD/01-KiCAD Files/AWG1000/DAC.kicad_sch (KiCad schematic)
At the start: 0 parts

Commit message: WIP.
Parts:
- added C? (x57): 22uF, symbol Device:C
- added C? (x12): 0.1uF, symbol Device:C
- added C? (x8): 4.7uF, symbol Device:C
- added FB? (x12): FerriteBead, symbol Device:FerriteBead
- added L? (x8): 1uH, symbol Device:L
- added R? (x59): 49.9, symbol Device:R_US
- added U? (x4): DAC3482IZAYR, ZAY196, symbol awg1000:DAC3482IZAYR
- added U? (x2): THS3217IRGVT, symbol awg1000:THS3217IRGVT
- added U? (x4): THS3095, symbol awg1000:THS3095
- added U?: CDCE62005RGZR, symbol awg1000:CDCE62005RGZR
- added Y?: LFTVXO076347CUTT, symbol awg1000:LFTVXO076347CUTT
Connections:
- new net: C?.1, L?.2, R?.1, R?.2, R?.2 (x2)
- new net: C?.1, C?.1, FB?.2, U?.1 (VCC_IN_SEC)
- new net: R?.1, R?.1, U?.2 (VIN-) (x4)
- new net: R?.1, R?.1, U?.12 (~PWRDWN)
- new net: R?.1, R?.1, R?.2, U?.12 (VIN-) (x2)
- new net: R?.2, R?.2, U?.11 (VOUT) (x2)
- new net: R?.1, R?.2, U?.15 (VMID_OUT) (x2)
- new net: R?.2, R?.2, U?.14 (VREF) (x2)
- new net: C?.1, C?.1, FB?.2, U?.18 (VCC_OUT)
- new net: C?.1, C?.1, FB?.2, U?.21 (VCC_OUT)
- new net: C?.2, U?.1 (VMID_IN) (x2)
- new net: C?.1, L?.2, R?.2, U?.2 (IN+) (x2)
- new net: C?.2, L?.2, R?.2, U?.3 (IN-) (x2)
- new net: R?.1, R?.1, U?.4 (PATHSEL) (x2)
- new net: R?.1, U?.6 (VO1) (x2)
- new net: R?.2, U?.9 (VIN+) (x2)
- new net: C?.1, Y?.4 (OUT)
- new net: C?.1, C?.1, FB?.2, U?.11 (VCC_OUT)
- new net: C?.1, L?.2, R?.1, R?.1 (x2)
- new net: C?.1, U?.4 (REG_CAP1)
- new net: C?.1, C?.1, FB?.2, U?.8 (VCC_OUT)
- new net: R?.1, R?.1, R?.2 (x2)
- new net: R?.2, R?.2, U?.6 (VOUT) (x4)
- new net: C?.1, L?.1, R?.2 (x2)
- new net: C?.1, C?.1, FB?.2, U?.5 (VCC1_PLL)
- new net: R?.1, U?.3 (VIN+) (x4)
- new net: C?.1, C?.1, FB?.2, Y?.1 (VC)
- new net: C?.1, R?.2 (x2)
- new net: U?.1 (REF), U?.1 (REF) (x2)
- new net: U?.4 (VS-), U?.4 (VS-) (x2)
- new net: U?.7 (VS+), U?.7 (VS+) (x2)
- new net: U?.8 (~PD), U?.8 (~PD) (x2)
- new net: C?.1, C?.1, FB?.2, U?.15 (VCC_AUXOUT)
- new net +3.3V_CLK: FB?.1, FB?.1, FB?.1, FB?.1, FB?.1, FB?.1, FB?.1, FB?.1, R?.1, R?.1, R?.2, R?.2
- new net -4.7V: C?.1, C?.1, C?.1, C?.1, FB?.1, FB?.1, U?.8 (-VCC1), U?.8 (-VCC1)
- new net 1.2V_DAC: U?.D9 (DACVDD), U?.E10 (DACVDD), U?.E5 (DIGVDD), U?.E6 (DIGVDD), U?.E7 (DIGVDD), U?.E9 (DACVDD), U?.F10 (DACVDD), U?.F5 (DIGVDD), U?.G10 (DACVDD), U?.H10 (DACVDD), U?.J10 (DACVDD), U?.J5 (DIGVDD), U?.K10 (DACVDD), U?.K5 (DIGVDD), U?.K6 (DIGVDD), U?.K7 (DIGVDD), U?.K9 (DACVDD), U?.L9 (DACVDD)
- new net 1.2V_DAC_CLK: C?.1, C?.1, U?.C12 (CLKVDD)
- new net 3.3V_DAC_AN: C?.1, C?.1, C?.1, C?.1, C?.1, C?.1, C?.1, C?.1, C?.1, C?.1, C?.1, C?.1, C?.1, C?.1, C?.1, C?.1, C?.1, C?.1, U?.D10 (AVDD), U?.E11 (AVDD), U?.F11 (AVDD), U?.G11 (AVDD), U?.H11 (AVDD), U?.J11 (AVDD), U?.K11 (AVDD), U?.L10 (AVDD)
- new net 3.3V_DAC_IO: U?.D5 (IOVDD), U?.D6 (IOVDD), U?.G5 (IOVDD), U?.H5 (IOVDD), U?.L5 (IOVDD), U?.L6 (IOVDD)
- new net 3095_1_OUT: R?.1
- new net 3095_2_OUT: R?.1
- new net 3217_1_out: C?.1, R?.1
- new net 3217_2_OUT: C?.1, R?.1
- new net 4.7V: C?.1, C?.1, C?.1, C?.1, FB?.1, FB?.1, R?.2, R?.2, U?.13 (+VCC1), U?.13 (+VCC1)
- new net D0_N: U?.P4 (D0N)
- new net D0_P: U?.N4 (D0P)
- new net D10_N: U?.D1 (D10N)
- new net D10_P: U?.D2 (D10P)
- new net D11_N: U?.C1 (D11N)
- new net D11_P: U?.C2 (D11P)
- new net D12_N: U?.B1 (D12N)
- new net D12_P: U?.A1 (D12P)
- new net D13_N: U?.B2 (D13N)
- new net D13_P: U?.A2 (D13P)
- new net D14_N: U?.B3 (D14N)
- new net D14_P: U?.A3 (D14P)
- new net D15_N: U?.B4 (D15N)
- new net D15_P: U?.A4 (D15P)
- new net D1_N: U?.P3 (D1N)
- new net D1_P: U?.N3 (D1P)
- new net D2_N: U?.P2 (D2N)
- new net D2_P: U?.N2 (D2P)
- new net D3_N: U?.P1 (D3N)
- new net D3_P: U?.N1 (D3P)
- new net D4_N: U?.M1 (D4N)
- new net D4_P: U?.M2 (D4P)
- new net D5_N: U?.L1 (D5N)
- new net D5_P: U?.L2 (D5P)
- new net D6_N: U?.K1 (D6N)
- new net D6_P: U?.K2 (D6P)
- new net D7_N: U?.J1 (D7N)
- new net D7_P: U?.J2 (D7P)
- new net D8_N: U?.F1 (D8N)
- new net D8_P: U?.F2 (D8P)
- new net D9_N: U?.E1 (D9N)
- new net D9_P: U?.E2 (D9P)
- new net DACCLK_N: C?.2, R?.2, U?.A11 (DACCLKN), U?.G1 (DATACLKN)
- new net DACCLK_P: C?.2, R?.1, U?.A12 (DACCLKP), U?.G2 (DATACLKP)
- new net DAC_CLK_N: C?.1, R?.2, R?.2, R?.2, U?.17 (U2N)
- new net DAC_CLK_P: C?.1, R?.2, U?.16 (U2P)
- new net FRAME_N: U?.H1 (FRAMEN)
- new net FRAME_P: U?.H2 (FRAMEP)
- new net GND: C?.1, C?.1, C?.1, C?.1, C?.2, C?.2, C?.2, C?.2, C?.2, C?.2, C?.2, C?.2, C?.2, C?.2, C?.2, C?.2, C?.2, C?.2, C?.2, C?.2, C?.2, C?.2, C?.2, C?.2, C?.2, C?.2, C?.2, C?.2, C?.2, C?.2, C?.2, C?.2, C?.2, C?.2, C?.2, C?.2, C?.2, C?.2, C?.2, C?.2, C?.2, C?.2, C?.2, C?.2, C?.2, C?.2, C?.2, C?.2, C?.2, C?.2, C?.2, C?.2, C?.2, C?.2, C?.2, C?.2, C?.2, C?.2, C?.2, C?.2, C?.2, C?.2, C?.2, C?.2, C?.2, C?.2, C?.2, C?.2, C?.2, C?.2, C?.2, C?.2, R?.1, R?.1, R?.1, R?.1, R?.1, R?.1, R?.1, R?.1, R?.1, R?.1, R?.1, R?.1, R?.2, R?.2, R?.2, R?.2, R?.2, R?.2, R?.2, R?.2, R?.2, R?.2, R?.2, R?.2, U?.17 (T_PAD), U?.17 (T_PAD), U?.2 (SEC_REF-), U?.36 (GND_VCO), U?.49 (GND_PAD), U?.7 (GND), U?.7 (GND), U?.A10 (GND), U?.A13 (GND), U?.A14 (GND), U?.B10 (GND), U?.B11 (GND), U?.B12 (GND), U?.B13 (GND), U?.B14 (GND), U?.C10 (GND), U?.C13 (GND), U?.C14 (GND), U?.C5 (GND), U?.C6 (GND), U?.C7 (GND), U?.C8 (GND), U?.C9 (GND), U?.D13 (GND), U?.D14 (GND), U?.D8 (GND), U?.E12 (GND), U?.E13 (GND), U?.E8 (GND), U?.F12 (GND), U?.F13 (GND), U?.F6 (GND), U?.F7 (GND), U?.F8 (GND), U?.F9 (GND), U?.G13 (GND), U?.G14 (GND), U?.G6 (GND), U?.G7 (GND), U?.G8 (GND), U?.G9 (GND), U?.H13 (GND), U?.H14 (GND), U?.H6 (GND), U?.H7 (GND), U?.H8 (GND), U?.H9 (GND), U?.J12 (GND), U?.J13 (GND), U?.J6 (GND), U?.J7 (GND), U?.J8 (GND), U?.J9 (GND), U?.K13 (GND), U?.K8 (GND), U?.L13 (GND), U?.L14 (GND), U?.L8 (GND), U?.M10 (GND), U?.M11 (GND), U?.M12 (GND), U?.M13 (GND), U?.M14 (GND), U?.M5 (GND), U?.M6 (GND), U?.M7 (GND), U?.M8 (GND), U?.M9 (GND), U?.N13 (GND), U?.N14 (GND), U?.P13 (GND), U?.P14 (GND), Y?.2 (GND)
- new net IOUT1_N: C?.1, C?.1, L?.1, L?.1, R?.2, R?.2, U?.E14 (IOUTIN)
- new net IOUT1_P: C?.2, C?.2, L?.1, L?.1, R?.1, R?.1, U?.K14 (IOUTQN)
- new net IOUT2_N: U?.J14 (IOUTQP)
- new net IOUT2_P: U?.F14 (IOUTIP)
- new net OSTR_N: U?.B9 (OSTRN)
- new net OSTR_P: U?.A9 (OSTRP)
- new net PARITY_N: U?.P5 (PARITYN)
- new net PARITY_P: U?.N5 (PARITYP)
- new net PLLAVDD: C?.1, C?.1, C?.1, U?.C11 (PLLAVDD), U?.D11 (PLLAVDD)
- new net SEC_CLK: C?.2, R?.1, R?.1, U?.3 (SEC_REF+)
- new net SYNC_N: U?.B5 (SYNCN)
- new net SYNC_P: U?.A5 (SYNCP)
- new net THS3217_I_N: C?.1, C?.1, C?.1, C?.1, FB?.2, FB?.2
- new net THS3217_I_P: C?.1, C?.1, C?.1, C?.1, FB?.2, FB?.2, U?.16 (+VCC2), U?.16 (+VCC2), U?.5 (-VCC2), U?.5 (-VCC2)
Other:
- note added: "DAC I/O"
- note added: "DAC POWER"
- note added: "DIFFERNETIAL TO SINGLE ENDDED"

Commit message: Update.
Parts:
- removed C? (x12): 0.1uF, symbol Device:C
- removed C? (x8): 4.7uF, symbol Device:C
- removed C? (x2): 22uF, symbol Device:C
- removed FB? (x8): FerriteBead, symbol Device:FerriteBead
- removed R? (x17): 49.9, symbol Device:R_US
- removed U?: CDCE62005RGZR, symbol awg1000:CDCE62005RGZR
- removed Y?: LFTVXO076347CUTT, symbol awg1000:LFTVXO076347CUTT
- added C270, C271, C272, C273, C275, C276, C289, C290, C293, C294, C296, C297: 220nF, Resistor_SMD:R_0402_1005Metric_Pad0.72x0.64mm_HandSolder, symbol Device:C
- added C274, C298: 9.1pF, Resistor_SMD:R_0402_1005Metric_Pad0.72x0.64mm_HandSolder, symbol Device:C
- added C278, C279, C280, C281, C282, C283, C299, C300, C303, C304, C306, C307: 10uF, Resistor_SMD:R_0402_1005Metric_Pad0.72x0.64mm_HandSolder, symbol Device:C
- added C313: 0.1uF, Resistor_SMD:R_0402_1005Metric_Pad0.72x0.64mm_HandSolder, symbol Device:C
- added D6, D7, D8, D9: D, symbol Device:D
- added K1, K2, K3, K4: EE2-5NU, Relay_SMD:Relay_DPDT_Kemet_EE2_NU, symbol Relay:EE2-5NU
- added Q1, Q2, Q3, Q4: BSN20, Package_TO_SOT_SMD:SOT-23, symbol Transistor_FET:BSN20
- added R104, R105, R65, R93: 49.9, Resistor_SMD:R_0402_1005Metric_Pad0.72x0.64mm_HandSolder, symbol Device:R_US
- added R109, R81: 30, Resistor_SMD:R_0402_1005Metric_Pad0.72x0.64mm_HandSolder, symbol Device:R_US
- added R110: 1.27k, Resistor_SMD:R_0402_1005Metric_Pad0.72x0.64mm_HandSolder, symbol Device:R_US
- added R112: 10, Resistor_SMD:R_0402_1005Metric_Pad0.72x0.64mm_HandSolder, symbol Device:R_US
- added R63, R64, R78, R79: 1k, Resistor_SMD:R_0402_1005Metric_Pad0.72x0.64mm_HandSolder, symbol Device:R_US
- added R66, R67, R69, R70, R71, R82, R83, R90, R91, R92: 10k, Resistor_SMD:R_0402_1005Metric_Pad0.72x0.64mm_HandSolder, symbol Device:R_US
- added R74: 20, Resistor_SMD:R_0402_1005Metric_Pad0.72x0.64mm_HandSolder, symbol Device:R_US
- added U30, U34: THS3095, Package_SO:Texas_R-PDSO-G8_EP2.95x4.9mm_Mask2.4x3.1mm_ThermalVias, symbol awg1000:THS3095
- C277, C302, C305, C337: renamed from C?; value 22uF -> 27pF; footprint (none) -> Resistor_SMD:R_0402_1005Metric_Pad0.72x0.64mm_HandSolder
- C284, C288: renamed from C?; value 22uF -> 10nF; footprint (none) -> Resistor_SMD:R_0402_1005Metric_Pad0.72x0.64mm_HandSolder
- C285, C286, C315, C316: renamed from C?; value 22uF -> 4.5pF; footprint (none) -> Resistor_SMD:R_0402_1005Metric_Pad0.72x0.64mm_HandSolder
- C287, C292, C312: renamed from C?; value 22uF -> 220nF; footprint (none) -> Resistor_SMD:R_0402_1005Metric_Pad0.72x0.64mm_HandSolder
- C291, C319: renamed from C?; value 22uF -> 3.2pF; footprint (none) -> Resistor_SMD:R_0402_1005Metric_Pad0.72x0.64mm_HandSolder
- C295, C308, C320, C321, C322, C323, C324, C325, C326, C327, C328, C330, C331, C332, C333, C335, C336, C338, C340, C342, C344, C345, C347, C348, C350, C351: renamed from C?; footprint (none) -> Resistor_SMD:R_0402_1005Metric_Pad0.72x0.64mm_HandSolder
- C301, C334: renamed from C?; value 22uF -> 8.2pF; footprint (none) -> Resistor_SMD:R_0402_1005Metric_Pad0.72x0.64mm_HandSolder
- C309, C311, C314, C318, C341, C346: renamed from C?; value 22uF -> 10nF; footprint (none) -> Resistor_SMD:R_0402_1005Metric_Pad0.72x0.64mm_HandSolder; VOLTAGE 6.3V -> 16V
- C310, C317, C329, C343, C349: renamed from C?; value 22uF -> 220nF; footprint (none) -> Resistor_SMD:R_0402_1005Metric_Pad0.72x0.64mm_HandSolder; VOLTAGE 6.3V -> 16V
- C339: renamed from C?; value 22uF -> 0; footprint (none) -> Resistor_SMD:R_0402_1005Metric_Pad0.72x0.64mm_HandSolder
- FB10, FB11, FB12, FB13: renamed from FB?; footprint (none) -> Inductor_SMD:L_0402_1005Metric_Pad0.77x0.64mm_HandSolder
- L16, L19: renamed from L?; value 1uH -> 56nH
- L17, L18, L21, L22: renamed from L?; value 1uH -> 30nH; footprint (none) -> Inductor_SMD:L_0402_1005Metric_Pad0.77x0.64mm_HandSolder
- L20, L23: renamed from L?; value 1uH -> 56nH; footprint (none) -> Inductor_SMD:L_0402_1005Metric_Pad0.77x0.64mm_HandSolder
- R100, R117, R118, R120, R121, R122, R124, R88, R89, R95, R96, R98: renamed from R?; value 49.9 -> 0; footprint (none) -> Resistor_SMD:R_0402_1005Metric_Pad0.72x0.64mm_HandSolder
- R101, R125: renamed from R?; value 49.9 -> 249; footprint (none) -> Resistor_SMD:R_0402_1005Metric_Pad0.72x0.64mm_HandSolder
- R102, R103, R113, R114, R115, R116, R119, R126, R75, R76, R77, R86, R87, R94: renamed from R?; footprint (none) -> Resistor_SMD:R_0402_1005Metric_Pad0.72x0.64mm_HandSolder
- R106, R127: renamed from R?; value 49.9 -> 162; footprint (none) -> Resistor_SMD:R_0402_1005Metric_Pad0.72x0.64mm_HandSolder
- R107, R108, R80, R84: renamed from R?; value 49.9 -> 30; footprint (none) -> Resistor_SMD:R_0402_1005Metric_Pad0.72x0.64mm_HandSolder
- R111, R85: renamed from R?; value 49.9 -> 40.2; footprint (none) -> Resistor_SMD:R_0402_1005Metric_Pad0.72x0.64mm_HandSolder
- R123, R68, R97, R99: renamed from R?; value 49.9 -> 150; footprint (none) -> Resistor_SMD:R_0402_1005Metric_Pad0.72x0.64mm_HandSolder
- R72, R73: renamed from R?; value 49.9 -> 20; footprint (none) -> Resistor_SMD:R_0402_1005Metric_Pad0.72x0.64mm_HandSolder
- U27: renamed from U?; footprint ZAY196 -> Package_BGA:Microchip_TFBGA-196_11x11mm_Layout14x14_P0.75mm_SMD
- U28, U29, U32, U33: renamed from U?; footprint (none) -> Package_SO:Texas_R-PDSO-G8_EP2.95x4.9mm_Mask2.4x3.1mm_ThermalVias
- U31, U35: renamed from U?; footprint (none) -> Package_DFN_QFN:QFN-16-1EP_4x4mm_P0.65mm_EP2.1x2.1mm_ThermalVias
Connections:
- net 1.2V_DAC: no longer U27.D9 (DACVDD), U27.E10 (DACVDD), U27.E9 (DACVDD), U27.F10 (DACVDD), U27.G10 (DACVDD), U27.H10 (DACVDD), U27.J10 (DACVDD), U27.K10 (DACVDD), U27.K5 (DIGVDD), U27.K6 (DIGVDD), U27.K7 (DIGVDD), U27.K9 (DACVDD)
- net 1.2V_DAC_CLK: now also U27.K9 (DACVDD); no longer U27.C12 (CLKVDD)
- net 3.3V_DAC_AN: now also U27.D5 (IOVDD), U27.D6 (IOVDD), U27.D9 (DACVDD), U27.E9 (DACVDD), U27.G5 (IOVDD), U27.H5 (IOVDD), U27.L5 (IOVDD), U27.L6 (IOVDD); no longer U27.D10 (AVDD), U27.E11 (AVDD), U27.F11 (AVDD), U27.G11 (AVDD), U27.H11 (AVDD), U27.J11 (AVDD), U27.K11 (AVDD), U27.L10 (AVDD)
- net 3.3V_DAC_IO: now also U27.A11 (DACCLKN), U27.B5 (SYNCN), U27.B9 (OSTRN), U27.G1 (DATACLKN), U27.H1 (FRAMEN), U27.P5 (PARITYN); no longer U27.D5 (IOVDD), U27.D6 (IOVDD), U27.G5 (IOVDD), U27.H5 (IOVDD), U27.L5 (IOVDD), U27.L6 (IOVDD)
- net 3217_1_out: now also R101.2, U31.11 (VOUT), R65.2
- net D0_N: now also U27.B8 (SLEEP); no longer U27.P4 (D0N)
- net D0_P: now also U27.J3 (NC); no longer U27.N4 (D0P)
- net D10_N: now also U27.B7 (NC); no longer U27.D1 (D10N)
- net D10_P: now also U27.M3 (NC); no longer U27.D2 (D10P)
- net D11_N: now also U27.C3 (NC); no longer U27.C1 (D11N)
- net D11_P: now also U27.M4 (NC); no longer U27.C2 (D11P)
- net D12_N: now also U27.C4 (NC); no longer U27.B1 (D12N)
- net D12_P: now also U27.N6 (NC); no longer U27.A1 (D12P)
- net D13_N: now also U27.D3 (NC); no longer U27.B2 (D13N)
- net D13_P: now also U27.N7 (NC); no longer U27.A2 (D13P)
- net D14_N: now also U27.D4 (NC); no longer U27.B3 (D14N)
- net D14_P: now also U27.N8 (NC); no longer U27.A3 (D14P)
- net D15_N: now also U27.E3 (NC); no longer U27.B4 (D15N)
- net D15_P: now also U27.N11 (NC); no longer U27.A4 (D15P)
- net D1_N: now also U27.N12 (ALARM); no longer U27.P3 (D1N)
- net D1_P: now also U27.J4 (NC); no longer U27.N3 (D1P)
- net D2_N: now also U27.G12 (EXTIO); no longer U27.P2 (D2N)
- net D2_P: now also U27.K3 (NC); no longer U27.N2 (D2P)
- net D3_N: now also U27.N10 (RESETB); no longer U27.P1 (D3N)
- net D3_P: now also U27.K4 (NC); no longer U27.N1 (D3P)
- net D4_N: now also U27.A8 (TESTMODE); no longer U27.M1 (D4N)
- net D4_P: now also U27.K12 (NC); no longer U27.M2 (D4P)
- net D5_N: now also U27.N9 (TXENABLE); no longer U27.L1 (D5N)
- net D5_P: now also U27.L3 (NC); no longer U27.L2 (D5P)
- net D6_N: no longer U27.K1 (D6N)
- net D6_P: now also U27.L4 (NC); no longer U27.K2 (D6P)
- net D7_N: now also U27.A6 (NC); no longer U27.J1 (D7N)
- net D7_P: now also U27.L7 (NC); no longer U27.J2 (D7P)
- net D8_N: now also U27.A7 (NC); no longer U27.F1 (D8N)
- net D8_P: now also U27.L11 (NC); no longer U27.F2 (D8P)
- net D9_N: now also U27.B6 (NC); no longer U27.E1 (D9N)
- net D9_P: now also U27.L12 (NC); no longer U27.E2 (D9P)
- net DACCLK_N: now also U27.D7 (VFUSE), U27.H12 (BIASJ); no longer U27.A11 (DACCLKN), U27.G1 (DATACLKN)
- net DACCLK_P: now also U27.G4 (NC), U27.H3 (NC); no longer U27.A12 (DACCLKP), U27.G2 (DATACLKP)
- net FRAME_N: now also U27.P9 (SCLK); no longer U27.H1 (FRAMEN)
- net FRAME_P: no longer U27.H2 (FRAMEP)
- net GND: now also R75.1, U27.A1 (D12P), U27.A12 (DACCLKP), U27.A2 (D13P), U27.A3 (D14P), U27.A4 (D15P), U27.A5 (SYNCP), U27.A9 (OSTRP), U27.C2 (D11P), U27.D2 (D10P), U27.E2 (D9P), U27.F14 (IOUTIP), U27.F2 (D8P), U27.G2 (DATACLKP), U27.H2 (FRAMEP), U27.J14 (IOUTQP), U27.J2 (D7P), U27.K2 (D6P), U27.L2 (D5P), U27.M2 (D4P), U27.N1 (D3P), U27.N2 (D2P), U27.N3 (D1P), U27.N4 (D0P), U27.N5 (PARITYP), C270.2, C271.1, C272.2, C273.1, C274.2, C275.2, C276.1, C278.2, C279.1, C280.2, C281.1, C282.2, C283.1, C289.2, C290.1, C293.2, C294.1, C296.2, C297.1, C298.2, C299.2, C300.1, C303.2, C304.1, C306.2, C307.1, C313.1, Q1.2 (S), Q2.2 (S), Q3.2 (S), Q4.2 (S), R105.1, R112.1, R66.2, R67.2, R82.2, R83.2; no longer R75.2, U27.A10 (GND), U27.A13 (GND), U27.A14 (GND), U27.B10 (GND), U27.B11 (GND), U27.B12 (GND), U27.B13 (GND), U27.B14 (GND), U27.C10 (GND), U27.C13 (GND), U27.C14 (GND), U27.D13 (GND), U27.D14 (GND), U27.E12 (GND), U27.E13 (GND), U27.F12 (GND), U27.F13 (GND), U27.G13 (GND), U27.G14 (GND), U27.H13 (GND), U27.H14 (GND), U27.J12 (GND), U27.J13 (GND), U27.K13 (GND), U27.L13 (GND), U27.L14 (GND), U27.M10 (GND), U27.M11 (GND), U27.M12 (GND), U27.M13 (GND), U27.M14 (GND), U27.N13 (GND), U27.N14 (GND), U27.P13 (GND), U27.P14 (GND)
- net IOUT1_N: now also U27.F3 (NC); no longer U27.E14 (IOUTIN)
- net IOUT1_P: now also U27.F4 (NC); no longer U27.K14 (IOUTQN)
- net IOUT2_N: now also U27.P8 (NC); no longer U27.J14 (IOUTQP)
- net IOUT2_P: now also U27.P7 (NC); no longer U27.F14 (IOUTIP)
- net OSTR_N: now also U27.P12 (SDO); no longer U27.B9 (OSTRN)
- net PARITY_N: now also U27.P11 (SDIO); no longer U27.P5 (PARITYN)
- net PARITY_P: now also U27.G3 (NC); no longer U27.N5 (PARITYP)
- net PLLAVDD: now also U27.K5 (DIGVDD), U27.K6 (DIGVDD); no longer U27.C11 (PLLAVDD), U27.D11 (PLLAVDD)
- net SYNC_N: now also U27.D12 (LPF); no longer U27.B5 (SYNCN)
- net SYNC_P: no longer U27.A5 (SYNCP)
- net THS3217_I_N: no longer C346.1, C349.1, FB13.2
- net THS3217_I_P: no longer C318.1, C329.1, FB12.2, U35.16 (+VCC2), U35.5 (-VCC2)
- net at L16.1: now also C274.1, R65.1
- net at C277.1, L16.2, R68.1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: now also R74.2
- net RF1-: now reaches U28.2 (VIN-)
- net RF1-: now also R75.2, U29.2 (VIN-), K2.9, U30.2 (VIN-)
- net CH2_DIS: now reaches U35.10 (DIS)
- net at L19.1: now also C298.1, R93.1
- net at C302.1, L19.2, R102.2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: now also R104.2
- net at R80.1, R84.1, R85.2: now also R81.1
- net RF1+: now reaches R84.2, U28.6 (VOUT)
- net RF1+: now also K2.4
- net at R107.1, R108.1, R111.2: now also R109.1
- net RF2-: now reaches U33.2 (VIN-)
- net RF2-: now also U32.2 (VIN-), K4.9, R105.2, U34.2 (VIN-)
- net at U28.1 (REF), U29.1 (REF): now also U30.1 (REF)
- net -15V: now reaches U28.4 (VS-), U29.4 (VS-)
- net -15V: now also U32.1 (REF), U33.1 (REF), C289.1, C290.2, C293.1, C294.2, C296.1, C297.2, C299.1, C300.2, C303.1, C304.2, C306.1, C307.2, U30.4 (VS-), U34.1 (REF)
- net +15V: now reaches U28.7 (VS+), U29.7 (VS+)
- net +15V: now also U32.7 (VS+), U33.7 (VS+), C270.1, C271.2, C272.1, C273.2, C275.1, C276.2, C278.1, C279.2, C280.1, C281.2, C282.1, C283.2, U30.7 (VS+), U34.7 (VS+)
- net 3095_1_EN: now reaches U28.8 (~{PD}), U29.8 (~{PD})
- net 3095_1_EN: now also U30.8 (~{PD})
- net RF2+: now reaches R107.2, U32.6 (VOUT)
- net RF2+: now also K4.4
- net CH1_DIS: now reaches U31.10 (DIS)
- net at U32.4 (VS-), U33.4 (VS-): now also U34.4 (VS-)
- net 3095_2_EN: now reaches U32.8 (~{PD}), U33.8 (~{PD})
- net 3095_2_EN: now also U34.8 (~{PD})
- net -4.7V renamed -7V
- net 4.7V renamed +7V
- net +7V: no longer U35.13 (+VCC1)
- removed net OSTR_P: U27.A9 (OSTRP)
- new net: Q2.1 (G), R64.2, R67.1
- new net: D7.2 (A), K2.1, Q2.3 (D)
- new net: K3.10, R90.1
- new net: K3.3, R90.2
- new net: Q1.1 (G), R63.2, R66.1
- new net: Q3.1 (G), R78.2, R82.1
- new net: D8.2 (A), K3.1, Q3.3 (D)
- new net: D9.1 (K), K4.12
- new net: D9.2 (A), K4.1, Q4.3 (D)
- new net: R109.2, U34.6 (VOUT)
- new net: D6.2 (A), K1.1, Q1.3 (D)
- new net: K1.10, R69.1
- new net: D6.1 (K), K1.12
- new net: K1.3, R69.2
- new net: K1.4, K2.3
- new net: K1.5, R70.2
- new net: K1.8, R70.1
- new net: K1.9, K2.10
- new net: R110.1, R112.2
- new net: K3.8, R91.1
- new net: K3.5, R91.2
- new net: Q4.1 (G), R79.2, R83.1
- new net: D8.1 (K), K3.12
- new net: C313.2, U27.E10 (DACVDD)
- new net: R110.2, U27.J11 (AVDD)
- new net: D7.1 (K), K2.12
- new net: R74.1, U30.3 (VIN+)
- new net: K4.5, R92.1
- new net: K4.8, R92.2
- new net: R104.1, U34.3 (VIN+)
- new net: K3.4, K4.3
- new net: K3.9, K4.10
- new net: K2.5, R71.1
- new net: K2.8, R71.2
- new net: R81.2, U30.6 (VOUT)
- new net 1: R63.1, R64.1, R78.1, R79.1
- new net 1.2V_DAC_DVDD: U27.D1 (D10N), U27.E1 (D9N), U27.F1 (D8N), U27.J1 (D7N), U27.K1 (D6N), U27.L1 (D5N), U27.M1 (D4N), U27.P1 (D3N)
- new net 1.2V_DAC_VDD: U27.P2 (D2N), U27.P3 (D1N), U27.P4 (D0N)
- new net 3217_2_out: R93.2
- new net DAC_MISO: U27.D10 (AVDD)
- new net DAC_MOSI: U27.G11 (AVDD)
- new net DAC_SCLK: U27.F11 (AVDD)
- new net THS3217_2_N: C346.1, C349.1, FB13.2
- new net THS3217_2_P: C318.1, C329.1, FB12.2, U35.16 (+VCC2), U35.5 (-VCC2)
Other:
- note added: "3rd Order Butterworth LPF BW: 200 MHz"
- note added: "CHANNEL 1"
- note added: "CHANNEL 2"
- note added: "GAIN SELECTION RELAYS"
- note added: "Interstage Filter BW 500 MHz"
- note added: "OUTPUT DRIVE OPAMPS"
- note added: "Reconstruction Filter BW 500 MHz"
- moved on the sheet: C277, C302, C320, C321, C322, C323, C324, C325, C326, C327, C328, L16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

Commit message: Update.
Parts:
- removed C320, C321, C322, C323, C324, C325, C326, C327, C338, C340, C344, C347, C351: 22uF, Resistor_SMD:R_0402_1005Metric_Pad0.72x0.64mm_HandSolder, symbol Device:C
- added C270, C271, C272, C273, C275, C276, C330, C331, C334, C337, C343, C345, C350: 0.1uF, awg1000:C0201_L, symbol Device:C
- added R55: 49.9, Resistor_SMD:R_0402_1005Metric_Pad0.72x0.64mm_HandSolder, symbol Device:R_US
- C280: renamed from C270; footprint Resistor_SMD:R_0402_1005Metric_Pad0.72x0.64mm_HandSolder -> awg1000:C0201_L
- C281: renamed from C271; footprint Resistor_SMD:R_0402_1005Metric_Pad0.72x0.64mm_HandSolder -> awg1000:C0201_L
- C282: renamed from C272; footprint Resistor_SMD:R_0402_1005Metric_Pad0.72x0.64mm_HandSolder -> awg1000:C0201_L
- C283: renamed from C273; footprint Resistor_SMD:R_0402_1005Metric_Pad0.72x0.64mm_HandSolder -> awg1000:C0201_L
- C285: renamed from C275; footprint Resistor_SMD:R_0402_1005Metric_Pad0.72x0.64mm_HandSolder -> awg1000:C0201_L
- C286: renamed from C276; footprint Resistor_SMD:R_0402_1005Metric_Pad0.72x0.64mm_HandSolder -> awg1000:C0201_L
- C297: renamed from C287; footprint Resistor_SMD:R_0402_1005Metric_Pad0.72x0.64mm_HandSolder -> awg1000:C0201_L
- C299: renamed from C289; footprint Resistor_SMD:R_0402_1005Metric_Pad0.72x0.64mm_HandSolder -> awg1000:C0201_L
- C300: renamed from C290; footprint Resistor_SMD:R_0402_1005Metric_Pad0.72x0.64mm_HandSolder -> awg1000:C0201_L
- C302: renamed from C292; footprint Resistor_SMD:R_0402_1005Metric_Pad0.72x0.64mm_HandSolder -> awg1000:C0201_L
- C303: renamed from C293; footprint Resistor_SMD:R_0402_1005Metric_Pad0.72x0.64mm_HandSolder -> awg1000:C0201_L
- C304: renamed from C294; footprint Resistor_SMD:R_0402_1005Metric_Pad0.72x0.64mm_HandSolder -> awg1000:C0201_L
- C306: renamed from C296; footprint Resistor_SMD:R_0402_1005Metric_Pad0.72x0.64mm_HandSolder -> awg1000:C0201_L
- C307: renamed from C297; footprint Resistor_SMD:R_0402_1005Metric_Pad0.72x0.64mm_HandSolder -> awg1000:C0201_L
- C320: renamed from C310; footprint Resistor_SMD:R_0402_1005Metric_Pad0.72x0.64mm_HandSolder -> awg1000:C0201_L
- C322: renamed from C312; footprint Resistor_SMD:R_0402_1005Metric_Pad0.72x0.64mm_HandSolder -> awg1000:C0201_L
- C323: renamed from C313; footprint Resistor_SMD:R_0402_1005Metric_Pad0.72x0.64mm_HandSolder -> awg1000:C0201_L
- C327: renamed from C317; footprint Resistor_SMD:R_0402_1005Metric_Pad0.72x0.64mm_HandSolder -> awg1000:C0201_L
- C332, C333, C335, C336, C342, C348: value 22uF -> 0.1uF; footprint Resistor_SMD:R_0402_1005Metric_Pad0.72x0.64mm_HandSolder -> awg1000:C0201_L
- C339: renamed from C329; footprint Resistor_SMD:R_0402_1005Metric_Pad0.72x0.64mm_HandSolder -> awg1000:C0201_L
- C353: renamed from C343; footprint Resistor_SMD:R_0402_1005Metric_Pad0.72x0.64mm_HandSolder -> awg1000:C0201_L
- C359: renamed from C349; footprint Resistor_SMD:R_0402_1005Metric_Pad0.72x0.64mm_HandSolder -> awg1000:C0201_L
- L16, L19: footprint (none) -> Inductor_SMD:L_0402_1005Metric_Pad0.77x0.64mm_HandSolder
- U27: footprint Package_BGA:Microchip_TFBGA-196_11x11mm_Layout14x14_P0.75mm_SMD -> awg1000:ZAY0196A
- renumbered C274 to C284, C277 to C287, C278 to C288, C279 to C289, C280 to C290, C281 to C291, C282 to C292, C283 to C293, C284 to C294, C285 to C295, C286 to C296, C288 to C298, C291 to C301, C295 to C305, C298 to C308, C299 to C309, C300 to C310, C301 to C311, C302 to C312, C303 to C313, C304 to C314, C305 to C315, C306 to C316, C307 to C317, C308 to C318, C309 to C319, C311 to C321, C314 to C324, C315 to C325, C316 to C326, C318 to C328, C319 to C329, C328 to C338, C330 to C340, C331 to C341, C334 to C344, C337 to C347, C339 to C349, C341 to C351, C345 to C355, C346 to C356, C350 to C360
Connections:
- net 3217_2_OUT is gone; now on net 3217_2_out: R126.1
- net +7V: now also U35.13 (+VCC1)
- net -15V: now also U32.4 (VS-), U33.4 (VS-), U34.4 (VS-); no longer U32.1 (REF), U33.1 (REF), U34.1 (REF)
- net 1.2V_DAC: now also C332.1, C333.1, C335.1, C336.1, C360.1, U27.E10 (DACVDD), U27.F10 (DACVDD), U27.G10 (DACVDD), U27.H10 (DACVDD), U27.J10 (DACVDD), U27.K10 (DACVDD), C334.1, C337.1, C343.1, C345.1; no longer U27.E5 (DIGVDD), U27.E6 (DIGVDD), U27.E7 (DIGVDD), U27.F5 (DIGVDD), U27.J5 (DIGVDD), U27.L9 (DACVDD)
- net 1.2V_DAC_CLK: now also C342.1, U27.C12 (CLKVDD); no longer C332.1, U27.K9 (DACVDD)
- net 1.2V_DAC_DVDD: now also U27.E5 (DIGVDD), U27.E6 (DIGVDD), U27.E7 (DIGVDD), U27.F5 (DIGVDD), U27.J5 (DIGVDD), U27.K5 (DIGVDD), U27.K6 (DIGVDD), U27.K7 (DIGVDD); no longer U27.D1 (D10N), U27.E1 (D9N), U27.F1 (D8N), U27.J1 (D7N), U27.K1 (D6N), U27.L1 (D5N), U27.M1 (D4N), U27.P1 (D3N)
- net 1.2V_DAC_VDD: now also U27.D9 (DACVDD), U27.E9 (DACVDD), U27.K9 (DACVDD), U27.L9 (DACVDD); no longer U27.P2 (D2N), U27.P3 (D1N), U27.P4 (D0N)
- net 3.3V_DAC_AN: now also U27.D10 (AVDD), U27.E11 (AVDD), U27.F11 (AVDD), U27.G11 (AVDD), U27.H11 (AVDD), U27.J11 (AVDD), U27.K11 (AVDD), U27.L10 (AVDD), C270.2, C271.2, C272.2, C273.2, C275.2, C276.2, C330.2, C331.2; no longer C333.1, C335.1, C336.1, C342.1, C360.1, U27.D5 (IOVDD), U27.D6 (IOVDD), U27.D9 (DACVDD), U27.E9 (DACVDD), U27.G5 (IOVDD), U27.H5 (IOVDD), U27.L5 (IOVDD), U27.L6 (IOVDD)
- net 3.3V_DAC_IO: now also U27.D5 (IOVDD), U27.D6 (IOVDD), U27.G5 (IOVDD), U27.H5 (IOVDD), U27.L5 (IOVDD), U27.L6 (IOVDD); no longer U27.A11 (DACCLKN), U27.B5 (SYNCN), U27.B9 (OSTRN), U27.G1 (DATACLKN), U27.H1 (FRAMEN), U27.P5 (PARITYN)
- net 3217_1_out: now also R55.1; no longer R101.2, U31.11 (VOUT)
- net D0_N: now also U27.P4 (D0N); no longer U27.B8 (SLEEP)
- net D0_P: now also U27.N4 (D0P); no longer U27.J3 (NC)
- net D10_N: now also U27.D1 (D10N); no longer U27.B7 (NC)
- net D10_P: now also U27.D2 (D10P); no longer U27.M3 (NC)
- net D11_N: now also U27.C1 (D11N); no longer U27.C3 (NC)
- net D11_P: now also U27.C2 (D11P); no longer U27.M4 (NC)
- net D12_N: now also U27.B1 (D12N); no longer U27.C4 (NC)
- net D12_P: now also U27.A1 (D12P); no longer U27.N6 (NC)
- net D13_N: now also U27.B2 (D13N); no longer U27.D3 (NC)
- net D13_P: now also U27.A2 (D13P); no longer U27.N7 (NC)
- net D14_N: now also U27.B3 (D14N); no longer U27.D4 (NC)
- net D14_P: now also U27.A3 (D14P); no longer U27.N8 (NC)
- net D15_N: now also U27.B4 (D15N); no longer U27.E3 (NC)
- net D15_P: now also U27.A4 (D15P); no longer U27.N11 (NC)
- net D1_N: now also U27.P3 (D1N); no longer U27.N12 (ALARM)
- net D1_P: now also U27.N3 (D1P); no longer U27.J4 (NC)
- net D2_N: now also U27.P2 (D2N); no longer U27.G12 (EXTIO)
- net D2_P: now also U27.N2 (D2P); no longer U27.K3 (NC)
- net D3_N: now also U27.P1 (D3N); no longer U27.N10 (RESETB)
- net D3_P: now also U27.N1 (D3P); no longer U27.K4 (NC)
- net D4_N: now also U27.M1 (D4N); no longer U27.A8 (TESTMODE)
- net D4_P: now also U27.M2 (D4P); no longer U27.K12 (NC)
- net D5_N: now also U27.L1 (D5N); no longer U27.N9 (TXENABLE)
- net D5_P: now also U27.L2 (D5P); no longer U27.L3 (NC)
- net D6_N: now also U27.K1 (D6N)
- net D6_P: now also U27.K2 (D6P); no longer U27.L4 (NC)
- net D7_N: now also U27.J1 (D7N); no longer U27.A6 (NC)
- net D7_P: now also U27.J2 (D7P); no longer U27.L7 (NC)
- net D8_N: now also U27.F1 (D8N); no longer U27.A7 (NC)
- net D8_P: now also U27.F2 (D8P); no longer U27.L11 (NC)
- net D9_N: now also U27.E1 (D9N); no longer U27.B6 (NC)
- net D9_P: now also U27.E2 (D9P); no longer U27.L12 (NC)
- net DACCLK_N: now also U27.A11 (DACCLKN), U27.G1 (DATACLKN); no longer U27.D7 (VFUSE), U27.H12 (BIASJ)
- net DACCLK_P: now also U27.A12 (DACCLKP), U27.G2 (DATACLKP); no longer U27.G4 (NC), U27.H3 (NC)
- net DAC_MISO: no longer U27.D10 (AVDD)
- net DAC_MOSI: no longer U27.G11 (AVDD)
- net DAC_SCLK: no longer U27.F11 (AVDD)
- net FRAME_N: now also U27.H1 (FRAMEN); no longer U27.P9 (SCLK)
- net FRAME_P: now also U27.H2 (FRAMEP)
- net GND: now also U27.A10 (GND), U27.A13 (GND), U27.A14 (GND), U27.B10 (GND), U27.B11 (GND), U27.B12 (GND), U27.B13 (GND), U27.B14 (GND), U27.C10 (GND), U27.C13 (GND), U27.C14 (GND), U27.D13 (GND), U27.D14 (GND), U27.E12 (GND), U27.E13 (GND), U27.F12 (GND), U27.F13 (GND), U27.G13 (GND), U27.G14 (GND), U27.H13 (GND), U27.H14 (GND), U27.J12 (GND), U27.J13 (GND), U27.K13 (GND), U27.L13 (GND), U27.L14 (GND), U27.M10 (GND), U27.M11 (GND), U27.M12 (GND), U27.M13 (GND), U27.M14 (GND), U27.N13 (GND), U27.N14 (GND), U27.P13 (GND), U27.P14 (GND), C270.1, C271.1, C272.1, C273.1, C275.1, C276.1, C330.1, C331.1, C334.2, C337.2, C343.2, C345.2, C350.2; no longer U27.A1 (D12P), U27.A12 (DACCLKP), U27.A2 (D13P), U27.A3 (D14P), U27.A4 (D15P), U27.A5 (SYNCP), U27.A9 (OSTRP), U27.C2 (D11P), U27.D2 (D10P), U27.E2 (D9P), U27.F14 (IOUTIP), U27.F2 (D8P), U27.G2 (DATACLKP), U27.H2 (FRAMEP), U27.J14 (IOUTQP), U27.J2 (D7P), U27.K2 (D6P), U27.L2 (D5P), U27.M2 (D4P), U27.N1 (D3P), U27.N2 (D2P), U27.N3 (D1P), U27.N4 (D0P), U27.N5 (PARITYP)
- net IOUT1_N: now also U27.K14 (IOUTQN); no longer U27.F3 (NC)
- net IOUT1_P: now also U27.J14 (IOUTQP); no longer U27.F4 (NC)
- net IOUT2_N: now also U27.E14 (IOUTIN); no longer U27.P8 (NC)
- net IOUT2_P: now also U27.F14 (IOUTIP); no longer U27.P7 (NC)
- net OSTR_N: now also U27.B9 (OSTRN); no longer U27.P12 (SDO)
- net PARITY_N: now also U27.P5 (PARITYN); no longer U27.P11 (SDIO)
- net PARITY_P: now also U27.N5 (PARITYP); no longer U27.G3 (NC)
- net PLLAVDD: now also U27.C11 (PLLAVDD), U27.D11 (PLLAVDD), C350.1; no longer U27.K5 (DIGVDD), U27.K6 (DIGVDD)
- net SYNC_N: now also U27.B5 (SYNCN); no longer U27.D12 (LPF)
- net SYNC_P: now also U27.A5 (SYNCP)
- net THS3217_2_N: now also U35.5 (-VCC2)
- net THS3217_2_P: no longer U35.5 (-VCC2)
- net THS3217_I_N: now also U31.5 (-VCC2)
- net THS3217_I_P: no longer U31.5 (-VCC2)
- net at C323.2: no longer U27.E10 (DACVDD)
- net at R110.2: no longer U27.J11 (AVDD)
- new net: R101.2, R55.2, U31.11 (VOUT)
- new net: U32.1 (REF), U33.1 (REF), U34.1 (REF)
Other:
- moved on the sheet: U27A, U27B, U27C, U27D

Commit message: Update.
Parts:
- added FB17, FB18: FerriteBead, Inductor_SMD:L_0402_1005Metric_Pad0.77x0.64mm_HandSolder, symbol Device:FerriteBead
- C270, C271, C272, C273, C275, C276, C280, C281, C282, C283, C284, C285, C286, C287, C288, C289, C290, C291, C292, C293, C294, C295, C296, C297, C298, C299, C300, C301, C302, C303, C304, C305, C306, C307, C308, C309, C310, C311, C312, C313, C314, C315, C316, C317, C318, C319, C320, C321, C322, C323, C324, C325, C326, C327, C328, C329, C330, C331, C332, C333, C334, C335, C336, C337, C338, C339, C340, C341, C342, C343, C344, C345, C347, C348, C349, C350, C351, C353, C355, C356, C359, C360: symbol Device:C -> awg1000:CAP_UNPOL
- D6, D7, D8, D9: footprint (none) -> Diode_SMD:D_SMA
- K1, K2, K3, K4: footprint Relay_SMD:Relay_DPDT_Kemet_EE2_NU -> awg1000:Relay_DPDT_Kemet_EE2_NU
- R100, R101, R102, R103, R104, R105, R106, R107, R108, R109, R110, R111, R112, R113, R114, R115, R116, R117, R118, R119, R120, R121, R122, R123, R124, R125, R126, R127, R55, R63, R64, R65, R66, R67, R68, R69, R70, R71, R72, R73, R74, R75, R76, R77, R78, R79, R80, R81, R82, R83, R84, R85, R86, R87, R88, R89, R90, R91, R92, R93, R94, R95, R96, R97, R98, R99: symbol Device:R_US -> awg1000:R
- U28, U29, U30, U32, U33, U34: footprint Package_SO:Texas_R-PDSO-G8_EP2.95x4.9mm_Mask2.4x3.1mm_ThermalVias -> awg1000:Texas_R-PDSO-G8_EP2.95x4.9mm_Mask2.4x3.1mm_ThermalVias
Connections:
- net 1.2V_DAC: no longer U27.E10 (DACVDD), U27.F10 (DACVDD), U27.G10 (DACVDD), U27.H10 (DACVDD), U27.J10 (DACVDD), U27.K10 (DACVDD)
- net 1.2V_DAC_VDD: now also U27.E10 (DACVDD), U27.F10 (DACVDD), U27.G10 (DACVDD), U27.H10 (DACVDD), U27.J10 (DACVDD), U27.K10 (DACVDD)
- net 3.3V_DAC_AN: now also FB17.1, FB18.1
- net 3.3V_DAC_IO: now also FB18.2
- net PLLAVDD: now also FB17.2
- net DACOSTR_P: now reaches U27.A9 (OSTRP)
- net OSTR_N renamed DACOSTR_N
- no-connect marks 0 -> 5
Other:
- note added: "1.2V"
- note added: "100mA"
- note added: "125mA"
- note added: "3.3V"
- note added: "500mA"
- note added: "705A"
- note added: "CURRENT"
- note added: "LINEAR"
- note added: "NET NAME"
- note added: "POWER SUPPLIES SUMMERY"
- note added: "SWITCHING"
- note added: "TYPE"
- note added: "VOLT"
