File: hardware/01-ECAD/01-KiCAD Files/AWG1000/INTERFACE.kicad_sch (KiCad schematic)
At the start: 0 parts

Commit message: WIP: update
Parts:
- added J? (x2): 031-6233, symbol Connector:Conn_Coaxial
Other:
- note added: "WAVEFORM OUTPUT"
Changed lines of the file:
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@@
+    (effects (font (size 5.08 5.08) (thickness 1.016) bold) (justify right bottom))
+  )
+  (text "WAVEFORM OUTPUT\n" (at 383.54 162.56 180)
     (effects (font (size 5.08 5.08) (thickness 1.016) bold) (justify right bottom))
   )
@@
     )
   )
+  (symbol (lib_id "Connector:Conn_Coaxial") (at 355.6 177.8 0) (unit 1)
+    (in_bom yes) (on_board yes)
+    (property "Reference" "J?" (id 0) (at 355.854 174.752 0))
+    (property "Value" "031-6233" (id 1) (at 358.521 177.8 90))
+    (property "Footprint" "" (id 2) (at 355.6 177.8 0)
+      (effects (font (size 1.27 1.27)) hide)
+    )
+    (property "Datasheet" " ~" (id 3) (at 355.6 177.8 0)
+      (effects (font (size 1.27 1.27)) hide)
+    )
+    (pin "1")
+    (pin "2")
+  )
+  (symbol (lib_id "Connector:Conn_Coaxial") (at 355.6 198.12 0) (unit 1)
+    (in_bom yes) (on_board yes)
+    (property "Reference" "J?" (id 0) (at 355.854 195.072 0))
+    (property "Value" "031-6233" (id 1) (at 358.521 198.12 90))
+    (property "Footprint" "" (id 2) (at 355.6 198.12 0)
+      (effects (font (size 1.27 1.27)) hide)
+    )
+    (property "Datasheet" " ~" (id 3) (at 355.6 198.12 0)
+      (effects (font (size 1.27 1.27)) hide)
+    )
+    (pin "1")
+    (pin "2")
+  )
 )

Commit message: WIP.
Parts:
- added J2: TF31-50S-0.5SH(800), awg1000:TF31-50S-0.5SH(800), symbol awg1000:LCD_FFC
- added J?: USB1040-GF-L-B, symbol awg1000:USB1040-GF-L-B
- gave numbers to parts that had none: 2
Connections:
- net LCD_B0: now also J2.19 (B0)
- net LCD_B1: now also J2.18 (B1)
- net LCD_B2: now also J2.17 (B2)
- net LCD_B3: now also J2.16 (B3)
- net LCD_B4: now also J2.15 (B4)
- net LCD_B5: now also J2.14 (B5)
- net LCD_B6: now also J2.13 (B6)
- net LCD_B7: now also J2.12 (B7)
- net LCD_CLK: now also J2.37 (DCLK)
- net LCD_ENABLE: now also J2.9 (DE)
- net LCD_G0: now also J2.27 (G0)
- net LCD_G1: now also J2.26 (G1)
- net LCD_G2: now also J2.25 (G2)
- net LCD_G3: now also J2.24 (G3)
- net LCD_G4: now also J2.23 (G4)
- net LCD_G5: now also J2.22 (G5)
- net LCD_G6: now also J2.21 (G6)
- net LCD_G7: now also J2.20 (G7)
- net LCD_HSYNC: now also J2.11 (HSYNC)
- net LCD_R0: now also J2.35 (R0)
- net LCD_R1: now also J2.34 (R1)
- net LCD_R2: now also J2.33 (R2)
- net LCD_R3: now also J2.32 (R3)
- net LCD_R4: now also J2.31 (R4)
- net LCD_R5: now also J2.30 (R5)
- net LCD_R6: now also J2.29 (R6)
- net LCD_R7: now also J2.28 (R7)
- net LCD_VSYNC: now also J2.10 (VSYNC)
- new net BKLT_N: J2.3 (LEDK), J2.4 (LEDK)
- new net BKLT_P: J2.1 (LEDA), J2.2 (LEDA)
- new net GND: J2.36 (GND), J2.38 (GND), J2.48 (GND), J2.5 (GND)
- no-connect marks 0 -> 3
Other:
- note removed: "USB"

Commit message: WIP
Parts:
- added C?: 220uF, awg1000:EEE-FK1H221GP, symbol awg1000:CAP_POL
- added C?: 0.1uF, symbol Device:C
- added FB? (x2): FerriteBead, symbol Device:FerriteBead
- added FL?: Filter_EMI_CommonMode, symbol Device:Filter_EMI_CommonMode
- added U?: SRV05-4, Package_TO_SOT_SMD:SOT-23-6, symbol Power_Protection:SRV05-4
Connections:
- net GND: now also J?.4 (GND), C?.2, C?.2, FB?.2, U?.2 (VN)
- net VBUS: now reaches J?.1 (VBUS)
- net VBUS: now also C?.1, C?.1, FB?.1, U?.5 (VP)
- net USB_N: now reaches J?.2 (D-)
- net USB_N: now also FL?.3, U?.1 (IO1)
- net USB_P: now reaches J?.3 (D+)
- net USB_P: now also FL?.1, U?.6 (IO4)
- net at J?.5 (S1): now also J?.6 (S2), FB?.1
- new net USB_5V: FB?.2
- new net USB_F_P: FL?.2, FL?.4
- no-connect marks 3 -> 5
Other:
- note added: "TOUCH INTERFACE"
- note added: "USB"
- moved on the sheet: J?

Commit message: WIP.
Parts:
- added C?: 0.1uF, symbol Device:C
- added J?: 031-6233, symbol Connector:Conn_Coaxial
- added R? (x3): 49.9, symbol Device:R_US
Connections:
- net GND: now also J?.2 (Ext), R?.1, R?.1
- new net: C?.2, J?.1 (In), R?.2
- new net CDC-PRIREF+: C?.1, R?.1, R?.2
Other:
- note added: "INTERFACE BNC CONNECTORS"
- note added: "TOUCH I2C"
- note removed: "TOUCH INTERFACE"
- note removed: "WAVEFORM OUTPUT"
- note removed: "https://www.alibaba.com/product-detail/PCAP-Touch-Industrial-Landscape-Capacitive-1024x600_60825225733.html?spm=a2700.galleryofferlist.normal_offer.d_image.6aee5bb9RCgBEq"
- moved on the sheet: C?, FB?, FL?, J?, U?

Commit message: Update.
Parts:
- removed J4: 031-6233, symbol Connector:Conn_Coaxial
- added C353: 0.1uF, Resistor_SMD:R_0402_1005Metric_Pad0.72x0.64mm_HandSolder, symbol Device:C
- added FB16: FerriteBead, Inductor_SMD:L_0402_1005Metric_Pad0.77x0.64mm_HandSolder, symbol Device:FerriteBead
- added FL2: Filter_EMI_CommonMode, symbol Device:Filter_EMI_CommonMode
- added J10: Micro_SD_Card_Det, symbol Connector:Micro_SD_Card_Det
- added J12, J13, J14, J16, J17, J18: 5-1634503-1, 5-1634503-1, symbol Connector:Conn_Coaxial
- added J5: USB_B, Connector_USB:USB_B_OST_USB-B1HSxx_Horizontal, symbol Connector:USB_B
- added J6: Conn_02x05_Odd_Even, symbol Connector_Generic:Conn_02x05_Odd_Even
- added J7: DB9_Male, symbol Connector:DB9_Male
- added J8: HDMI_A, Connector_HDMI:HDMI_A_Contact_Technology_HDMI-19APL2_Horizontal, symbol Connector:HDMI_A
- added J9: RJ45_Amphenol_RJMG1BD3B8K1ANR, Connector_RJ:RJ45_Amphenol_RJMG1BD3B8K1ANR, symbol Connector:RJ45_Amphenol_RJMG1BD3B8K1ANR
- added R128, R129, R130, R131, R132: 49.9, Resistor_SMD:R_0402_1005Metric_Pad0.72x0.64mm_HandSolder, symbol Device:R_US
- added SW1: SW_Push, symbol Switch:SW_Push
- added SW2: SW_DIP_x04, symbol Switch:SW_DIP_x04
- added U39: MAX3232, symbol Interface_UART:MAX3232
- C354, C355: renamed from C?; footprint (none) -> Resistor_SMD:R_0402_1005Metric_Pad0.72x0.64mm_HandSolder
- FB14, FB15: renamed from FB?; footprint (none) -> Inductor_SMD:L_0402_1005Metric_Pad0.77x0.64mm_HandSolder
- J11: renamed from J?; value 031-6233 -> 5-1634503-1; footprint (none) -> 5-1634503-1; Part Number (none) -> 5-1634503-1
- J15: renamed from J3; value 031-6233 -> 5-1634503-1; footprint (none) -> 5-1634503-1; Part Number (none) -> 5-1634503-1
- J3: renamed from J?; footprint (none) -> Connector_USB:USB_A_Molex_67643_Horizontal
- R133, R134, R135: renamed from R?; footprint (none) -> Resistor_SMD:R_0402_1005Metric_Pad0.72x0.64mm_HandSolder
- gave numbers to parts that had none: 3
- renumbered J2 to J4
Connections:
- net GND: now also J15.2 (Ext), C353.2, FB16.2, J10.6 (VSS), J16.2 (Ext), R129.2, R130.2, R131.2, R132.2, SW1.1; no longer J4.36 (GND), J4.38 (GND), J4.48 (GND), J4.5 (GND)
- net USB_N: no longer FL1.3, J3.2 (D-)
- net USB_P: no longer FL1.1, J3.3 (D+)
- net 3095_1_OUT: now reaches J15.1 (In)
- net USB_5V renamed OTG_VBUS
- net OTG_VBUS: now also C353.1
- net USB_F_P renamed OTG_DN
- net OTG_DN: no longer FL1.2
- new net: J9.R4 (TCT), J9.R5 (RCT)
- new net: FB16.1, J10.11 (SHIELD)
- new net: J4.36 (GND), J4.38 (GND), J4.48 (GND), J4.5 (GND)
- new net: FL2.1, J5.3 (D+)
- new net: FL2.3, J5.2 (D-)
- new net 3.3V_SW_DELAYED: SW2.4
- new net 3095_2_OUT: J16.1 (In)
- new net 3V0_STBY: SW2.1, SW2.2, SW2.3
- new net BOOT_M0: R131.1, SW2.6
- new net BOOT_M1: R130.1, SW2.7
- new net ETH_RX_N: J9.R3 (RD+)
- new net ETH_RX_P: J9.R6 (RD-)
- new net ETH_TX_N: J9.R2 (TD-)
- new net ETH_TX_P: J9.R1 (TD+)
- new net H1_DN: FL2.4
- new net H1_DP: FL2.2
- new net JTAG_NRST: J6.10 (Pin_10)
- new net JTAG_TCK: J6.4 (Pin_4)
- new net JTAG_TDI: J6.8 (Pin_8)
- new net JTAG_TDO: J6.6 (Pin_6)
- new net JTAG_TMS: J6.2 (Pin_2)
- new net OTG_DP: FL1.2
- new net OTG_N: FL1.3, J3.2 (D-)
- new net OTG_P: FL1.1, J3.3 (D+)
- new net RST_SW: R128.1, SW1.2
- new net SD_CLK: J10.5 (CLK)
- new net SD_CMD: J10.3 (CMD)
- new net SD_D0: J10.7 (DAT0)
- new net SD_D1: J10.8 (DAT1)
- new net SD_D2: J10.1 (DAT2)
- new net SD_D3: J10.2 (DAT3/CD)
- new net SPI_NOR_WP: R129.1, SW2.8
- new net TAMPER: R132.1, SW2.5
- no-connect marks 5 -> 6
Other:
- note added: "BOOT&SPI CNTRL"
- note added: "ETHERNET"
- note added: "FORCED MPU REBOOT"
- note added: "HDMI"
- note added: "LVDS"
- note added: "RS232"
- note added: "SD CARD"
- note added: "USB HOST"
- note added: "USB OTG"
- note removed: "USB"
- moved on the sheet: C352, C354, C355, FB14, FB15, FL1, J11, J15, J3, R133, R134, R135

Commit message: Update.
Parts:
- removed FL2: Filter_EMI_CommonMode, symbol Device:Filter_EMI_CommonMode
- removed J12, J14: 5-1634503-1, 5-1634503-1, symbol Connector:Conn_Coaxial
- removed J5: USB_B, Connector_USB:USB_B_OST_USB-B1HSxx_Horizontal, symbol Connector:USB_B
- removed J7: DB9_Male, symbol Connector:DB9_Male
- removed U39: MAX3232, symbol Interface_UART:MAX3232
- added U39: TPD12S520DBT, Package_SO:TSSOP-38_4.4x9.7mm_P0.5mm, symbol Interface_HDMI:TPD12S520DBT
- J10: footprint (none) -> Connector_Card:microSD_HC_Hirose_DM3AT-SF-PEJM5
- SW2: footprint (none) -> Connector_PinHeader_1.27mm:PinHeader_2x04_P1.27mm_Vertical
- renumbered C352 to C362, C353 to C363, C354 to C364, C355 to C365, U38 to U37
Connections:
- net HDMI_D2_P: now reaches J8.1 (D2+)
- net HDMI_D2_P: now also U39.35 (TMDS_D2+), U39.4 (TMDS_D2+)
- net HDMI_CLK_P: now reaches J8.10 (CK+)
- net HDMI_CLK_P: now also U39.13 (TMDS_CK+), U39.26 (TMDS_CK+)
- net HDMI_CLK_N: now reaches J8.12 (CK-)
- net HDMI_CLK_N: now also U39.15 (TMDS_CK-), U39.24 (TMDS_CK-)
- net HDMI_D2_N: now reaches J8.3 (D2-)
- net HDMI_D2_N: now also U39.33 (TMDS_D2-), U39.6 (TMDS_D2-)
- net HDMI_D1_P: now reaches J8.4 (D1+)
- net HDMI_D1_P: now also U39.32 (TMDS_D1+), U39.7 (TMDS_D1+)
- net HDMI_D1_N: now reaches J8.6 (D1-)
- net HDMI_D1_N: now also U39.30 (TMDS_D1-), U39.9 (TMDS_D1-)
- net HDMI_D0_P: now reaches J8.7 (D0+)
- net HDMI_D0_P: now also U39.10 (TMDS_D0+), U39.29 (TMDS_D0+)
- net HDMI_D0_N: now reaches J8.9 (D0-)
- net HDMI_D0_N: now also U39.12 (TMDS_D0-), U39.27 (TMDS_D0-)
- new net: U39.11 (TMDS_GND), U39.14 (TMDS_GND), U39.25 (TMDS_GND), U39.28 (TMDS_GND), U39.31 (TMDS_GND), U39.34 (TMDS_GND), U39.5 (TMDS_GND), U39.8 (TMDS_GND)
- new net: U39.3 (GND), U39.36 (GND)
- no-connect marks 6 -> 5
Other:
- note removed: "RS232"
- note removed: "USB HOST"
- moved on the sheet: J8

Commit message: Update.
Parts:
- removed C362: 220uF, awg1000:EEE-FK1H221GP, symbol awg1000:CAP_POL
- removed J17: 5-1634503-1, 5-1634503-1, symbol Connector:Conn_Coaxial
- removed J8: HDMI_A, Connector_HDMI:HDMI_A_Contact_Technology_HDMI-19APL2_Horizontal, symbol Connector:HDMI_A
- added C361, C362: 22uF, Resistor_SMD:R_0402_1005Metric_Pad0.72x0.64mm_HandSolder, symbol awg1000:CAP_UNPOL
- added J2: 10029449-111RLF, awg1000:10029449-111RLF, symbol awg1000:10029449-111RLF
- C363, C364, C365: symbol Device:C -> awg1000:CAP_UNPOL
- FL1: value Filter_EMI_CommonMode -> 0603USB-251MLC; footprint (none) -> Inductor_SMD:L_CommonModeChoke_Coilcraft_0603USB; symbol Device:Filter_EMI_CommonMode -> awg1000:ommon Mode Filter Choke
- J3: value USB1040-GF-L-B -> 0676432910; footprint Connector_USB:USB_A_Molex_67643_Horizontal -> awg1000:USB_A_Molex_67643_Horizontal
- J9: value RJ45_Amphenol_RJMG1BD3B8K1ANR -> RJMG1BD3B8K1ANR; footprint Connector_RJ:RJ45_Amphenol_RJMG1BD3B8K1ANR -> awg1000:RJ45_Amphenol_RJMG1BD3B8K1ANR
- R128, R129, R130, R131, R132, R133, R134, R135: symbol Device:R_US -> awg1000:R
Connections:
- net CDC-PRIREF+: now also R133.1, R134.2; no longer R133.2, R134.1
- net GND: now also R133.2, R135.2, C361.2, C362.2; no longer R133.1, R135.1
- net HDMI_CLK_N: now also J2.12 (CK-)
- net HDMI_CLK_P: now also J2.10 (CK+)
- net HDMI_D0_N: now also J2.9 (D0-)
- net HDMI_D0_P: now also J2.7 (D0+)
- net HDMI_D1_N: now also J2.6 (D1-)
- net HDMI_D1_P: now also J2.4 (D1+)
- net HDMI_D2_N: now also J2.3 (D2-)
- net HDMI_D2_P: now also J2.1 (D2+)
- net OTG_DN: now also FL1.3; no longer FL1.4
- net OTG_N: now also FL1.4; no longer FL1.3
- net VBUS: now also C361.1, C362.1
- net at C365.2, J11.1 (In): now also R135.1; no longer R135.2
Other:
- note added: "BNC CONNECTORS"
- note added: "EXTERNAL REF. I/O"
- note removed: "INTERFACE BNC CONNECTORS"
- note removed: "LVDS"
- moved on the sheet: J11, J18, R133, R134, R135
