File: hardware/01-ECAD/01-KiCAD Files/AWG1000/PM.kicad_sch (KiCad schematic)
At the start: 4 parts

Commit message: WIP: update
Parts:
- removed C?: 220uF, symbol Device:C_Polarized_US
- added C1, C2: 220uF, awg1000:EEE-FK1H221GP, symbol awg1000:CAP_POL
- added J1: B4P-VH(LF)(SN), Connector_JST:JST_VH_B4P-VH_1x04_P3.96mm_Vertical, symbol awg1000:CONN4X1
- added U3: MCIMX6L8DVN10AB, symbol awg1000:MCIMX6L8DVN10AB
- gave numbers to parts that had none: 3
Connections:
- net GND: now also C1.2, C2.2, J1.1, J1.2, U3.A1 (GND1), U3.A24 (GND4), U3.A4 (GND2), U3.A7 (GND3), U3.AA1 (GND88), U3.AA2 (GND89), U3.AB10 (GND91), U3.AB14 (GND92), U3.AB18 (GND93), U3.AC18 (GND94), U3.AD1 (GND96), U3.AD24 (GND95), U3.AD4 (GND97), U3.AD7 (GND98), U3.C10 (GND6), U3.C14 (GND7), U3.C19 (GND8), U3.C6 (GND5), U3.D1 (GND9), U3.D2 (GND10), U3.E5 (GND11), U3.G1 (GND12), U3.G10 (GND15), U3.G11 (GND16), U3.G13 (GND17), U3.G14 (GND18), U3.G15 (GND19), U3.G17 (GND20), U3.G18 (GND21), U3.G8 (GND13), U3.G9 (GND14), U3.H18 (GND24), U3.H22 (GND25), U3.H3 (GND22), U3.H7 (GND23), U3.J5 (GND26), U3.K1 (GND27), U3.L10 (GND31), U3.L11 (GND32), U3.L12 (GND33), U3.L13 (GND34), U3.L14 (GND35), U3.L15 (GND36), U3.L16 (GND37), U3.L7 (GND29), U3.L9 (GND30), U3.M10 (GND43), U3.M11 (GND44), U3.M12 (GND45), U3.M13 (GND46), U3.M14 (GND47), U3.M15 (GND48), U3.M16 (GND49), U3.M17 (GND38), U3.M5 (GND39), U3.M7 (GND40), U3.M8 (GND41), U3.M9 (GND42), U3.N10 (GND54), U3.N11 (GND55), U3.N12 (GND56), U3.N13 (GND57), U3.N14 (GND58), U3.N15 (GND59), U3.N16 (GND60), U3.N17 (GND50), U3.N22 (GND70), U3.N3 (GND28), U3.N7 (GND51), U3.N8 (GND52), U3.N9 (GND53), U3.P10 (GND62), U3.P11 (GND63), U3.P12 (GND64), U3.P13 (GND65), U3.P14 (GND66), U3.P15 (GND67), U3.P16 (GND68), U3.P9 (GND61), U3.R1 (GND69), U3.T5 (GND71), U3.U18 (GND74), U3.U22 (GND90), U3.U3 (GND72), U3.U7 (GND73), U3.V1 (GND75), U3.V10 (GND78), U3.V11 (GND79), U3.V12 (GND80), U3.V13 (GND81), U3.V14 (GND82), U3.V15 (GND83), U3.V16 (GND84), U3.V17 (GND85), U3.V18 (GND86), U3.V8 (GND76), U3.V9 (GND77), U3.Y5 (GND87)
- new net VCC: C1.1, C2.1, J1.3, J1.4
Other:
- note added: "MPU GND"
- note added: "MPU PMIC"
- note added: "POWER INPUT"
- note removed: "POWER MANAGEMENT"
- moved on the sheet: C3

Commit message: WIP.
Parts:
- added TP1, TP2: TestPoint, symbol awg1000:TestPoint
- added unit 8 of U1
- C1, C2: Voltage 50V -> V
- J1: Part Number (none) -> B4P-VH(LF)(SN)
- renumbered U3 to U1, U1 to U2
Connections:
- net GND: now also TP2.1
- net VCC renamed VIN_ACDC
- net VIN_ACDC: now also TP1.1
- new net 1V2_DDR_SW: U1.A24 (VDD_ARM_CAP6), U1.H18 (DRAM_PWR5), U1.L10 (DRAM_PWR6), U1.L11 (VDD_SOC_CAP8), U1.N16 (VDD_HIGH_IN4), U1.N8 (DRAM_PWR2), U1.N9 (DRAM_PWR7), U1.U18 (VDD_SOC_CAP1), U1.U7 (DRAM_PWR4), U1.V15 (VDD_ARM_CAP2)
- new net VDD_ARM_CAP: U1.A24 (VDD_ARM_CAP6), U1.A7 (VDD_ARM_CAP5), U1.C10 (VDD_PLL_CAP), U1.C6 (VDD_ARM_CAP7), U1.V14 (VDD_ARM_CAP1), U1.V15 (VDD_ARM_CAP2), U1.V16 (VDD_ARM_CAP3), U1.V17 (VDD_ARM_CAP4)
- new net VDD_ARM_IN: U1.A1 (VDD_ARM_IN5), U1.A4 (VDD_ARM_IN6), U1.AD7 (VDD_ARM_IN4), U1.V11 (VDD_ARM_IN1), U1.V12 (VDD_ARM_IN2), U1.V13 (VDD_ARM_IN3)
- new net VDD_HIGH_CAP: U1.M10 (VDD_HIGH_CAP1), U1.M11 (VDD_HIGH_CAP2), U1.P10 (VDD_HIGH_CAP4), U1.P9 (VDD_SNVS_IN)
- new net VDD_PU_CAP: U1.L15 (VDD_PU_CAP1), U1.L16 (VDD_PU_CAP2), U1.M17 (VDD_PU_CAP3), U1.N10 (VDD_PU_CAP4), U1.N11 (VDD_PU_CAP5), U1.N12 (VDD_PU_CAP6)
- new net VDD_SNVS_CAP: U1.V10 (VDD_SOC_IN2)
- new net VDD_SOC_CAP: U1.AB18 (VDD_SOC_CAP4), U1.AC18 (VDD_SOC_CAP5), U1.AD24 (VDD_SOC_CAP6), U1.H22 (VDD_SOC_CAP7), U1.L11 (VDD_SOC_CAP8), U1.M14 (VDD_SOC_CAP9), U1.U18 (VDD_SOC_CAP1), U1.V1 (VDD_SOC_CAP2), U1.V8 (VDD_SOC_CAP3)
- new net VDD_SOC_IN: U1.AD1 (VDD_SOC_IN3), U1.AD4 (VDD_SOC_IN4), U1.M12 (VDD_SOC_IN5), U1.M13 (VDD_SOC_IN6), U1.M5 (VDD_PU_IN1), U1.M7 (VDD_PU_IN2), U1.N13 (VDD_PU_IN3), U1.N14 (VDD_PU_IN4), U1.P11 (VDD_SOC_IN7), U1.P12 (VDD_SOC_IN8), U1.P13 (VDD_SOC_IN9), U1.V10 (VDD_SOC_IN2), U1.V9 (VDD_SOC_IN1)
Other:
- moved on the sheet: U1I

Commit message: WIP.
Parts:
- removed C3: 0.1uF, symbol Device:C
- added C? (x8): 22uF, symbol Device:C
- added C? (x10): 4.7uF, symbol Device:C
- added C?: 0.1uF, symbol Device:C
- added C? (x8): 0.22uF, symbol Device:C
- added D?: D_TVS, symbol Device:D_TVS
- added D?: D_Schottky, symbol Device:D_Schottky
- added L? (x5): 1uH, symbol Device:L
- added R? (x14): 0, symbol Device:R_US
- added U?: TPS61165DBVR, symbol awg1000:TPS61165DBVR
Connections:
- net GND: now also C4.1, U2.12 (GNDREF1), U2.2 (SD_VSEL), U2.26 (GNDREF2), U2.40 (GNDREF), U2.5 (ICTEST), C?.2, C?.2, C?.2, C?.2, C?.2, C?.2, C?.2, C?.2, C?.2, C?.2, C?.2, C?.2, C?.2, C?.2, C?.2, C?.2, C?.2, C?.2, C?.2, C?.2, C?.2, C?.2, C?.2, C?.2, C?.2, C?.2, D?.1 (A1), R?.1, R?.1, R?.2, U?.4 (GND)
- net PF3000_VIN: now also U2.10 (SW1BIN), U2.18 (SW2IN), U2.28 (SW3IN), U2.38 (SWBSTFB), U2.7 (SW1AIN), C?.1, C?.1, C?.1, L?.1, L?.1, R?.1, R?.1, R?.1
- net VDD_ARM_IN: now also U2.6 (SW1AFB), C?.1, C?.1
- net VDD_SOC_IN: now also U2.11 (SW1BFB), C?.1, C?.1
- net VIN_ACDC: now also D?.2 (A2)
- net at C4.2: now also U2.44 (VCOREREF)
- net REF_CLK_24M: now reaches U2.1 (~INT)
- net VLDO1IN: now reaches U2.13 (VLDO1IN)
- net VLDO1IN: now also C?.1, R?.2, R?.2
- net 1V8_VLDO1: now reaches U2.14 (VLDO1)
- net 1V8_VLDO1: now also C?.1
- net 1V5_VLDO2: now reaches U2.15 (VLDO2)
- net 1V5_VLDO2: now also C?.1
- net VLDO2IN: now reaches U2.16 (VLDO2IN)
- net VLDO2IN: now also C?.1, R?.2, R?.2
- net at U2.17 (SW2LX): now also L?.2
- net 3V15_VDDHIGH_SW2: now reaches U2.19 (SW2FB)
- net 3V15_VDDHIGH_SW2: now also U2.47 (VDDIO), C?.1, C?.1, L?.1, R?.1, R?.1, R?.1
- net 3V0_VLDO3: now reaches U2.20 (VLDO3)
- net VLDO3IN: now reaches U2.21 (VLDO34IN)
- net VLDO3IN: now also C?.1, R?.2, R?.2
- net 1V8_VLDO4: now reaches U2.22 (VLDO4)
- net 1V8_VLDO4: now also C?.1
- net at U2.23 (VHALF): now also C?.1, C?.2
- net at U2.24 (VINREFDDR): now also C?.1
- net DRAM_VREF: now reaches U2.25 (VREFDDR)
- net DRAM_VREF: now also C?.1
- net 1V2_DDR_SW3: now reaches U2.27 (SW3FB)
- net 1V2_DDR_SW3: now also C?.1, C?.1, L?.2
- net at U2.29 (SW3LX): now also L?.1
- net at U2.3 (RESETBMCU): now also R?.2
- net at U2.31 (VPWR): now also R?.2
- net 2V8_VGEN6: now reaches U2.32 (V33)
- net 2V8_VGEN6: now also C?.1
- net VCC_SDX: now reaches U2.33 (VCC_SD)
- net 3V0_VSNVS: now reaches U2.34 (VSNVS)
- net 3V0_VSNVS: now also C?.1, C?.1
- net at U2.39 (VDDOTP): now also R?.1
- net PMIC_STBY_REQ: now reaches U2.4 (STANDBY)
- net at U2.41 (VCORE): now also C?.1
- net VCOREDIG: now reaches U2.43 (VCOREDIG)
- net at U2.45 (SDA): now also R?.2
- net at U2.48 (PWRON): now also R?.2, R?.2
- net at U2.64 (SCL): now also R?.2
- net at U2.8 (SW1ALX): now also L?.2
- net at U2.9 (SW1BLX): now also L?.2
- new net: C?.1, U?.5 (COMP)
- new net: C?.1, L?.1, U?.1 (VIN)
- new net: D?.2 (A), L?.2, U?.3 (SW)
- new net 3V0_STBY: R?.1
- new net BCKLT_CTRL: U?.2 (CTRL)
- new net PMIC_ON_REQ: R?.1, R?.1, R?.1
- new net POR_B: R?.1
- new net V: C?.1, D?.1 (K), R?.2, U?.6 (FB)
- no-connect marks 0 -> 1
Other:
- note added: "LCD BACKLIGHT DRIVER"
- moved on the sheet: C1, C2, C4, TP1, TP2, U1H, U1I, U2

Commit message: Update.
Parts:
- removed C? (x8): 22uF, symbol Device:C
- removed C? (x10): 4.7uF, symbol Device:C
- removed C?: 0.1uF, symbol Device:C
- removed C? (x8): 0.22uF, symbol Device:C
- removed D?: D_Schottky, symbol Device:D_Schottky
- removed L? (x5): 1uH, symbol Device:L
- removed R? (x14): 0, symbol Device:R_US
- removed U1: MCIMX6L8DVN10AB, symbol awg1000:MCIMX6L8DVN10AB
- removed U2: MC34PF3000A5EP, Package_DFN_QFN:NXP_LQFN-48-1EP_7x7mm_P0.5mm_EP3.5x3.5mm_16xMask0.45x0.45_ThermalVias, symbol awg1000:MC34PF3000A5EP
- removed U?: TPS61165DBVR, symbol awg1000:TPS61165DBVR
- added C1, C104, C106, C15, C2, C3, C41, C45, C46, C5, C56, C95: 4.7uF, awg1000:C0402_L, symbol Device:C
- added C10, C11, C12, C14, C40, C49, C50, C51, C52, C53, C6, C7, C70, C9: 0.47uF, Resistor_SMD:R_0402_1005Metric_Pad0.72x0.64mm_HandSolder, symbol Device:C
- added C100, C101, C103, C105, C107, C108, C110, C83, C84, C85, C86, C87, C88, C89, C90, C91, C92, C93, C94, C96, C97, C98, C99: 22uF, Capacitor_SMD:C_0603_1608Metric_Pad1.08x0.95mm_HandSolder, symbol Device:C
- added C102, C109, C111, C112, C24, C31, C35, C38, C43, C44, C61, C64, C73, C75: 220nF, Resistor_SMD:R_0402_1005Metric_Pad0.72x0.64mm_HandSolder, symbol Device:C
- added C16, C18, C19, C20, C23, C47, C55, C58, C66, C76: 33uF, Capacitor_SMD:CP_Elec_6.3x7.7, symbol awg1000:CAP_POL
- added C17, C21, C22, C25, C26, C27, C28, C29, C30, C32, C33, C34, C36, C37, C39, C42, C48, C54, C57, C59, C60, C62, C63, C65, C67, C68, C69, C71, C72, C74, C77, C78, C79, C80, C81, C82: 10uF, Capacitor_SMD:C_1206_3216Metric, symbol Device:C
- added D2, D3, D4, D5: D_Schottky, symbol Device:D_Schottky
- added L1, L10, L2, L3, L4, L5, L6, L7, L8, L9: 47uH, Inductor_SMD:L_Bourns_SRR1260, symbol Device:L
- added L11: 1uH, symbol Device:L
- added L12, L13, L14, L15: 1uH, awg1000:74404024010, symbol Device:L
- added R1, R18, R23, R24, R25, R26, R27, R28, R29, R30, R31, R32, R33, R34: 0, Resistor_SMD:R_0402_1005Metric_Pad0.72x0.64mm_HandSolder, symbol Device:R_US
- added R10, R11, R13, R15, R19, R20, R3, R5, R7, R9: 7.15k, Resistor_SMD:R_0402_1005Metric_Pad0.72x0.64mm_HandSolder, symbol Device:R_US
- added R12, R14, R16, R2, R21, R4, R6, R8: 100k, Resistor_SMD:R_0402_1005Metric_Pad0.72x0.64mm_HandSolder, symbol Device:R_US
- added R17, R22: 16.5k, Resistor_SMD:R_0402_1005Metric_Pad0.72x0.64mm_HandSolder, symbol Device:R_US
- added TP3: TestPoint, symbol awg1000:TestPoint
- added U1, U10, U2, U3, U4, U6, U7, U8: LMR23610ADDA, Package_SO:SOIC-8-1EP_3.9x4.9mm_P1.27mm_EP2.29x3mm_ThermalVias, symbol awg1000:LMR23610ADDA
- added U11, U12: MCP1702T-3302E_CB, Package_TO_SOT_SMD:SOT-23, symbol awg1000:MCP1702T-3302E_CB
- added U13, U14: MCP1702T-1202E_CB, Package_TO_SOT_SMD:SOT-23, symbol awg1000:MCP1702T-1202E_CB
- added U15: TPS61165DBVR, symbol awg1000:TPS61165DBVR
- added U16: MMPF0100F3ANES, Package_DFN_QFN:QFN-56-1EP_8x8mm_P0.5mm_EP4.3x4.3mm_ThermalVias, symbol awg1000:MMPF0100F3ANES
- added U5, U9: TPS54531DDA, Package_SO:SOIC-8-1EP_3.9x4.9mm_P1.27mm_EP2.29x3mm_ThermalVias, symbol awg1000:TPS54531DDA
- C4: value 0.1uF -> 4.7uF; footprint (none) -> awg1000:C0402_L; Part Number (none) -> C1005X5R1A475K050BE; VOLTAGE 50V -> 10V
- D1: renamed from D?; footprint (none) -> Diode_SMD:D_SMC
- TP1, TP2: footprint (none) -> TestPoint:TestPoint_Pad_D1.0mm
- renumbered C2 to C13, C1 to C8
Connections:
- net 3V0_STBY: now also D4.1 (K), U16.43 (VSNVS)
- net BCKLT_CTRL: now also U15.2 (CTRL)
- net GND: now also C100.1, C101.1, C102.1, C103.1, C104.2, C105.1, C106.2, C107.1, C108.1, C109.2, C110.1, C112.2, C15.1, C16.2, C17.1, C18.2, C19.2, C2.1, C20.2, C21.1, C22.2, C23.2, C24.1, C25.1, C26.2, C27.1, C28.2, C29.1, C3.1, C30.1, C31.2, C32.1, C33.2, C34.1, C35.2, C36.1, C37.1, C38.2, C39.1, C41.1, C42.1, C43.2, C44.1, C46.1, C47.2, C48.1, C5.1, C51.2, C53.2, C54.1, C55.2, C56.1, C57.1, C58.2, C59.1, C60.2, C61.1, C62.1, C63.1, C64.2, C65.1, C66.2, C67.1, C7.2, C71.1, C72.2, C73.1, C74.1, C75.2, C76.2, C79.1, C80.1, C83.1, C84.1, C85.1, C86.2, C87.1, C88.1, C89.1, C9.2, C90.2, C91.1, C92.1, C93.1, C94.2, C95.2, C96.1, C97.1, C98.1, C99.2, L2.2, L8.2, R11.2, R13.1, R15.1, R16.1, R20.2, R22.1, R29.1, R3.1, R32.1, R33.1, R4.1, R7.1, R9.1, U1.6 (AGND), U1.8 (PGND), U1.9 (PAD), U10.6 (AGND), U10.8 (PGND), U10.9 (PAD), U11.1 (GND), U12.1 (GND), U13.1 (GND), U14.1 (GND), U15.4 (GND), U16.14 (SW1VSSSNS), U16.15 (GREF1), U16.32 (SW3VSSSNS), U16.48 (GNDREF), U16.57 (EPAD), U3.6 (AGND), U3.8 (PGND), U3.9 (PAD), U4.6 (AGND), U4.8 (PGND), U4.9 (PAD), U5.7 (GND), U6.6 (AGND), U6.8 (PGND), U6.9 (PAD), U7.6 (AGND), U7.8 (PGND), U7.9 (PAD), U9.7 (GND)
- net PMIC_ON_REQ: now also R25.1
- net V: now also C106.1, D5.1 (K), R32.2, U15.6 (FB)
- net VCOREDIG: now also R34.1, U16.51 (VCOREDIG)
- net VDD_ARM_IN: now also C84.2, C88.2, C92.2, C97.2, L12.1, U16.6 (SW1FB)
- net VDD_SOC_IN: now also C100.2, C101.2, C103.2, L13.1, U16.13 (SW1CFB)
- net VIN_ACDC: now also C17.2, C22.1, C24.2, C26.1, C28.1, C31.1, C33.1, C35.1, C36.2, C38.1, C43.1, C44.2, C57.2, C60.1, C61.2, C64.1, C65.2, C72.1, C73.2, C75.1, U1.5 (EN/SYNC), U1.7 (VIN), U10.5 (EN/SYNC), U10.7 (VIN), U2.5 (EN/SYNC), U2.7 (VIN), U3.5 (EN/SYNC), U3.7 (VIN), U4.5 (EN/SYNC), U4.7 (VIN), U5.2 (VIN), U5.3 (EN), U6.5 (EN/SYNC), U6.7 (VIN), U7.5 (EN/SYNC), U7.7 (VIN), U8.5 (EN/SYNC), U8.7 (VIN), U9.2 (VIN), U9.3 (EN)
- net at C4.2: now also U3.3 (VCC)
- new net: C52.1, L8.1, U8.1 (SW)
- new net: C52.2, U8.2 (BOOT)
- new net: R4.2, R5.2, U2.4 (FB)
- new net: R10.2, R11.1, U5.5 (VSNS)
- new net: C51.1, R18.1
- new net: C53.1, R18.2, U9.6 (COMP)
- new net: C7.1, R1.1
- new net: C9.1, R1.2, U5.6 (COMP)
- new net: C19.1, C27.2, C37.2
- new net: C95.1, L11.1, U15.1 (VIN)
- new net: D5.2 (A), L11.2, U15.3 (SW)
- new net: C104.1, U15.5 (COMP)
- new net: C49.1, L7.1, U7.1 (SW)
- new net: C111.2, C112.1, U16.29 (VHALF)
- new net: R19.2, R20.1, U9.5 (VSNS)
- new net: R8.2, R9.2, U4.4 (FB)
- new net: C109.1, U16.49 (VCORE)
- new net: C1.2, U2.3 (VCC)
- new net: R14.2, R15.2, U7.4 (FB)
- new net: C70.1, L10.1, U10.1 (SW)
- new net: C70.2, U10.2 (BOOT)
- new net: C102.2, U16.52 (VCOREREF)
- new net: C12.1, L3.1, U3.1 (SW)
- new net: C12.2, U3.2 (BOOT)
- new net: R6.2, R7.2, U3.4 (FB)
- new net: C11.1, L2.1, U2.1 (SW)
- new net: C11.2, U2.2 (BOOT)
- new net: R27.2, U16.53 (SDA)
- new net: C49.2, U7.2 (BOOT)
- new net: C14.1, L4.1, U4.1 (SW)
- new net: C14.2, U4.2 (BOOT)
- new net: C10.1, L1.1, U1.1 (SW)
- new net: L15.1, U16.35 (SW3BLX), U16.36 (SW3ALX)
- new net: C45.2, U8.3 (VCC)
- new net: R12.2, R13.2, U6.4 (FB)
- new net: R16.2, R17.2, U8.4 (FB)
- new net: C40.1, L6.1, U6.1 (SW)
- new net: C40.2, U6.2 (BOOT)
- new net: R24.1, R25.2, R26.2
- new net: C41.2, U7.3 (VCC)
- new net: C10.2, U1.2 (BOOT)
- new net: R23.2, R24.2, U16.56 (PWRON)
- new net: C15.2, U6.3 (VCC)
- new net: C3.2, U5.4 (SS)
- new net: R21.2, R22.2, U10.4 (FB)
- new net: C6.1, L5.1, U5.8 (PH)
- new net: C5.2, U4.3 (VCC)
- new net: C50.2, U9.1 (BOOT)
- new net: C46.2, U9.4 (SS)
- new net: C50.1, L9.1, U9.8 (PH)
- new net: C56.2, U10.3 (VCC)
- new net: C6.2, U5.1 (BOOT)
- new net: R33.2, R34.2, U16.47 (VDDOTP)
- new net: R30.1, U16.2 (SDWNB)
- new net: R2.2, R3.2, U1.4 (FB)
- new net: C2.2, U1.3 (VCC)
- new net: L13.2, U16.11 (SW1CLX)
- new net: L14.2, U16.22 (SW2LX)
- new net: R29.2, U16.5 (ICTEST)
- new net: R28.2, U16.54 (SCL)
- new net: L12.2, U16.8 (SW1ALX), U16.9 (SW1BLX)
- new net +15V: C47.1, C48.2, C54.2, L6.2, R12.1, TP3.1
- new net +7V: C76.1, C79.2, C80.2, L10.2, R21.1
- new net +VREF_DDR: U16.31 (VREFDDR)
- new net -15V: C1.1, C20.1, C29.2, C39.2, R5.1, U2.6 (AGND), U2.8 (PGND), U2.9 (PAD)
- new net -7V: C45.1, C58.1, C62.2, C67.2, R17.1, U8.6 (AGND), U8.8 (PGND), U8.9 (PAD)
- new net 1.2V_DAC: U13.2 (VOUT)
- new net 1.2V_DAC_CLK: U14.2 (VOUT)
- new net 1.2V_DAC_DVDD: C55.1, C59.2, C63.2, L4.2, L7.2, R14.1, R8.1
- new net 1.5V_DDR: C111.1, C83.2, C87.2, C91.2, C96.2, L15.2, U16.30 (VINREFDDR), U16.38 (SW3AFB)
- new net 1.5V_GEN2: U16.18 (VGEN2)
- new net 1.8V_SW: C108.2, C110.2
- new net 1V8_GEN4: U16.28 (VGEN4)
- new net 2.5V_FPGA: C18.1, C25.2, C34.2, L3.2, R6.1
- new net 2.5V_GEN5: U16.39 (VGEN5)
- new net 3.3V_DAC_AN: U11.2 (VOUT)
- new net 3.3V_DAC_IO: U12.2 (VOUT)
- new net 3.3V_SW: C23.1, C32.2, C42.2, C85.2, C86.1, C89.2, C90.1, C93.2, C94.1, C98.2, C99.1, L5.2, R10.1, R23.1, R30.2, R31.2, U16.10 (SW1BIN), U16.12 (SW1CIN), U16.17 (VIN1), U16.23 (SW2IN_1), U16.24 (SW2IN_2), U16.27 (VIN2), U16.34 (SW3BIN), U16.37 (SW3AIN), U16.40 (VIN3), U16.50 (VIN), U16.7 (SW1AIN)
- new net 3.3V_SW_DELAYED: C66.1, C71.2, C74.2, L9.2, R19.1, U16.55 (VDDIO)
- new net 3.6V: C16.1, C21.2, C30.2, L1.2, R2.1, U11.3 (VIN), U12.3 (VIN), U13.3 (VIN), U14.3 (VIN)
- new net 3V_VDDHIGH: C105.2, C107.2, D4.2 (A), L14.1, U16.25 (SW2FB)
- new net IMX_POR: U16.3 (RESETBMCU)
- new net PMIC_I2C_SCL: R28.1
- new net PMIC_I2C_SDA: R27.1
- new net PMIC_INT_B: R31.1, U16.1 (INTB)
- new net PMIC_STDBY: U16.4 (STANDBY)
- no-connect marks 1 -> 9
Other:
- note added: "-15V SMPS"
- note added: "-7V SMPS"
- note added: "15V SMPS"
- note added: "3.3V/XA"
- note added: "7V SMPS"
- note added: "DAC PWR"
- note added: "FPGA 3.3V"
- note added: "FPGA VCC CORE"
- note added: "PERIPHERAL SMPS"
- note added: "PMIC_VIN"
- note removed: "MPU GND"

Commit message: Update.
Parts:
- added C346, C352: 10uF, Capacitor_SMD:C_1206_3216Metric, symbol Device:C
- added H1, H2, H3, H4: MountingHole_Pad, MountingHole:MountingHole_3.2mm_M3_ISO7380_Pad_TopBottom, symbol Mechanical:MountingHole_Pad
- C102, C109, C111, C112, C24, C31, C35, C38, C43, C44, C61, C64, C73, C75: footprint Resistor_SMD:R_0402_1005Metric_Pad0.72x0.64mm_HandSolder -> awg1000:C0201_L
- L11: footprint (none) -> awg1000:74404024010
- U15: footprint (none) -> Package_TO_SOT_SMD:SOT-23-6_Handsoldering
Connections:
- net 1.2V_DAC: now also C81.2
- net 1.2V_DAC_CLK: now also C82.2
- net 1.2V_DAC_DVDD: now also C19.1, C27.2, C37.2
- net 3.3V_DAC_AN: now also C77.2
- net 3.3V_DAC_IO: now also C346.2
- net 3.6V: now also C68.2, C69.2, C78.2, C352.2
- net GND: now also C68.1, C69.1, C77.1, C78.1, C81.1, C82.1, C346.1, C352.1, H1.1, H2.1, H3.1, H4.1
Other:
- moved on the sheet: C68, C69, C77, C78, C81

Commit message: Update.
Parts:
- removed C346, C68: 10uF, Capacitor_SMD:C_1206_3216Metric, symbol Device:C
- removed J1: B4P-VH(LF)(SN), Connector_JST:JST_VH_B4P-VH_1x04_P3.96mm_Vertical, symbol awg1000:CONN4X1
- removed U12: MCP1702T-3302E_CB, Package_TO_SOT_SMD:SOT-23, symbol awg1000:MCP1702T-3302E_CB
- added J1: B2P-VH(LF)(SN), awg1000:JST_VH_B2P-VH-B_1x02_P3.96mm_Vertical, symbol awg1000:CONN_2X1
- C1, C104, C106, C15, C2, C3, C4, C41, C45, C46, C5, C56, C95: footprint awg1000:C0402_L -> Capacitor_SMD:C_0402_1005Metric_Pad0.74x0.62mm_HandSolder; symbol Device:C -> awg1000:CAP_UNPOL; Part Number C1005X5R1A475K050BE -> (none)
- C10, C11, C12, C14, C40, C49, C50, C51, C52, C53, C6, C7, C70, C9: symbol Device:C -> awg1000:CAP_UNPOL; Part Number CGB2A1X5R1C474K033BC -> (none)
- C100, C101, C103, C105, C107, C108, C110, C83, C84, C85, C86, C87, C88, C89, C90, C91, C92, C93, C94, C96, C97, C98, C99: symbol Device:C -> awg1000:CAP_UNPOL
- C102, C109, C111, C112, C24, C31, C35, C38, C43, C44, C61, C64, C73, C75: symbol Device:C -> awg1000:CAP_UNPOL; Part Number UMK107B7224KA-TR -> (none)
- C17, C21, C22, C25, C26, C27, C28, C29, C30, C32, C33, C34, C352, C36, C37, C39, C42, C48, C54, C57, C59, C60, C62, C63, C65, C67, C69, C71, C72, C74, C77, C78, C79, C80, C81, C82: symbol Device:C -> awg1000:CAP_UNPOL; Part Number C3216X7R1H106K160AE -> (none)
- R1, R12, R14, R16, R18, R2, R21, R23, R24, R25, R26, R27, R28, R29, R30, R31, R32, R33, R34, R4, R6, R8: symbol Device:R_US -> awg1000:R
- R10, R11, R13, R15, R19, R20, R3, R5, R7, R9: symbol Device:R_US -> awg1000:R; Part Number RC0402FR-137K15L -> (none)
- R17, R22: symbol Device:R_US -> awg1000:R; Part Number CRCW040216K5FKEDC -> (none)
- U1, U10, U2, U3, U4, U5, U6, U7, U8, U9: footprint Package_SO:SOIC-8-1EP_3.9x4.9mm_P1.27mm_EP2.29x3mm_ThermalVias -> awg1000:SOIC-8-1EP_3.9x4.9mm_P1.27mm_EP2.29x3mm_ThermalVias
- U16: footprint Package_DFN_QFN:QFN-56-1EP_8x8mm_P0.5mm_EP4.3x4.3mm_ThermalVias -> awg1000:QFN-56-1EP_8x8mm_P0.5mm_EP4.3x4.3mm_ThermalVias
Connections:
- net +15V: now also C48.1, C54.1; no longer C48.2, C54.2
- net +7V: now also C79.1, C80.1; no longer C79.2, C80.2
- net 1.2V_DAC_CLK: now also C82.1; no longer C82.2
- net 1.2V_DAC_DVDD: now also C27.1, C37.1, C59.1, C63.1; no longer C27.2, C37.2, C59.2, C63.2
- net 2.5V_FPGA: now also C25.1, C34.1; no longer C25.2, C34.2
- net 3.3V_DAC_AN: now also C77.1; no longer C77.2
- net 3.3V_SW: now also C32.1, C42.1, R30.1, R31.1; no longer C32.2, C42.2, R30.2, R31.2
- net 3.3V_SW_DELAYED: now also C71.1, C74.1; no longer C71.2, C74.2
- net 3.6V: now also C21.1, C30.1, C352.1, C69.1, C78.1; no longer C21.2, C30.2, C352.2, C69.2, C78.2
- net GND: now also C15.2, C2.2, C21.2, C22.1, C25.2, C26.1, C27.2, C28.1, C3.2, C30.2, C31.1, C32.2, C33.1, C34.2, C35.1, C352.2, C37.2, C38.1, C4.2, C41.2, C42.2, C43.1, C46.2, C48.2, C5.2, C51.1, C54.2, C56.2, C59.2, C60.1, C63.2, C64.1, C69.2, C7.1, C71.2, C72.1, C74.2, C75.1, C77.2, C78.2, C79.2, C80.2, C81.2, C82.2, C9.1, U5.5 (VSNS), U5.9 (PAD), U9.5 (VSNS), U9.9 (PAD), J1.2; no longer C15.1, C2.1, C21.1, C22.2, C25.1, C26.2, C27.1, C28.2, C3.1, C30.1, C31.2, C32.1, C33.2, C34.1, C35.2, C352.1, C37.1, C38.2, C4.1, C41.1, C42.1, C43.2, C46.1, C48.1, C5.1, C51.2, C54.1, C56.1, C59.1, C60.2, C63.1, C64.2, C69.1, C7.2, C71.1, C72.2, C74.1, C75.2, C77.1, C78.1, C79.1, C80.1, C81.1, C82.1, C9.2, U5.7 (GND), U9.7 (GND)
- net PMIC_INT_B: now also R31.2; no longer R31.1
- net VIN_ACDC: now also C22.2, C26.2, C28.2, C31.2, C33.2, C35.2, C38.2, C43.2, C60.2, C64.2, C72.2, C75.2, J1.1; no longer C22.1, C26.1, C28.1, C31.1, C33.1, C35.1, C38.1, C43.1, C60.1, C64.1, C72.1, C75.1
- net at R10.2, R11.1: now also U5.7 (GND); no longer U5.5 (VSNS)
- net at R18.1: now also C53.1; no longer C51.1
- net at R18.2, U9.6 (COMP): now also C51.2; no longer C53.1
- net at R1.1: now also C9.2; no longer C7.1
- net at R1.2, U5.6 (COMP): now also C7.2; no longer C9.1
- net at U4.3 (VCC): now also C5.1; no longer C5.2
- net at L7.1, U7.1 (SW): now also C49.2; no longer C49.1
- net at R19.2, R20.1: now also U9.7 (GND); no longer U9.5 (VSNS)
- net at L10.1, U10.1 (SW): now also C70.2; no longer C70.1
- net at U10.2 (BOOT): now also C70.1; no longer C70.2
- net at L3.1, U3.1 (SW): now also C12.2; no longer C12.1
- net at U3.2 (BOOT): now also C12.1; no longer C12.2
- net at U7.2 (BOOT): now also C49.1; no longer C49.2
- net at L4.1, U4.1 (SW): now also C14.2; no longer C14.1
- net at U4.2 (BOOT): now also C14.1; no longer C14.2
- net at L1.1, U1.1 (SW): now also C10.2; no longer C10.1
- net at U3.3 (VCC): now also C4.1; no longer C4.2
- net at L6.1, U6.1 (SW): now also C40.2; no longer C40.1
- net at U6.2 (BOOT): now also C40.1; no longer C40.2
- net at U7.3 (VCC): now also C41.1; no longer C41.2
- net at U1.2 (BOOT): now also C10.1; no longer C10.2
- net at U6.3 (VCC): now also C15.1; no longer C15.2
- net at U5.4 (SS): now also C3.1; no longer C3.2
- net at L5.1, U5.8 (PH): now also C6.2; no longer C6.1
- net at U9.4 (SS): now also C46.1; no longer C46.2
- net at U10.3 (VCC): now also C56.1; no longer C56.2
- net at U5.1 (BOOT): now also C6.1; no longer C6.2
- net at U16.2 (SDWNB): now also R30.2; no longer R30.1
- net at U1.3 (VCC): now also C2.1; no longer C2.2
- net 1.2V_DAC renamed 1.2V_DAC_VDD
- net 1.2V_DAC_VDD: now also C81.1; no longer C81.2
- no-connect marks 9 -> 33
Other:
- note added: "-15V 1A SMPS"
- note added: "-7V 1A SMPS"
- note added: "15V 1A SMPS"
- note added: "3.3V 5A PERIPHERALS SMPS"
- note added: "3.3V 5A PMIC_VIN"
- note added: "7V 1A SMPS"
- note added: "LDO"
- note added: "POWER SUPPLIES TREE"
- note added: "SW"
- note removed: "-15V SMPS"
- note removed: "-7V SMPS"
- note removed: "15V SMPS"
- note removed: "7V SMPS"
- note removed: "PERIPHERAL SMPS"
- note removed: "PMIC_VIN"
- moved on the sheet: C47, C76, D5, H1, H2, H3, H4, L10, L11, L6, R1, R12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
