File: hardware/01-ECAD/01-KiCAD Files/FPGA.kicad_sch (KiCad schematic)
At the start: 5 parts, among them U24 AS4C256M16D3LC-12BCN, U25 AS4C256M16D3LC-12BCN, U8 10CX085YU484I6G

Commit message: Update.
Parts:
- added C27 (x6): 33uF, Capacitor_Tantalum_SMD:CP_EIA-3528-12_Kemet-T, symbol awg1000:CAP_POL
- added C35 (x20): 10uF, Capacitor_SMD:C_0402_1005Metric, symbol awg1000:CAP_UNPOL
- added FB5 (x2): FerriteBead, Inductor_SMD:L_0402_1005Metric_Pad0.77x0.64mm_HandSolder, symbol Device:FerriteBead
- added R8, R9: 2K, awg1000:C0201_L, symbol awg1000:R
Connections:
- net 1.5V_DDR is gone; now on net FPGA_1.5V: U24.A1 (VDDQ), U24.A8 (VDDQ), U24.B2 (VDD), U24.C1 (VDDQ), U24.C9 (VDDQ), U24.D2 (VDDQ), U24.D9 (VDD), U24.E9 (VDDQ), U24.F1 (VDDQ), U24.G7 (VDD), U24.H2 (VDDQ), U24.H9 (VDDQ), U24.K2 (VDD), U24.K8 (VDD), U24.N1 (VDD), U24.N9 (VDD), U24.R1 (VDD), U24.R9 (VDD), U25.A1 (VDDQ), U25.A8 (VDDQ), U25.B2 (VDD), U25.C1 (VDDQ), U25.C9 (VDDQ), U25.D2 (VDDQ), U25.D9 (VDD), U25.E9 (VDDQ), U25.F1 (VDDQ), U25.G7 (VDD), U25.H2 (VDDQ), U25.H9 (VDDQ), U25.K2 (VDD), U25.K8 (VDD), U25.N1 (VDD), U25.N9 (VDD), U25.R1 (VDD), U25.R9 (VDD)
- net DRAM_DQS2_P: no longer U25.G3 (~{LDQS})
- net FPGA_0.9V: now also U8.K12 (VCCP), U8.K14 (VCCP), U8.N15 (VCCERAM), U8.N8 (VCCERAM), U8.P12 (VCCP), U8.P14 (VCCP), C27.1, C27.1, C27.1, C27.1, C27.1, C27.1, C35.1, C35.1, C35.1, C35.1, C35.1, C35.1, C35.1, C35.1, C35.2, C35.2, C35.2, C35.2, C35.2, C35.2, C35.2, C35.2, C35.2, C35.2, C35.2, C35.2
- net GND: now also C27.2, C27.2, C27.2, C27.2, C27.2, C27.2, C35.1, C35.1, C35.1, C35.1, C35.1, C35.1, C35.1, C35.1, C35.1, C35.1, C35.1, C35.1, C35.2, C35.2, C35.2, C35.2, C35.2, C35.2, C35.2, C35.2, R8.1, R9.1
- net at U8.A22 (RREF_TL): now also R9.2
- net at U8.AB19 (RREF_BL): now also R8.2
- net FPGA_IO_1.8V: now reaches U8.C9 (VCCIO2L)
- net FPGA_IO_1.8V: now also U8.D11 (VCCIO2L), U8.F10 (VCCIO2L), U8.T9 (VCCPGM), U8.U9 (VCCPGM), U8.V9 (VCCIO2A), U8.W6 (VCCIO2A), U8.Y8 (VCCIO2A)
- net FPGA_1.5V: now reaches U8.D16 (VCCIO2K)
- net FPGA_1.5V: now also U8.F15 (VCCIO2K), U8.H14 (VCCIO2K), U8.T15 (VCCIO2J), U8.U12 (VCCIO2J), U8.V14 (VCCIO2J)
- net TSDN: now reaches U8.E4 (TEMPDIODEn)
- net TSDP: now reaches U8.E5 (TEMPDIODEp)
- net FPGA_1.8V: now reaches U8.J14 (VCCPT)
- net FPGA_1.8V: now also U8.J8 (VCCPT), U8.R14 (VCCPT), U8.R9 (VCCPT), U8.T8 (VCCBAT), FB5.1, FB5.1
- net FPGA_0.95V: now reaches U8.J19 (VCCR_GXBL1C)
- net FPGA_0.95V: now also U8.J20 (VCCR_GXBL1C), U8.N19 (VCCT_GXBL1C), U8.N20 (VCCT_GXBL1C)
- net at U8.L19 (VCCH_GXBL): now also FB5.2
- net at U8.M11 (VCCA_PLL): now also U8.M13 (VCCA_PLL), FB5.2
- net VCCCSNS: now reaches U8.M8 (VCCLSENSE)
- net GNDCSNS: now reaches U8.M9 (GNDSENSE)
- new net DRAM_DQS2_N: U25.G3 (~{LDQS})
Other:
- moved on the sheet: U8A, U8B, U8C, U8D, U8E, U8F, U8G
