File: hardware/01-ECAD/01-KiCAD Files/PM.kicad_sch (KiCad schematic)
At the start: 124 parts, among them J2 B4P-VH(LF)(SN), U1 MCP1702T-1202E_CB, U11 LMR23610ADDA, U12 LMR23610ADDA, U2 LMR23610ADDA, U2 SIC402ACD-T1-GE3, U3 TPS61165DBVR, U4 MCP1702T-3302E_CB, U5 LMR23610ADDA, U5 MP2147GD-Z, U6 MCP1702T-1202E_CB, U7 LMR23610ADDA, U9 LMR23610ADDA

Commit message: Update.
Parts:
- added C17: 2.2uF, Capacitor_SMD:C_0402_1005Metric, symbol DQSBC:C
- added C74 (x3), C78 (x3): 100nF, Capacitor_SMD:C_0201_0603Metric, symbol awg1000:CAP_UNPOL
- added C75 (x3), C76 (x3), C77 (x3): 22uF, Capacitor_SMD:C_0603_1608Metric, symbol awg1000:CAP_UNPOL
- added L6: 47uH, Inductor_SMD:L_Vishay_IHLP-6767, symbol Device:L
- added L8 (x3): 0.47uH, Inductor_SMD:L_1008_2520Metric, symbol Device:L
- added R25 (x3): 180K, Resistor_SMD:R_0402_1005Metric_Pad0.72x0.64mm_HandSolder, symbol awg1000:R
- added R26 (x3): 360K, Resistor_SMD:R_0402_1005Metric_Pad0.72x0.64mm_HandSolder, symbol awg1000:R
- added R5 (x2): 7.15k, Resistor_SMD:R_0402_1005Metric, symbol awg1000:R
- added U10: ~, awg1000:SIC431AED-T1-GE3, symbol awg1000:SIC431AED-T1-GE3
- added U5 (x3): MP2147GD-Z, awg1000:MP2147GD-Z, symbol DQSBC:MP2147GD-Z
Connections:
- net 3.3V_SW_DELAYED is gone; now on net 3.3V_SW: C76.2, C78.2, U5.11 (VIN2), U5.8 (VIN1)
- net 3.3V_SW: now also C76.2, C76.2, C76.2, C78.2, C78.2, C78.2, U10.1 (VIN1), U10.2 (VIN2), U10.22 (VIN3), U10.26 (VIN4), U5.11 (VIN2), U5.11 (VIN2), U5.11 (VIN2), U5.8 (VIN1), U5.8 (VIN1), U5.8 (VIN1)
- net FPGA_0.9V: now also L6.2, R5.1, U10.18 (VOUT); no longer C74.1, C75.1, C77.1, L8.2, R25.1, U5.2 (OUT)
- net FPGA_1.5V: now also C74.1, C75.1, C77.1, L8.2, R25.1, U5.2 (OUT)
- net FPGA_1.8V: now also C74.1, C75.1, C77.1, L8.2, R25.1, U5.2 (OUT)
- net GND: now also C74.2, C74.2, C74.2, C75.2, C75.2, C75.2, C76.1, C76.1, C76.1, C77.2, C77.2, C77.2, C78.1, C78.1, C78.1, R26.2, R26.2, R26.2, R5.2, U10.13 (PGND3), U10.16 (AGND1), U10.25 (AGND2), U10.27 (PGND4), U10.3 (PGND1), U10.4 (PGND2), U5.10 (GND), U5.10 (GND), U5.10 (GND)
- net P_MODE: now also U5.6 (MODE), U5.6 (MODE), U5.6 (MODE); no longer U5.6 (MODE)
- new net: R25.2, R26.1, U5.3 (FB) (x3)
- new net: C17.1, U10.23 (BOOT)
- new net: C17.2, U10.24 (PHASE)
- new net: L8.1, U5.1 (SW), U5.9 (SW) (x3)
- new net: R5.1, R5.2, U10.17 (VFB)
- new net: L6.1, U10.5 (SW1), U10.6 (SW2), U10.7 (SW3), U10.8 (SW4), U10.9 (SW5)
- new net FPGA_0.95V: C74.1, C75.1, C77.1, L8.2, R25.1, U5.2 (OUT)
- new net FPGA_IO_1.8V: C74.1, C75.1, C77.1, L8.2, R25.1, U5.2 (OUT)
- no-connect marks 4 -> 13
Other:
- moved on the sheet: C1, C10, C11, C13, C14, C15, C16, C17, C18, C19, C2, C20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
